Commit message: add modification to vertex conflict resolution to fix conflict tree getting infinitely expanded wrongly

File: assets/warehouse/shelves.urdf (robot description, URDF)
Before this commit: robot struct, 421 links, 420 joints
Links:
- removed link block_10_10
- removed link block_10_11
- removed link block_10_13
- removed link block_10_14
- removed link block_10_15
- removed link block_10_16
- removed link block_10_17
- removed link block_10_18
- removed link block_10_19
- removed link block_10_2
- removed link block_10_20
- removed link block_10_21
- removed link block_10_22
- removed link block_10_24
- removed link block_10_25
- removed link block_10_26
- removed link block_10_27
- removed link block_10_28
- removed link block_10_29
- removed link block_10_3
- removed link block_10_30
- removed link block_10_31
- removed link block_10_32
- removed link block_10_33
- removed link block_10_4
- removed link block_10_5
- removed link block_10_6
- removed link block_10_7
- removed link block_10_8
- removed link block_10_9
- removed link block_11_10
- removed link block_11_11
- removed link block_11_13
- removed link block_11_14
- removed link block_11_15
- removed link block_11_16
- removed link block_11_17
- removed link block_11_18
- removed link block_11_19
- removed link block_11_2
- removed link block_11_20
- removed link block_11_21
- removed link block_11_22
- removed link block_11_24
- removed link block_11_25
- removed link block_11_26
- removed link block_11_27
- removed link block_11_28
- removed link block_11_29
- removed link block_11_3
- removed link block_11_30
- removed link block_11_31
- removed link block_11_32
- removed link block_11_33
- removed link block_11_4
- removed link block_11_5
- removed link block_11_6
- removed link block_11_7
- removed link block_11_8
- removed link block_11_9
- removed link block_14_10
- removed link block_14_11
- removed link block_14_13
- removed link block_14_14
- removed link block_14_15
- removed link block_14_16
- removed link block_14_17
- removed link block_14_18
- removed link block_14_19
- removed link block_14_2
- removed link block_14_20
- removed link block_14_21
- removed link block_14_22
- removed link block_14_24
- removed link block_14_25
- removed link block_14_26
- removed link block_14_27
- removed link block_14_28
- removed link block_14_29
- removed link block_14_3
- removed link block_14_30
- removed link block_14_31
- removed link block_14_32
- removed link block_14_33
- removed link block_14_4
- removed link block_14_5
- removed link block_14_6
- removed link block_14_7
- removed link block_14_8
- removed link block_14_9
- removed link block_15_10
- removed link block_15_11
- removed link block_15_13
- removed link block_15_14
- removed link block_15_15
- removed link block_15_16
- removed link block_15_17
- removed link block_15_18
- removed link block_15_19
- removed link block_15_2
- removed link block_15_20
- removed link block_15_21
- removed link block_15_22
- removed link block_15_24
- removed link block_15_25
- removed link block_15_26
- removed link block_15_27
- removed link block_15_28
- removed link block_15_29
- removed link block_15_3
- removed link block_15_30
- removed link block_15_31
- removed link block_15_32
- removed link block_15_33
- removed link block_15_4
- removed link block_15_5
- removed link block_15_6
- removed link block_15_7
- removed link block_15_8
- removed link block_15_9
- removed link block_18_10
- removed link block_18_11
- removed link block_18_13
- removed link block_18_14
- removed link block_18_15
- removed link block_18_16
- removed link block_18_17
- removed link block_18_18
- removed link block_18_19
- removed link block_18_2
- removed link block_18_20
- removed link block_18_21
- removed link block_18_22
- removed link block_18_24
- removed link block_18_25
- removed link block_18_26
- removed link block_18_27
- removed link block_18_28
- removed link block_18_29
- removed link block_18_3
- removed link block_18_30
- removed link block_18_31
- removed link block_18_32
- removed link block_18_33
- removed link block_18_4
- removed link block_18_5
- removed link block_18_6
- removed link block_18_7
- removed link block_18_8
- removed link block_18_9
- removed link block_19_10
- removed link block_19_11
- removed link block_19_13
- removed link block_19_14
- removed link block_19_15
- removed link block_19_16
- removed link block_19_17
- removed link block_19_18
- removed link block_19_19
- removed link block_19_2
- removed link block_19_20
- removed link block_19_21
- removed link block_19_22
- removed link block_19_24
- removed link block_19_25
- removed link block_19_26
- removed link block_19_27
- removed link block_19_28
- removed link block_19_29
- removed link block_19_3
- removed link block_19_30
- removed link block_19_31
- removed link block_19_32
- removed link block_19_33
- removed link block_19_4
- removed link block_19_5
- removed link block_19_6
- removed link block_19_7
- removed link block_19_8
- removed link block_19_9
- removed link block_22_10
- removed link block_22_11
- removed link block_22_13
- removed link block_22_14
- removed link block_22_15
- removed link block_22_16
- removed link block_22_17
- removed link block_22_18
- removed link block_22_19
- removed link block_22_2
- removed link block_22_20
- removed link block_22_21
- removed link block_22_22
- removed link block_22_24
- removed link block_22_25
- removed link block_22_26
- removed link block_22_27
- removed link block_22_28
- removed link block_22_29
- removed link block_22_3
- removed link block_22_30
- removed link block_22_31
- removed link block_22_32
- removed link block_22_33
- removed link block_22_4
- removed link block_22_5
- removed link block_22_6
- removed link block_22_7
- removed link block_22_8
- removed link block_22_9
- removed link block_23_10
- removed link block_23_11
- removed link block_23_13
- removed link block_23_14
- removed link block_23_15
- removed link block_23_16
- removed link block_23_17
- removed link block_23_18
- removed link block_23_19
- removed link block_23_2
- removed link block_23_20
- removed link block_23_21
- removed link block_23_22
- removed link block_23_24
- removed link block_23_25
- removed link block_23_26
- removed link block_23_27
- removed link block_23_28
- removed link block_23_29
- removed link block_23_3
- removed link block_23_30
- removed link block_23_31
- removed link block_23_32
- removed link block_23_33
- removed link block_23_4
- removed link block_23_5
- removed link block_23_6
- removed link block_23_7
- removed link block_23_8
- removed link block_23_9
- removed link block_26_10
- removed link block_26_11
- removed link block_26_13
- removed link block_26_14
- removed link block_26_15
- removed link block_26_16
- removed link block_26_17
- removed link block_26_18
- removed link block_26_19
- removed link block_26_2
- removed link block_26_20
- removed link block_26_21
- removed link block_26_22
- removed link block_26_24
- removed link block_26_25
- removed link block_26_26
- removed link block_26_27
- removed link block_26_28
- removed link block_26_29
- removed link block_26_3
- removed link block_26_30
- removed link block_26_31
- removed link block_26_32
- removed link block_26_33
- removed link block_26_4
- removed link block_26_5
- removed link block_26_6
- removed link block_26_7
- removed link block_26_8
- removed link block_26_9
- removed link block_27_10
- removed link block_27_11
- removed link block_27_13
- removed link block_27_14
- removed link block_27_15
- removed link block_27_16
- removed link block_27_17
- removed link block_27_18
- removed link block_27_19
- removed link block_27_2
- removed link block_27_20
- removed link block_27_21
- removed link block_27_22
- removed link block_27_24
- removed link block_27_25
- removed link block_27_26
- removed link block_27_27
- removed link block_27_28
- removed link block_27_29
- removed link block_27_3
- removed link block_27_30
- removed link block_27_31
- removed link block_27_32
- removed link block_27_33
- removed link block_27_4
- removed link block_27_5
- removed link block_27_6
- removed link block_27_7
- removed link block_27_8
- removed link block_27_9
- removed link block_2_10
- removed link block_2_11
- removed link block_2_13
- removed link block_2_14
- removed link block_2_15
- removed link block_2_16
- removed link block_2_17
- removed link block_2_18
- removed link block_2_19
- removed link block_2_20
- removed link block_2_21
- removed link block_2_22
- removed link block_2_24
- removed link block_2_25
- removed link block_2_26
- removed link block_2_27
- removed link block_2_28
- removed link block_2_29
- removed link block_2_30
- removed link block_2_31
- removed link block_2_32
- removed link block_2_33
- removed link block_2_4
- removed link block_2_5
- removed link block_2_6
- removed link block_2_7
- removed link block_2_8
- removed link block_2_9
- removed link block_3_10
- removed link block_3_11
- removed link block_3_13
- removed link block_3_14
- removed link block_3_15
- removed link block_3_16
- removed link block_3_17
- removed link block_3_18
- removed link block_3_19
- removed link block_3_2
- removed link block_3_20
- removed link block_3_21
- removed link block_3_22
- removed link block_3_24
- removed link block_3_25
- removed link block_3_26
- removed link block_3_27
- removed link block_3_28
- removed link block_3_29
- removed link block_3_3
- removed link block_3_30
- removed link block_3_31
- removed link block_3_32
- removed link block_3_33
- removed link block_3_4
- removed link block_3_5
- removed link block_3_6
- removed link block_3_7
- removed link block_3_8
- removed link block_3_9
- removed link block_6_10
- removed link block_6_11
- removed link block_6_13
- removed link block_6_14
- removed link block_6_15
- removed link block_6_16
- removed link block_6_17
- removed link block_6_18
- removed link block_6_19
- removed link block_6_2
- removed link block_6_20
- removed link block_6_21
- removed link block_6_22
- removed link block_6_24
- removed link block_6_25
- removed link block_6_26
- removed link block_6_27
- removed link block_6_28
- removed link block_6_29
- removed link block_6_3
- removed link block_6_30
- removed link block_6_31
- removed link block_6_32
- removed link block_6_33
- removed link block_6_4
- removed link block_6_5
- removed link block_6_6
- removed link block_6_7
- removed link block_6_8
- removed link block_6_9
- removed link block_7_10
- removed link block_7_11
- removed link block_7_13
- removed link block_7_14
- removed link block_7_15
- removed link block_7_16
- removed link block_7_17
- removed link block_7_18
- removed link block_7_19
- removed link block_7_2
- removed link block_7_20
- removed link block_7_21
- removed link block_7_22
- removed link block_7_24
- removed link block_7_25
- removed link block_7_26
- removed link block_7_27
- removed link block_7_28
- removed link block_7_29
- removed link block_7_3
- removed link block_7_30
- removed link block_7_31
- removed link block_7_32
- removed link block_7_33
- removed link block_7_4
- removed link block_7_5
- removed link block_7_6
- removed link block_7_7
- removed link block_7_8
- removed link block_7_9
- added link block_0_2, mass 0; collision box size=0.7 0.7 0.7; visual box size=1.0 1.0 1
- added link block_1_2, mass 0; collision box size=0.7 0.7 0.7; visual box size=1.0 1.0 1
- added link block_2_1, mass 0; collision box size=0.7 0.7 0.7; visual box size=1.0 1.0 1
Joints:
- removed joint joint_block_10_10
- removed joint joint_block_10_11
- removed joint joint_block_10_13
- removed joint joint_block_10_14
- removed joint joint_block_10_15
- removed joint joint_block_10_16
- removed joint joint_block_10_17
- removed joint joint_block_10_18
- removed joint joint_block_10_19
- removed joint joint_block_10_2
- removed joint joint_block_10_20
- removed joint joint_block_10_21
- removed joint joint_block_10_22
- removed joint joint_block_10_24
- removed joint joint_block_10_25
- removed joint joint_block_10_26
- removed joint joint_block_10_27
- removed joint joint_block_10_28
- removed joint joint_block_10_29
- removed joint joint_block_10_3
- removed joint joint_block_10_30
- removed joint joint_block_10_31
- removed joint joint_block_10_32
- removed joint joint_block_10_33
- removed joint joint_block_10_4
- removed joint joint_block_10_5
- removed joint joint_block_10_6
- removed joint joint_block_10_7
- removed joint joint_block_10_8
- removed joint joint_block_10_9
- removed joint joint_block_11_10
- removed joint joint_block_11_11
- removed joint joint_block_11_13
- removed joint joint_block_11_14
- removed joint joint_block_11_15
- removed joint joint_block_11_16
- removed joint joint_block_11_17
- removed joint joint_block_11_18
- removed joint joint_block_11_19
- removed joint joint_block_11_2
- removed joint joint_block_11_20
- removed joint joint_block_11_21
- removed joint joint_block_11_22
- removed joint joint_block_11_24
- removed joint joint_block_11_25
- removed joint joint_block_11_26
- removed joint joint_block_11_27
- removed joint joint_block_11_28
- removed joint joint_block_11_29
- removed joint joint_block_11_3
- removed joint joint_block_11_30
- removed joint joint_block_11_31
- removed joint joint_block_11_32
- removed joint joint_block_11_33
- removed joint joint_block_11_4
- removed joint joint_block_11_5
- removed joint joint_block_11_6
- removed joint joint_block_11_7
- removed joint joint_block_11_8
- removed joint joint_block_11_9
- removed joint joint_block_14_10
- removed joint joint_block_14_11
- removed joint joint_block_14_13
- removed joint joint_block_14_14
- removed joint joint_block_14_15
- removed joint joint_block_14_16
- removed joint joint_block_14_17
- removed joint joint_block_14_18
- removed joint joint_block_14_19
- removed joint joint_block_14_2
- removed joint joint_block_14_20
- removed joint joint_block_14_21
- removed joint joint_block_14_22
- removed joint joint_block_14_24
- removed joint joint_block_14_25
- removed joint joint_block_14_26
- removed joint joint_block_14_27
- removed joint joint_block_14_28
- removed joint joint_block_14_29
- removed joint joint_block_14_3
- removed joint joint_block_14_30
- removed joint joint_block_14_31
- removed joint joint_block_14_32
- removed joint joint_block_14_33
- removed joint joint_block_14_4
- removed joint joint_block_14_5
- removed joint joint_block_14_6
- removed joint joint_block_14_7
- removed joint joint_block_14_8
- removed joint joint_block_14_9
- removed joint joint_block_15_10
- removed joint joint_block_15_11
- removed joint joint_block_15_13
- removed joint joint_block_15_14
- removed joint joint_block_15_15
- removed joint joint_block_15_16
- removed joint joint_block_15_17
- removed joint joint_block_15_18
- removed joint joint_block_15_19
- removed joint joint_block_15_2
- removed joint joint_block_15_20
- removed joint joint_block_15_21
- removed joint joint_block_15_22
- removed joint joint_block_15_24
- removed joint joint_block_15_25
- removed joint joint_block_15_26
- removed joint joint_block_15_27
- removed joint joint_block_15_28
- removed joint joint_block_15_29
- removed joint joint_block_15_3
- removed joint joint_block_15_30
- removed joint joint_block_15_31
- removed joint joint_block_15_32
- removed joint joint_block_15_33
- removed joint joint_block_15_4
- removed joint joint_block_15_5
- removed joint joint_block_15_6
- removed joint joint_block_15_7
- removed joint joint_block_15_8
- removed joint joint_block_15_9
- removed joint joint_block_18_10
- removed joint joint_block_18_11
- removed joint joint_block_18_13
- removed joint joint_block_18_14
- removed joint joint_block_18_15
- removed joint joint_block_18_16
- removed joint joint_block_18_17
- removed joint joint_block_18_18
- removed joint joint_block_18_19
- removed joint joint_block_18_2
- removed joint joint_block_18_20
- removed joint joint_block_18_21
- removed joint joint_block_18_22
- removed joint joint_block_18_24
- removed joint joint_block_18_25
- removed joint joint_block_18_26
- removed joint joint_block_18_27
- removed joint joint_block_18_28
- removed joint joint_block_18_29
- removed joint joint_block_18_3
- removed joint joint_block_18_30
- removed joint joint_block_18_31
- removed joint joint_block_18_32
- removed joint joint_block_18_33
- removed joint joint_block_18_4
- removed joint joint_block_18_5
- removed joint joint_block_18_6
- removed joint joint_block_18_7
- removed joint joint_block_18_8
- removed joint joint_block_18_9
- removed joint joint_block_19_10
- removed joint joint_block_19_11
- removed joint joint_block_19_13
- removed joint joint_block_19_14
- removed joint joint_block_19_15
- removed joint joint_block_19_16
- removed joint joint_block_19_17
- removed joint joint_block_19_18
- removed joint joint_block_19_19
- removed joint joint_block_19_2
- removed joint joint_block_19_20
- removed joint joint_block_19_21
- removed joint joint_block_19_22
- removed joint joint_block_19_24
- removed joint joint_block_19_25
- removed joint joint_block_19_26
- removed joint joint_block_19_27
- removed joint joint_block_19_28
- removed joint joint_block_19_29
- removed joint joint_block_19_3
- removed joint joint_block_19_30
- removed joint joint_block_19_31
- removed joint joint_block_19_32
- removed joint joint_block_19_33
- removed joint joint_block_19_4
- removed joint joint_block_19_5
- removed joint joint_block_19_6
- removed joint joint_block_19_7
- removed joint joint_block_19_8
- removed joint joint_block_19_9
- removed joint joint_block_22_10
- removed joint joint_block_22_11
- removed joint joint_block_22_13
- removed joint joint_block_22_14
- removed joint joint_block_22_15
- removed joint joint_block_22_16
- removed joint joint_block_22_17
- removed joint joint_block_22_18
- removed joint joint_block_22_19
- removed joint joint_block_22_2
- removed joint joint_block_22_20
- removed joint joint_block_22_21
- removed joint joint_block_22_22
- removed joint joint_block_22_24
- removed joint joint_block_22_25
- removed joint joint_block_22_26
- removed joint joint_block_22_27
- removed joint joint_block_22_28
- removed joint joint_block_22_29
- removed joint joint_block_22_3
- removed joint joint_block_22_30
- removed joint joint_block_22_31
- removed joint joint_block_22_32
- removed joint joint_block_22_33
- removed joint joint_block_22_4
- removed joint joint_block_22_5
- removed joint joint_block_22_6
- removed joint joint_block_22_7
- removed joint joint_block_22_8
- removed joint joint_block_22_9
- removed joint joint_block_23_10
- removed joint joint_block_23_11
- removed joint joint_block_23_13
- removed joint joint_block_23_14
- removed joint joint_block_23_15
- removed joint joint_block_23_16
- removed joint joint_block_23_17
- removed joint joint_block_23_18
- removed joint joint_block_23_19
- removed joint joint_block_23_2
- removed joint joint_block_23_20
- removed joint joint_block_23_21
- removed joint joint_block_23_22
- removed joint joint_block_23_24
- removed joint joint_block_23_25
- removed joint joint_block_23_26
- removed joint joint_block_23_27
- removed joint joint_block_23_28
- removed joint joint_block_23_29
- removed joint joint_block_23_3
- removed joint joint_block_23_30
- removed joint joint_block_23_31
- removed joint joint_block_23_32
- removed joint joint_block_23_33
- removed joint joint_block_23_4
- removed joint joint_block_23_5
- removed joint joint_block_23_6
- removed joint joint_block_23_7
- removed joint joint_block_23_8
- removed joint joint_block_23_9
- removed joint joint_block_26_10
- removed joint joint_block_26_11
- removed joint joint_block_26_13
- removed joint joint_block_26_14
- removed joint joint_block_26_15
- removed joint joint_block_26_16
- removed joint joint_block_26_17
- removed joint joint_block_26_18
- removed joint joint_block_26_19
- removed joint joint_block_26_2
- removed joint joint_block_26_20
- removed joint joint_block_26_21
- removed joint joint_block_26_22
- removed joint joint_block_26_24
- removed joint joint_block_26_25
- removed joint joint_block_26_26
- removed joint joint_block_26_27
- removed joint joint_block_26_28
- removed joint joint_block_26_29
- removed joint joint_block_26_3
- removed joint joint_block_26_30
- removed joint joint_block_26_31
- removed joint joint_block_26_32
- removed joint joint_block_26_33
- removed joint joint_block_26_4
- removed joint joint_block_26_5
- removed joint joint_block_26_6
- removed joint joint_block_26_7
- removed joint joint_block_26_8
- removed joint joint_block_26_9
- removed joint joint_block_27_10
- removed joint joint_block_27_11
- removed joint joint_block_27_13
- removed joint joint_block_27_14
- removed joint joint_block_27_15
- removed joint joint_block_27_16
- removed joint joint_block_27_17
- removed joint joint_block_27_18
- removed joint joint_block_27_19
- removed joint joint_block_27_2
- removed joint joint_block_27_20
- removed joint joint_block_27_21
- removed joint joint_block_27_22
- removed joint joint_block_27_24
- removed joint joint_block_27_25
- removed joint joint_block_27_26
- removed joint joint_block_27_27
- removed joint joint_block_27_28
- removed joint joint_block_27_29
- removed joint joint_block_27_3
- removed joint joint_block_27_30
- removed joint joint_block_27_31
- removed joint joint_block_27_32
- removed joint joint_block_27_33
- removed joint joint_block_27_4
- removed joint joint_block_27_5
- removed joint joint_block_27_6
- removed joint joint_block_27_7
- removed joint joint_block_27_8
- removed joint joint_block_27_9
- removed joint joint_block_2_10
- removed joint joint_block_2_11
- removed joint joint_block_2_13
- removed joint joint_block_2_14
- removed joint joint_block_2_15
- removed joint joint_block_2_16
- removed joint joint_block_2_17
- removed joint joint_block_2_18
- removed joint joint_block_2_19
- removed joint joint_block_2_20
- removed joint joint_block_2_21
- removed joint joint_block_2_22
- removed joint joint_block_2_24
- removed joint joint_block_2_25
- removed joint joint_block_2_26
- removed joint joint_block_2_27
- removed joint joint_block_2_28
- removed joint joint_block_2_29
- removed joint joint_block_2_30
- removed joint joint_block_2_31
- removed joint joint_block_2_32
- removed joint joint_block_2_33
- removed joint joint_block_2_4
- removed joint joint_block_2_5
- removed joint joint_block_2_6
- removed joint joint_block_2_7
- removed joint joint_block_2_8
- removed joint joint_block_2_9
- removed joint joint_block_3_10
- removed joint joint_block_3_11
- removed joint joint_block_3_13
- removed joint joint_block_3_14
- removed joint joint_block_3_15
- removed joint joint_block_3_16
- removed joint joint_block_3_17
- removed joint joint_block_3_18
- removed joint joint_block_3_19
- removed joint joint_block_3_2
- removed joint joint_block_3_20
- removed joint joint_block_3_21
- removed joint joint_block_3_22
- removed joint joint_block_3_24
- removed joint joint_block_3_25
- removed joint joint_block_3_26
- removed joint joint_block_3_27
- removed joint joint_block_3_28
- removed joint joint_block_3_29
- removed joint joint_block_3_3
- removed joint joint_block_3_30
- removed joint joint_block_3_31
- removed joint joint_block_3_32
- removed joint joint_block_3_33
- removed joint joint_block_3_4
- removed joint joint_block_3_5
- removed joint joint_block_3_6
- removed joint joint_block_3_7
- removed joint joint_block_3_8
- removed joint joint_block_3_9
- removed joint joint_block_6_10
- removed joint joint_block_6_11
- removed joint joint_block_6_13
- removed joint joint_block_6_14
- removed joint joint_block_6_15
- removed joint joint_block_6_16
- removed joint joint_block_6_17
- removed joint joint_block_6_18
- removed joint joint_block_6_19
- removed joint joint_block_6_2
- removed joint joint_block_6_20
- removed joint joint_block_6_21
- removed joint joint_block_6_22
- removed joint joint_block_6_24
- removed joint joint_block_6_25
- removed joint joint_block_6_26
- removed joint joint_block_6_27
- removed joint joint_block_6_28
- removed joint joint_block_6_29
- removed joint joint_block_6_3
- removed joint joint_block_6_30
- removed joint joint_block_6_31
- removed joint joint_block_6_32
- removed joint joint_block_6_33
- removed joint joint_block_6_4
- removed joint joint_block_6_5
- removed joint joint_block_6_6
- removed joint joint_block_6_7
- removed joint joint_block_6_8
- removed joint joint_block_6_9
- removed joint joint_block_7_10
- removed joint joint_block_7_11
- removed joint joint_block_7_13
- removed joint joint_block_7_14
- removed joint joint_block_7_15
- removed joint joint_block_7_16
- removed joint joint_block_7_17
- removed joint joint_block_7_18
- removed joint joint_block_7_19
- removed joint joint_block_7_2
- removed joint joint_block_7_20
- removed joint joint_block_7_21
- removed joint joint_block_7_22
- removed joint joint_block_7_24
- removed joint joint_block_7_25
- removed joint joint_block_7_26
- removed joint joint_block_7_27
- removed joint joint_block_7_28
- removed joint joint_block_7_29
- removed joint joint_block_7_3
- removed joint joint_block_7_30
- removed joint joint_block_7_31
- removed joint joint_block_7_32
- removed joint joint_block_7_33
- removed joint joint_block_7_4
- removed joint joint_block_7_5
- removed joint joint_block_7_6
- removed joint joint_block_7_7
- removed joint joint_block_7_8
- removed joint joint_block_7_9
- added joint joint_block_0_2: type fixed, parent struct_base, child block_0_2, origin xyz=0.5 1.5 0.5 rpy=0 0 0
- added joint joint_block_1_2: type fixed, parent struct_base, child block_1_2, origin xyz=0.5 0.5 0.5 rpy=0 0 0
- added joint joint_block_2_1: type fixed, parent struct_base, child block_2_1, origin xyz=-0.5 -0.5 0.5 rpy=0 0 0
- joint joint_block_2_2: origin xyz=-15.5 12.5 0.5 rpy=0 0 0 -> xyz=0.5 -0.5 0.5 rpy=0 0 0
- joint joint_block_2_3: origin xyz=-14.5 12.5 0.5 rpy=0 0 0 -> xyz=1.5 -0.5 0.5 rpy=0 0 0
