Commit message: add modification to vertex conflict resolution to fix conflict tree getting infinitely expanded wrongly

File: assets/warehouse/workstations.urdf (robot description, URDF)
Before this commit: robot struct, 21 links, 20 joints
Links:
- removed link block_10_0
- removed link block_10_35
- removed link block_13_0
- removed link block_13_35
- removed link block_16_0
- removed link block_16_35
- removed link block_19_0
- removed link block_19_35
- removed link block_1_0
- removed link block_1_35
- removed link block_22_0
- removed link block_22_35
- removed link block_25_0
- removed link block_25_35
- removed link block_28_0
- removed link block_28_35
- removed link block_4_0
- removed link block_4_35
- removed link block_7_0
- removed link block_7_35
- added link block_0_0, mass 0; visual box size=1.0 1.0 1.5
- added link block_0_1, mass 0; visual box size=1.0 1.0 1.5
Joints:
- removed joint joint_block_10_0
- removed joint joint_block_10_35
- removed joint joint_block_13_0
- removed joint joint_block_13_35
- removed joint joint_block_16_0
- removed joint joint_block_16_35
- removed joint joint_block_19_0
- removed joint joint_block_19_35
- removed joint joint_block_1_0
- removed joint joint_block_1_35
- removed joint joint_block_22_0
- removed joint joint_block_22_35
- removed joint joint_block_25_0
- removed joint joint_block_25_35
- removed joint joint_block_28_0
- removed joint joint_block_28_35
- removed joint joint_block_4_0
- removed joint joint_block_4_35
- removed joint joint_block_7_0
- removed joint joint_block_7_35
- added joint joint_block_0_0: type fixed, parent struct_base, child block_0_0, origin xyz=-1.5 1.5 0.75 rpy=0 0 0
- added joint joint_block_0_1: type fixed, parent struct_base, child block_0_1, origin xyz=-0.5 1.5 0.75 rpy=0 0 0

Commit message: fix robots potentitally deadlocking when retriggering CBS after picking up a delivery

File: assets/warehouse/shelves.urdf (robot description, URDF)
Before this commit: robot struct, 6 links, 5 joints
Links:
- removed link block_0_2
- removed link block_1_2
Joints:
- removed joint joint_block_0_2
- removed joint joint_block_1_2

File: assets/warehouse/workstations.urdf (robot description, URDF)
Before this commit: robot struct, 3 links, 2 joints
Links:
- added link block_0_2, mass 0; visual box size=1.0 1.0 1.5
- added link block_0_3, mass 0; visual box size=1.0 1.0 1.5
Joints:
- added joint joint_block_0_2: type fixed, parent struct_base, child block_0_2, origin xyz=0.5 1.5 0.75 rpy=0 0 0
- added joint joint_block_0_3: type fixed, parent struct_base, child block_0_3, origin xyz=1.5 1.5 0.75 rpy=0 0 0

Commit message: remove commented code

File: assets/warehouse/shelves.urdf (robot description, URDF)
Before this commit: robot struct, 65 links, 64 joints
Links:
- removed link block_0_4
- removed link block_0_5
- removed link block_0_8
- removed link block_0_9
- removed link block_10_4
- removed link block_10_5
- removed link block_10_8
- removed link block_10_9
- removed link block_11_4
- removed link block_11_5
- removed link block_11_8
- removed link block_11_9
- removed link block_12_4
- removed link block_12_5
- removed link block_12_8
- removed link block_12_9
- removed link block_13_4
- removed link block_13_5
- removed link block_13_8
- removed link block_13_9
- removed link block_14_4
- removed link block_14_5
- removed link block_14_8
- removed link block_14_9
- removed link block_15_4
- removed link block_15_5
- removed link block_15_8
- removed link block_15_9
- removed link block_16_4
- removed link block_16_5
- removed link block_16_8
- removed link block_16_9
- removed link block_17_4
- removed link block_17_5
- removed link block_17_8
- removed link block_17_9
- removed link block_1_4
- removed link block_1_5
- removed link block_1_8
- removed link block_1_9
- removed link block_2_4
- removed link block_2_5
- removed link block_2_8
- removed link block_2_9
- removed link block_3_4
- removed link block_3_5
- removed link block_3_8
- removed link block_3_9
- removed link block_4_4
- removed link block_4_5
- removed link block_4_8
- removed link block_4_9
- removed link block_5_4
- removed link block_5_5
- removed link block_5_8
- removed link block_5_9
- removed link block_6_4
- removed link block_6_5
- removed link block_6_8
- removed link block_6_9
- removed link block_7_4
- removed link block_7_5
- removed link block_7_8
- removed link block_7_9
- added link block_0_2, mass 0; collision box size=0.7 0.7 0.7; visual box size=1.0 1.0 1
- added link block_1_2, mass 0; collision box size=0.7 0.7 0.7; visual box size=1.0 1.0 1
- added link block_2_1, mass 0; collision box size=0.7 0.7 0.7; visual box size=1.0 1.0 1
- added link block_2_2, mass 0; collision box size=0.7 0.7 0.7; visual box size=1.0 1.0 1
- added link block_2_3, mass 0; collision box size=0.7 0.7 0.7; visual box size=1.0 1.0 1
Joints:
- removed joint joint_block_0_4
- removed joint joint_block_0_5
- removed joint joint_block_0_8
- removed joint joint_block_0_9
- removed joint joint_block_10_4
- removed joint joint_block_10_5
- removed joint joint_block_10_8
- removed joint joint_block_10_9
- removed joint joint_block_11_4
- removed joint joint_block_11_5
- removed joint joint_block_11_8
- removed joint joint_block_11_9
- removed joint joint_block_12_4
- removed joint joint_block_12_5
- removed joint joint_block_12_8
- removed joint joint_block_12_9
- removed joint joint_block_13_4
- removed joint joint_block_13_5
- removed joint joint_block_13_8
- removed joint joint_block_13_9
- removed joint joint_block_14_4
- removed joint joint_block_14_5
- removed joint joint_block_14_8
- removed joint joint_block_14_9
- removed joint joint_block_15_4
- removed joint joint_block_15_5
- removed joint joint_block_15_8
- removed joint joint_block_15_9
- removed joint joint_block_16_4
- removed joint joint_block_16_5
- removed joint joint_block_16_8
- removed joint joint_block_16_9
- removed joint joint_block_17_4
- removed joint joint_block_17_5
- removed joint joint_block_17_8
- removed joint joint_block_17_9
- removed joint joint_block_1_4
- removed joint joint_block_1_5
- removed joint joint_block_1_8
- removed joint joint_block_1_9
- removed joint joint_block_2_4
- removed joint joint_block_2_5
- removed joint joint_block_2_8
- removed joint joint_block_2_9
- removed joint joint_block_3_4
- removed joint joint_block_3_5
- removed joint joint_block_3_8
- removed joint joint_block_3_9
- removed joint joint_block_4_4
- removed joint joint_block_4_5
- removed joint joint_block_4_8
- removed joint joint_block_4_9
- removed joint joint_block_5_4
- removed joint joint_block_5_5
- removed joint joint_block_5_8
- removed joint joint_block_5_9
- removed joint joint_block_6_4
- removed joint joint_block_6_5
- removed joint joint_block_6_8
- removed joint joint_block_6_9
- removed joint joint_block_7_4
- removed joint joint_block_7_5
- removed joint joint_block_7_8
- removed joint joint_block_7_9
- added joint joint_block_0_2: type fixed, parent struct_base, child block_0_2, origin xyz=0.5 1.5 0.5 rpy=0 0 0
- added joint joint_block_1_2: type fixed, parent struct_base, child block_1_2, origin xyz=0.5 0.5 0.5 rpy=0 0 0
- added joint joint_block_2_1: type fixed, parent struct_base, child block_2_1, origin xyz=-0.5 -0.5 0.5 rpy=0 0 0
- added joint joint_block_2_2: type fixed, parent struct_base, child block_2_2, origin xyz=0.5 -0.5 0.5 rpy=0 0 0
- added joint joint_block_2_3: type fixed, parent struct_base, child block_2_3, origin xyz=1.5 -0.5 0.5 rpy=0 0 0

File: assets/warehouse/workstations.urdf (robot description, URDF)
Before this commit: robot struct, 13 links, 12 joints
Links:
- removed link block_10_0
- removed link block_10_13
- removed link block_13_0
- removed link block_13_13
- removed link block_16_0
- removed link block_16_13
- removed link block_1_0
- removed link block_1_13
- removed link block_4_0
- removed link block_4_13
- removed link block_7_0
- removed link block_7_13
- added link block_0_0, mass 0; visual box size=1.0 1.0 1.5
- added link block_0_1, mass 0; visual box size=1.0 1.0 1.5
Joints:
- removed joint joint_block_10_0
- removed joint joint_block_10_13
- removed joint joint_block_13_0
- removed joint joint_block_13_13
- removed joint joint_block_16_0
- removed joint joint_block_16_13
- removed joint joint_block_1_0
- removed joint joint_block_1_13
- removed joint joint_block_4_0
- removed joint joint_block_4_13
- removed joint joint_block_7_0
- removed joint joint_block_7_13
- added joint joint_block_0_0: type fixed, parent struct_base, child block_0_0, origin xyz=-1.5 1.5 0.75 rpy=0 0 0
- added joint joint_block_0_1: type fixed, parent struct_base, child block_0_1, origin xyz=-0.5 1.5 0.75 rpy=0 0 0
