Commit message: refactor code

File: assets/warehouse/endpoints.urdf (robot description, URDF)
Before this commit: robot struct, 23 links, 22 joints
Links:
- link block_10_0: geometry visual box size=1.0 1.0 1.25
- link block_10_35: geometry visual box size=1.0 1.0 1.25
- link block_13_0: geometry visual box size=1.0 1.0 1.25
- link block_13_35: geometry visual box size=1.0 1.0 1.25
- link block_16_0: geometry visual box size=1.0 1.0 1.25
- link block_16_35: geometry visual box size=1.0 1.0 1.25
- link block_19_0: geometry visual box size=1.0 1.0 1.25
- link block_19_35: geometry visual box size=1.0 1.0 1.25
- link block_1_0: geometry visual box size=1.0 1.0 1.25
- link block_1_35: geometry visual box size=1.0 1.0 1.25
- link block_22_0: geometry visual box size=1.0 1.0 1.25
- link block_22_35: geometry visual box size=1.0 1.0 1.25
- link block_25_0: geometry visual box size=1.0 1.0 1.25
- link block_25_35: geometry visual box size=1.0 1.0 1.25
- link block_28_0: geometry visual box size=1.0 1.0 1.25
- link block_28_35: geometry visual box size=1.0 1.0 1.25
- link block_31_0: geometry visual box size=1.0 1.0 1.25
- link block_31_35: geometry visual box size=1.0 1.0 1.25
- link block_4_0: geometry visual box size=1.0 1.0 1.25
- link block_4_35: geometry visual box size=1.0 1.0 1.25
- link block_7_0: geometry visual box size=1.0 1.0 1.25
- link block_7_35: geometry visual box size=1.0 1.0 1.25

Commit message: fix floor offset bug

File: assets/warehouse/endpoints.urdf (robot description, URDF)
Before this commit: robot struct, 391 links, 390 joints
Links:
- added link block_28_10, mass 0; visual box size=1.0 1.0 0.1
- added link block_28_11, mass 0; visual box size=1.0 1.0 0.1
- added link block_28_13, mass 0; visual box size=1.0 1.0 0.1
- added link block_28_14, mass 0; visual box size=1.0 1.0 0.1
- added link block_28_15, mass 0; visual box size=1.0 1.0 0.1
- added link block_28_16, mass 0; visual box size=1.0 1.0 0.1
- added link block_28_17, mass 0; visual box size=1.0 1.0 0.1
- added link block_28_18, mass 0; visual box size=1.0 1.0 0.1
- added link block_28_19, mass 0; visual box size=1.0 1.0 0.1
- added link block_28_2, mass 0; visual box size=1.0 1.0 0.1
- added link block_28_20, mass 0; visual box size=1.0 1.0 0.1
- added link block_28_21, mass 0; visual box size=1.0 1.0 0.1
- added link block_28_22, mass 0; visual box size=1.0 1.0 0.1
- added link block_28_24, mass 0; visual box size=1.0 1.0 0.1
- added link block_28_25, mass 0; visual box size=1.0 1.0 0.1
- added link block_28_26, mass 0; visual box size=1.0 1.0 0.1
- added link block_28_27, mass 0; visual box size=1.0 1.0 0.1
- added link block_28_28, mass 0; visual box size=1.0 1.0 0.1
- added link block_28_29, mass 0; visual box size=1.0 1.0 0.1
- added link block_28_3, mass 0; visual box size=1.0 1.0 0.1
- added link block_28_30, mass 0; visual box size=1.0 1.0 0.1
- added link block_28_31, mass 0; visual box size=1.0 1.0 0.1
- added link block_28_32, mass 0; visual box size=1.0 1.0 0.1
- added link block_28_33, mass 0; visual box size=1.0 1.0 0.1
- added link block_28_4, mass 0; visual box size=1.0 1.0 0.1
- added link block_28_5, mass 0; visual box size=1.0 1.0 0.1
- added link block_28_6, mass 0; visual box size=1.0 1.0 0.1
- added link block_28_7, mass 0; visual box size=1.0 1.0 0.1
- added link block_28_8, mass 0; visual box size=1.0 1.0 0.1
- added link block_28_9, mass 0; visual box size=1.0 1.0 0.1
Joints:
- added joint joint_block_28_10: type fixed, parent struct_base, child block_28_10, origin xyz=-7.5 -13.5 0.05 rpy=0 0 0
- added joint joint_block_28_11: type fixed, parent struct_base, child block_28_11, origin xyz=-6.5 -13.5 0.05 rpy=0 0 0
- added joint joint_block_28_13: type fixed, parent struct_base, child block_28_13, origin xyz=-4.5 -13.5 0.05 rpy=0 0 0
- added joint joint_block_28_14: type fixed, parent struct_base, child block_28_14, origin xyz=-3.5 -13.5 0.05 rpy=0 0 0
- added joint joint_block_28_15: type fixed, parent struct_base, child block_28_15, origin xyz=-2.5 -13.5 0.05 rpy=0 0 0
- added joint joint_block_28_16: type fixed, parent struct_base, child block_28_16, origin xyz=-1.5 -13.5 0.05 rpy=0 0 0
- added joint joint_block_28_17: type fixed, parent struct_base, child block_28_17, origin xyz=-0.5 -13.5 0.05 rpy=0 0 0
- added joint joint_block_28_18: type fixed, parent struct_base, child block_28_18, origin xyz=0.5 -13.5 0.05 rpy=0 0 0
- added joint joint_block_28_19: type fixed, parent struct_base, child block_28_19, origin xyz=1.5 -13.5 0.05 rpy=0 0 0
- added joint joint_block_28_2: type fixed, parent struct_base, child block_28_2, origin xyz=-15.5 -13.5 0.05 rpy=0 0 0
- added joint joint_block_28_20: type fixed, parent struct_base, child block_28_20, origin xyz=2.5 -13.5 0.05 rpy=0 0 0
- added joint joint_block_28_21: type fixed, parent struct_base, child block_28_21, origin xyz=3.5 -13.5 0.05 rpy=0 0 0
- added joint joint_block_28_22: type fixed, parent struct_base, child block_28_22, origin xyz=4.5 -13.5 0.05 rpy=0 0 0
- added joint joint_block_28_24: type fixed, parent struct_base, child block_28_24, origin xyz=6.5 -13.5 0.05 rpy=0 0 0
- added joint joint_block_28_25: type fixed, parent struct_base, child block_28_25, origin xyz=7.5 -13.5 0.05 rpy=0 0 0
- added joint joint_block_28_26: type fixed, parent struct_base, child block_28_26, origin xyz=8.5 -13.5 0.05 rpy=0 0 0
- added joint joint_block_28_27: type fixed, parent struct_base, child block_28_27, origin xyz=9.5 -13.5 0.05 rpy=0 0 0
- added joint joint_block_28_28: type fixed, parent struct_base, child block_28_28, origin xyz=10.5 -13.5 0.05 rpy=0 0 0
- added joint joint_block_28_29: type fixed, parent struct_base, child block_28_29, origin xyz=11.5 -13.5 0.05 rpy=0 0 0
- added joint joint_block_28_3: type fixed, parent struct_base, child block_28_3, origin xyz=-14.5 -13.5 0.05 rpy=0 0 0
- added joint joint_block_28_30: type fixed, parent struct_base, child block_28_30, origin xyz=12.5 -13.5 0.05 rpy=0 0 0
- added joint joint_block_28_31: type fixed, parent struct_base, child block_28_31, origin xyz=13.5 -13.5 0.05 rpy=0 0 0
- added joint joint_block_28_32: type fixed, parent struct_base, child block_28_32, origin xyz=14.5 -13.5 0.05 rpy=0 0 0
- added joint joint_block_28_33: type fixed, parent struct_base, child block_28_33, origin xyz=15.5 -13.5 0.05 rpy=0 0 0
- added joint joint_block_28_4: type fixed, parent struct_base, child block_28_4, origin xyz=-13.5 -13.5 0.05 rpy=0 0 0
- added joint joint_block_28_5: type fixed, parent struct_base, child block_28_5, origin xyz=-12.5 -13.5 0.05 rpy=0 0 0
- added joint joint_block_28_6: type fixed, parent struct_base, child block_28_6, origin xyz=-11.5 -13.5 0.05 rpy=0 0 0
- added joint joint_block_28_7: type fixed, parent struct_base, child block_28_7, origin xyz=-10.5 -13.5 0.05 rpy=0 0 0
- added joint joint_block_28_8: type fixed, parent struct_base, child block_28_8, origin xyz=-9.5 -13.5 0.05 rpy=0 0 0
- added joint joint_block_28_9: type fixed, parent struct_base, child block_28_9, origin xyz=-8.5 -13.5 0.05 rpy=0 0 0
