Commit message: A* implementation

File: assets/warehouse/workstations.urdf (robot description, URDF)
Before this commit: robot struct, 21 links, 20 joints
Links:
- link block_10_0: geometry visual box size=1.0 1.0 1.5
- link block_10_35: geometry visual box size=1.0 1.0 1.5
- link block_13_0: geometry visual box size=1.0 1.0 1.5
- link block_13_35: geometry visual box size=1.0 1.0 1.5
- link block_16_0: geometry visual box size=1.0 1.0 1.5
- link block_16_35: geometry visual box size=1.0 1.0 1.5
- link block_19_0: geometry visual box size=1.0 1.0 1.5
- link block_19_35: geometry visual box size=1.0 1.0 1.5
- link block_1_0: geometry visual box size=1.0 1.0 1.5
- link block_1_35: geometry visual box size=1.0 1.0 1.5
- link block_22_0: geometry visual box size=1.0 1.0 1.5
- link block_22_35: geometry visual box size=1.0 1.0 1.5
- link block_25_0: geometry visual box size=1.0 1.0 1.5
- link block_25_35: geometry visual box size=1.0 1.0 1.5
- link block_28_0: geometry visual box size=1.0 1.0 1.5
- link block_28_35: geometry visual box size=1.0 1.0 1.5
- link block_4_0: geometry visual box size=1.0 1.0 1.5
- link block_4_35: geometry visual box size=1.0 1.0 1.5
- link block_7_0: geometry visual box size=1.0 1.0 1.5
- link block_7_35: geometry visual box size=1.0 1.0 1.5
Joints:
- joint joint_block_10_0: origin xyz=-17.5 4.5 0.625 rpy=0 0 0 -> xyz=-17.5 4.5 0.75 rpy=0 0 0
- joint joint_block_10_35: origin xyz=17.5 4.5 0.625 rpy=0 0 0 -> xyz=17.5 4.5 0.75 rpy=0 0 0
- joint joint_block_13_0: origin xyz=-17.5 1.5 0.625 rpy=0 0 0 -> xyz=-17.5 1.5 0.75 rpy=0 0 0
- joint joint_block_13_35: origin xyz=17.5 1.5 0.625 rpy=0 0 0 -> xyz=17.5 1.5 0.75 rpy=0 0 0
- joint joint_block_16_0: origin xyz=-17.5 -1.5 0.625 rpy=0 0 0 -> xyz=-17.5 -1.5 0.75 rpy=0 0 0
- joint joint_block_16_35: origin xyz=17.5 -1.5 0.625 rpy=0 0 0 -> xyz=17.5 -1.5 0.75 rpy=0 0 0
- joint joint_block_19_0: origin xyz=-17.5 -4.5 0.625 rpy=0 0 0 -> xyz=-17.5 -4.5 0.75 rpy=0 0 0
- joint joint_block_19_35: origin xyz=17.5 -4.5 0.625 rpy=0 0 0 -> xyz=17.5 -4.5 0.75 rpy=0 0 0
- joint joint_block_1_0: origin xyz=-17.5 13.5 0.625 rpy=0 0 0 -> xyz=-17.5 13.5 0.75 rpy=0 0 0
- joint joint_block_1_35: origin xyz=17.5 13.5 0.625 rpy=0 0 0 -> xyz=17.5 13.5 0.75 rpy=0 0 0
- joint joint_block_22_0: origin xyz=-17.5 -7.5 0.625 rpy=0 0 0 -> xyz=-17.5 -7.5 0.75 rpy=0 0 0
- joint joint_block_22_35: origin xyz=17.5 -7.5 0.625 rpy=0 0 0 -> xyz=17.5 -7.5 0.75 rpy=0 0 0
- joint joint_block_25_0: origin xyz=-17.5 -10.5 0.625 rpy=0 0 0 -> xyz=-17.5 -10.5 0.75 rpy=0 0 0
- joint joint_block_25_35: origin xyz=17.5 -10.5 0.625 rpy=0 0 0 -> xyz=17.5 -10.5 0.75 rpy=0 0 0
- joint joint_block_28_0: origin xyz=-17.5 -13.5 0.625 rpy=0 0 0 -> xyz=-17.5 -13.5 0.75 rpy=0 0 0
- joint joint_block_28_35: origin xyz=17.5 -13.5 0.625 rpy=0 0 0 -> xyz=17.5 -13.5 0.75 rpy=0 0 0
- joint joint_block_4_0: origin xyz=-17.5 10.5 0.625 rpy=0 0 0 -> xyz=-17.5 10.5 0.75 rpy=0 0 0
- joint joint_block_4_35: origin xyz=17.5 10.5 0.625 rpy=0 0 0 -> xyz=17.5 10.5 0.75 rpy=0 0 0
- joint joint_block_7_0: origin xyz=-17.5 7.5 0.625 rpy=0 0 0 -> xyz=-17.5 7.5 0.75 rpy=0 0 0
- joint joint_block_7_35: origin xyz=17.5 7.5 0.625 rpy=0 0 0 -> xyz=17.5 7.5 0.75 rpy=0 0 0
