Commit message: add deleting endpoint visual once delivery terminates and new delivery is assigned to a robot

File: assets/warehouse/endpoints.urdf (robot description, URDF)
Before this commit: robot struct, 65 links, 64 joints
Joints:
- joint joint_block_0_2: origin xyz=-3.5 8.5 0.15 rpy=0 0 0 -> xyz=-4.5 8.5 0.15 rpy=0 0 0
- joint joint_block_0_5: origin xyz=-0.5 8.5 0.15 rpy=0 0 0 -> xyz=-1.5 8.5 0.15 rpy=0 0 0
- joint joint_block_0_6: origin xyz=0.5 8.5 0.15 rpy=0 0 0 -> xyz=-0.5 8.5 0.15 rpy=0 0 0
- joint joint_block_0_9: origin xyz=3.5 8.5 0.15 rpy=0 0 0 -> xyz=2.5 8.5 0.15 rpy=0 0 0
- joint joint_block_10_2: origin xyz=-3.5 -1.5 0.15 rpy=0 0 0 -> xyz=-4.5 -1.5 0.15 rpy=0 0 0
- joint joint_block_10_5: origin xyz=-0.5 -1.5 0.15 rpy=0 0 0 -> xyz=-1.5 -1.5 0.15 rpy=0 0 0
- joint joint_block_10_6: origin xyz=0.5 -1.5 0.15 rpy=0 0 0 -> xyz=-0.5 -1.5 0.15 rpy=0 0 0
- joint joint_block_10_9: origin xyz=3.5 -1.5 0.15 rpy=0 0 0 -> xyz=2.5 -1.5 0.15 rpy=0 0 0
- joint joint_block_11_2: origin xyz=-3.5 -2.5 0.15 rpy=0 0 0 -> xyz=-4.5 -2.5 0.15 rpy=0 0 0
- joint joint_block_11_5: origin xyz=-0.5 -2.5 0.15 rpy=0 0 0 -> xyz=-1.5 -2.5 0.15 rpy=0 0 0
- joint joint_block_11_6: origin xyz=0.5 -2.5 0.15 rpy=0 0 0 -> xyz=-0.5 -2.5 0.15 rpy=0 0 0
- joint joint_block_11_9: origin xyz=3.5 -2.5 0.15 rpy=0 0 0 -> xyz=2.5 -2.5 0.15 rpy=0 0 0
- joint joint_block_12_2: origin xyz=-3.5 -3.5 0.15 rpy=0 0 0 -> xyz=-4.5 -3.5 0.15 rpy=0 0 0
- joint joint_block_12_5: origin xyz=-0.5 -3.5 0.15 rpy=0 0 0 -> xyz=-1.5 -3.5 0.15 rpy=0 0 0
- joint joint_block_12_6: origin xyz=0.5 -3.5 0.15 rpy=0 0 0 -> xyz=-0.5 -3.5 0.15 rpy=0 0 0
- joint joint_block_12_9: origin xyz=3.5 -3.5 0.15 rpy=0 0 0 -> xyz=2.5 -3.5 0.15 rpy=0 0 0
- joint joint_block_13_2: origin xyz=-3.5 -4.5 0.15 rpy=0 0 0 -> xyz=-4.5 -4.5 0.15 rpy=0 0 0
- joint joint_block_13_5: origin xyz=-0.5 -4.5 0.15 rpy=0 0 0 -> xyz=-1.5 -4.5 0.15 rpy=0 0 0
- joint joint_block_13_6: origin xyz=0.5 -4.5 0.15 rpy=0 0 0 -> xyz=-0.5 -4.5 0.15 rpy=0 0 0
- joint joint_block_13_9: origin xyz=3.5 -4.5 0.15 rpy=0 0 0 -> xyz=2.5 -4.5 0.15 rpy=0 0 0
- joint joint_block_14_2: origin xyz=-3.5 -5.5 0.15 rpy=0 0 0 -> xyz=-4.5 -5.5 0.15 rpy=0 0 0
- joint joint_block_14_5: origin xyz=-0.5 -5.5 0.15 rpy=0 0 0 -> xyz=-1.5 -5.5 0.15 rpy=0 0 0
- joint joint_block_14_6: origin xyz=0.5 -5.5 0.15 rpy=0 0 0 -> xyz=-0.5 -5.5 0.15 rpy=0 0 0
- joint joint_block_14_9: origin xyz=3.5 -5.5 0.15 rpy=0 0 0 -> xyz=2.5 -5.5 0.15 rpy=0 0 0
- joint joint_block_15_2: origin xyz=-3.5 -6.5 0.15 rpy=0 0 0 -> xyz=-4.5 -6.5 0.15 rpy=0 0 0
- joint joint_block_15_5: origin xyz=-0.5 -6.5 0.15 rpy=0 0 0 -> xyz=-1.5 -6.5 0.15 rpy=0 0 0
- joint joint_block_15_6: origin xyz=0.5 -6.5 0.15 rpy=0 0 0 -> xyz=-0.5 -6.5 0.15 rpy=0 0 0
- joint joint_block_15_9: origin xyz=3.5 -6.5 0.15 rpy=0 0 0 -> xyz=2.5 -6.5 0.15 rpy=0 0 0
- joint joint_block_16_2: origin xyz=-3.5 -7.5 0.15 rpy=0 0 0 -> xyz=-4.5 -7.5 0.15 rpy=0 0 0
- joint joint_block_16_5: origin xyz=-0.5 -7.5 0.15 rpy=0 0 0 -> xyz=-1.5 -7.5 0.15 rpy=0 0 0
- joint joint_block_16_6: origin xyz=0.5 -7.5 0.15 rpy=0 0 0 -> xyz=-0.5 -7.5 0.15 rpy=0 0 0
- joint joint_block_16_9: origin xyz=3.5 -7.5 0.15 rpy=0 0 0 -> xyz=2.5 -7.5 0.15 rpy=0 0 0
- joint joint_block_17_2: origin xyz=-3.5 -8.5 0.15 rpy=0 0 0 -> xyz=-4.5 -8.5 0.15 rpy=0 0 0
- joint joint_block_17_5: origin xyz=-0.5 -8.5 0.15 rpy=0 0 0 -> xyz=-1.5 -8.5 0.15 rpy=0 0 0
- joint joint_block_17_6: origin xyz=0.5 -8.5 0.15 rpy=0 0 0 -> xyz=-0.5 -8.5 0.15 rpy=0 0 0
- joint joint_block_17_9: origin xyz=3.5 -8.5 0.15 rpy=0 0 0 -> xyz=2.5 -8.5 0.15 rpy=0 0 0
- joint joint_block_1_2: origin xyz=-3.5 7.5 0.15 rpy=0 0 0 -> xyz=-4.5 7.5 0.15 rpy=0 0 0
- joint joint_block_1_5: origin xyz=-0.5 7.5 0.15 rpy=0 0 0 -> xyz=-1.5 7.5 0.15 rpy=0 0 0
- joint joint_block_1_6: origin xyz=0.5 7.5 0.15 rpy=0 0 0 -> xyz=-0.5 7.5 0.15 rpy=0 0 0
- joint joint_block_1_9: origin xyz=3.5 7.5 0.15 rpy=0 0 0 -> xyz=2.5 7.5 0.15 rpy=0 0 0
- joint joint_block_2_2: origin xyz=-3.5 6.5 0.15 rpy=0 0 0 -> xyz=-4.5 6.5 0.15 rpy=0 0 0
- joint joint_block_2_5: origin xyz=-0.5 6.5 0.15 rpy=0 0 0 -> xyz=-1.5 6.5 0.15 rpy=0 0 0
- joint joint_block_2_6: origin xyz=0.5 6.5 0.15 rpy=0 0 0 -> xyz=-0.5 6.5 0.15 rpy=0 0 0
- joint joint_block_2_9: origin xyz=3.5 6.5 0.15 rpy=0 0 0 -> xyz=2.5 6.5 0.15 rpy=0 0 0
- joint joint_block_3_2: origin xyz=-3.5 5.5 0.15 rpy=0 0 0 -> xyz=-4.5 5.5 0.15 rpy=0 0 0
- joint joint_block_3_5: origin xyz=-0.5 5.5 0.15 rpy=0 0 0 -> xyz=-1.5 5.5 0.15 rpy=0 0 0
- joint joint_block_3_6: origin xyz=0.5 5.5 0.15 rpy=0 0 0 -> xyz=-0.5 5.5 0.15 rpy=0 0 0
- joint joint_block_3_9: origin xyz=3.5 5.5 0.15 rpy=0 0 0 -> xyz=2.5 5.5 0.15 rpy=0 0 0
- joint joint_block_4_2: origin xyz=-3.5 4.5 0.15 rpy=0 0 0 -> xyz=-4.5 4.5 0.15 rpy=0 0 0
- joint joint_block_4_5: origin xyz=-0.5 4.5 0.15 rpy=0 0 0 -> xyz=-1.5 4.5 0.15 rpy=0 0 0
- joint joint_block_4_6: origin xyz=0.5 4.5 0.15 rpy=0 0 0 -> xyz=-0.5 4.5 0.15 rpy=0 0 0
- joint joint_block_4_9: origin xyz=3.5 4.5 0.15 rpy=0 0 0 -> xyz=2.5 4.5 0.15 rpy=0 0 0
- joint joint_block_5_2: origin xyz=-3.5 3.5 0.15 rpy=0 0 0 -> xyz=-4.5 3.5 0.15 rpy=0 0 0
- joint joint_block_5_5: origin xyz=-0.5 3.5 0.15 rpy=0 0 0 -> xyz=-1.5 3.5 0.15 rpy=0 0 0
- joint joint_block_5_6: origin xyz=0.5 3.5 0.15 rpy=0 0 0 -> xyz=-0.5 3.5 0.15 rpy=0 0 0
- joint joint_block_5_9: origin xyz=3.5 3.5 0.15 rpy=0 0 0 -> xyz=2.5 3.5 0.15 rpy=0 0 0
- joint joint_block_6_2: origin xyz=-3.5 2.5 0.15 rpy=0 0 0 -> xyz=-4.5 2.5 0.15 rpy=0 0 0
- joint joint_block_6_5: origin xyz=-0.5 2.5 0.15 rpy=0 0 0 -> xyz=-1.5 2.5 0.15 rpy=0 0 0
- joint joint_block_6_6: origin xyz=0.5 2.5 0.15 rpy=0 0 0 -> xyz=-0.5 2.5 0.15 rpy=0 0 0
- joint joint_block_6_9: origin xyz=3.5 2.5 0.15 rpy=0 0 0 -> xyz=2.5 2.5 0.15 rpy=0 0 0
- joint joint_block_7_2: origin xyz=-3.5 1.5 0.15 rpy=0 0 0 -> xyz=-4.5 1.5 0.15 rpy=0 0 0
- joint joint_block_7_5: origin xyz=-0.5 1.5 0.15 rpy=0 0 0 -> xyz=-1.5 1.5 0.15 rpy=0 0 0
- joint joint_block_7_6: origin xyz=0.5 1.5 0.15 rpy=0 0 0 -> xyz=-0.5 1.5 0.15 rpy=0 0 0
- joint joint_block_7_9: origin xyz=3.5 1.5 0.15 rpy=0 0 0 -> xyz=2.5 1.5 0.15 rpy=0 0 0

File: assets/warehouse/shelves.urdf (robot description, URDF)
Before this commit: robot struct, 65 links, 64 joints
Joints:
- joint joint_block_0_3: origin xyz=-2.5 8.5 0.5 rpy=0 0 0 -> xyz=-3.5 8.5 0.5 rpy=0 0 0
- joint joint_block_0_4: origin xyz=-1.5 8.5 0.5 rpy=0 0 0 -> xyz=-2.5 8.5 0.5 rpy=0 0 0
- joint joint_block_0_7: origin xyz=1.5 8.5 0.5 rpy=0 0 0 -> xyz=0.5 8.5 0.5 rpy=0 0 0
- joint joint_block_0_8: origin xyz=2.5 8.5 0.5 rpy=0 0 0 -> xyz=1.5 8.5 0.5 rpy=0 0 0
- joint joint_block_10_3: origin xyz=-2.5 -1.5 0.5 rpy=0 0 0 -> xyz=-3.5 -1.5 0.5 rpy=0 0 0
- joint joint_block_10_4: origin xyz=-1.5 -1.5 0.5 rpy=0 0 0 -> xyz=-2.5 -1.5 0.5 rpy=0 0 0
- joint joint_block_10_7: origin xyz=1.5 -1.5 0.5 rpy=0 0 0 -> xyz=0.5 -1.5 0.5 rpy=0 0 0
- joint joint_block_10_8: origin xyz=2.5 -1.5 0.5 rpy=0 0 0 -> xyz=1.5 -1.5 0.5 rpy=0 0 0
- joint joint_block_11_3: origin xyz=-2.5 -2.5 0.5 rpy=0 0 0 -> xyz=-3.5 -2.5 0.5 rpy=0 0 0
- joint joint_block_11_4: origin xyz=-1.5 -2.5 0.5 rpy=0 0 0 -> xyz=-2.5 -2.5 0.5 rpy=0 0 0
- joint joint_block_11_7: origin xyz=1.5 -2.5 0.5 rpy=0 0 0 -> xyz=0.5 -2.5 0.5 rpy=0 0 0
- joint joint_block_11_8: origin xyz=2.5 -2.5 0.5 rpy=0 0 0 -> xyz=1.5 -2.5 0.5 rpy=0 0 0
- joint joint_block_12_3: origin xyz=-2.5 -3.5 0.5 rpy=0 0 0 -> xyz=-3.5 -3.5 0.5 rpy=0 0 0
- joint joint_block_12_4: origin xyz=-1.5 -3.5 0.5 rpy=0 0 0 -> xyz=-2.5 -3.5 0.5 rpy=0 0 0
- joint joint_block_12_7: origin xyz=1.5 -3.5 0.5 rpy=0 0 0 -> xyz=0.5 -3.5 0.5 rpy=0 0 0
- joint joint_block_12_8: origin xyz=2.5 -3.5 0.5 rpy=0 0 0 -> xyz=1.5 -3.5 0.5 rpy=0 0 0
- joint joint_block_13_3: origin xyz=-2.5 -4.5 0.5 rpy=0 0 0 -> xyz=-3.5 -4.5 0.5 rpy=0 0 0
- joint joint_block_13_4: origin xyz=-1.5 -4.5 0.5 rpy=0 0 0 -> xyz=-2.5 -4.5 0.5 rpy=0 0 0
- joint joint_block_13_7: origin xyz=1.5 -4.5 0.5 rpy=0 0 0 -> xyz=0.5 -4.5 0.5 rpy=0 0 0
- joint joint_block_13_8: origin xyz=2.5 -4.5 0.5 rpy=0 0 0 -> xyz=1.5 -4.5 0.5 rpy=0 0 0
- joint joint_block_14_3: origin xyz=-2.5 -5.5 0.5 rpy=0 0 0 -> xyz=-3.5 -5.5 0.5 rpy=0 0 0
- joint joint_block_14_4: origin xyz=-1.5 -5.5 0.5 rpy=0 0 0 -> xyz=-2.5 -5.5 0.5 rpy=0 0 0
- joint joint_block_14_7: origin xyz=1.5 -5.5 0.5 rpy=0 0 0 -> xyz=0.5 -5.5 0.5 rpy=0 0 0
- joint joint_block_14_8: origin xyz=2.5 -5.5 0.5 rpy=0 0 0 -> xyz=1.5 -5.5 0.5 rpy=0 0 0
- joint joint_block_15_3: origin xyz=-2.5 -6.5 0.5 rpy=0 0 0 -> xyz=-3.5 -6.5 0.5 rpy=0 0 0
- joint joint_block_15_4: origin xyz=-1.5 -6.5 0.5 rpy=0 0 0 -> xyz=-2.5 -6.5 0.5 rpy=0 0 0
- joint joint_block_15_7: origin xyz=1.5 -6.5 0.5 rpy=0 0 0 -> xyz=0.5 -6.5 0.5 rpy=0 0 0
- joint joint_block_15_8: origin xyz=2.5 -6.5 0.5 rpy=0 0 0 -> xyz=1.5 -6.5 0.5 rpy=0 0 0
- joint joint_block_16_3: origin xyz=-2.5 -7.5 0.5 rpy=0 0 0 -> xyz=-3.5 -7.5 0.5 rpy=0 0 0
- joint joint_block_16_4: origin xyz=-1.5 -7.5 0.5 rpy=0 0 0 -> xyz=-2.5 -7.5 0.5 rpy=0 0 0
- joint joint_block_16_7: origin xyz=1.5 -7.5 0.5 rpy=0 0 0 -> xyz=0.5 -7.5 0.5 rpy=0 0 0
- joint joint_block_16_8: origin xyz=2.5 -7.5 0.5 rpy=0 0 0 -> xyz=1.5 -7.5 0.5 rpy=0 0 0
- joint joint_block_17_3: origin xyz=-2.5 -8.5 0.5 rpy=0 0 0 -> xyz=-3.5 -8.5 0.5 rpy=0 0 0
- joint joint_block_17_4: origin xyz=-1.5 -8.5 0.5 rpy=0 0 0 -> xyz=-2.5 -8.5 0.5 rpy=0 0 0
- joint joint_block_17_7: origin xyz=1.5 -8.5 0.5 rpy=0 0 0 -> xyz=0.5 -8.5 0.5 rpy=0 0 0
- joint joint_block_17_8: origin xyz=2.5 -8.5 0.5 rpy=0 0 0 -> xyz=1.5 -8.5 0.5 rpy=0 0 0
- joint joint_block_1_3: origin xyz=-2.5 7.5 0.5 rpy=0 0 0 -> xyz=-3.5 7.5 0.5 rpy=0 0 0
- joint joint_block_1_4: origin xyz=-1.5 7.5 0.5 rpy=0 0 0 -> xyz=-2.5 7.5 0.5 rpy=0 0 0
- joint joint_block_1_7: origin xyz=1.5 7.5 0.5 rpy=0 0 0 -> xyz=0.5 7.5 0.5 rpy=0 0 0
- joint joint_block_1_8: origin xyz=2.5 7.5 0.5 rpy=0 0 0 -> xyz=1.5 7.5 0.5 rpy=0 0 0
- joint joint_block_2_3: origin xyz=-2.5 6.5 0.5 rpy=0 0 0 -> xyz=-3.5 6.5 0.5 rpy=0 0 0
- joint joint_block_2_4: origin xyz=-1.5 6.5 0.5 rpy=0 0 0 -> xyz=-2.5 6.5 0.5 rpy=0 0 0
- joint joint_block_2_7: origin xyz=1.5 6.5 0.5 rpy=0 0 0 -> xyz=0.5 6.5 0.5 rpy=0 0 0
- joint joint_block_2_8: origin xyz=2.5 6.5 0.5 rpy=0 0 0 -> xyz=1.5 6.5 0.5 rpy=0 0 0
- joint joint_block_3_3: origin xyz=-2.5 5.5 0.5 rpy=0 0 0 -> xyz=-3.5 5.5 0.5 rpy=0 0 0
- joint joint_block_3_4: origin xyz=-1.5 5.5 0.5 rpy=0 0 0 -> xyz=-2.5 5.5 0.5 rpy=0 0 0
- joint joint_block_3_7: origin xyz=1.5 5.5 0.5 rpy=0 0 0 -> xyz=0.5 5.5 0.5 rpy=0 0 0
- joint joint_block_3_8: origin xyz=2.5 5.5 0.5 rpy=0 0 0 -> xyz=1.5 5.5 0.5 rpy=0 0 0
- joint joint_block_4_3: origin xyz=-2.5 4.5 0.5 rpy=0 0 0 -> xyz=-3.5 4.5 0.5 rpy=0 0 0
- joint joint_block_4_4: origin xyz=-1.5 4.5 0.5 rpy=0 0 0 -> xyz=-2.5 4.5 0.5 rpy=0 0 0
- joint joint_block_4_7: origin xyz=1.5 4.5 0.5 rpy=0 0 0 -> xyz=0.5 4.5 0.5 rpy=0 0 0
- joint joint_block_4_8: origin xyz=2.5 4.5 0.5 rpy=0 0 0 -> xyz=1.5 4.5 0.5 rpy=0 0 0
- joint joint_block_5_3: origin xyz=-2.5 3.5 0.5 rpy=0 0 0 -> xyz=-3.5 3.5 0.5 rpy=0 0 0
- joint joint_block_5_4: origin xyz=-1.5 3.5 0.5 rpy=0 0 0 -> xyz=-2.5 3.5 0.5 rpy=0 0 0
- joint joint_block_5_7: origin xyz=1.5 3.5 0.5 rpy=0 0 0 -> xyz=0.5 3.5 0.5 rpy=0 0 0
- joint joint_block_5_8: origin xyz=2.5 3.5 0.5 rpy=0 0 0 -> xyz=1.5 3.5 0.5 rpy=0 0 0
- joint joint_block_6_3: origin xyz=-2.5 2.5 0.5 rpy=0 0 0 -> xyz=-3.5 2.5 0.5 rpy=0 0 0
- joint joint_block_6_4: origin xyz=-1.5 2.5 0.5 rpy=0 0 0 -> xyz=-2.5 2.5 0.5 rpy=0 0 0
- joint joint_block_6_7: origin xyz=1.5 2.5 0.5 rpy=0 0 0 -> xyz=0.5 2.5 0.5 rpy=0 0 0
- joint joint_block_6_8: origin xyz=2.5 2.5 0.5 rpy=0 0 0 -> xyz=1.5 2.5 0.5 rpy=0 0 0
- joint joint_block_7_3: origin xyz=-2.5 1.5 0.5 rpy=0 0 0 -> xyz=-3.5 1.5 0.5 rpy=0 0 0
- joint joint_block_7_4: origin xyz=-1.5 1.5 0.5 rpy=0 0 0 -> xyz=-2.5 1.5 0.5 rpy=0 0 0
- joint joint_block_7_7: origin xyz=1.5 1.5 0.5 rpy=0 0 0 -> xyz=0.5 1.5 0.5 rpy=0 0 0
- joint joint_block_7_8: origin xyz=2.5 1.5 0.5 rpy=0 0 0 -> xyz=1.5 1.5 0.5 rpy=0 0 0

File: assets/warehouse/wall.urdf (robot description, URDF)
Before this commit: robot struct, 65 links, 64 joints
Links:
- removed link block_10_13
- removed link block_11_13
- removed link block_12_13
- removed link block_13_13
- removed link block_14_13
- removed link block_15_13
- removed link block_16_13
- removed link block_17_13
- removed link block_18_13
- removed link block_1_13
- removed link block_2_13
- removed link block_3_13
- removed link block_4_13
- removed link block_5_13
- removed link block_6_13
- removed link block_7_13
- removed link block_8_13
- removed link block_9_13
- added link block_0_14, mass 0; collision box size=1.0 1.0 3.0; visual box size=1.0 1.0 3
- added link block_0_15, mass 0; collision box size=1.0 1.0 3.0; visual box size=1.0 1.0 3
- added link block_10_15, mass 0; collision box size=1.0 1.0 3.0; visual box size=1.0 1.0 3
- added link block_11_15, mass 0; collision box size=1.0 1.0 3.0; visual box size=1.0 1.0 3
- added link block_12_15, mass 0; collision box size=1.0 1.0 3.0; visual box size=1.0 1.0 3
- added link block_13_15, mass 0; collision box size=1.0 1.0 3.0; visual box size=1.0 1.0 3
- added link block_14_15, mass 0; collision box size=1.0 1.0 3.0; visual box size=1.0 1.0 3
- added link block_15_15, mass 0; collision box size=1.0 1.0 3.0; visual box size=1.0 1.0 3
- added link block_16_15, mass 0; collision box size=1.0 1.0 3.0; visual box size=1.0 1.0 3
- added link block_17_15, mass 0; collision box size=1.0 1.0 3.0; visual box size=1.0 1.0 3
- added link block_18_15, mass 0; collision box size=1.0 1.0 3.0; visual box size=1.0 1.0 3
- added link block_19_14, mass 0; collision box size=1.0 1.0 3.0; visual box size=1.0 1.0 3
- added link block_19_15, mass 0; collision box size=1.0 1.0 3.0; visual box size=1.0 1.0 3
- added link block_1_15, mass 0; collision box size=1.0 1.0 3.0; visual box size=1.0 1.0 3
- added link block_2_15, mass 0; collision box size=1.0 1.0 3.0; visual box size=1.0 1.0 3
- added link block_3_15, mass 0; collision box size=1.0 1.0 3.0; visual box size=1.0 1.0 3
- added link block_4_15, mass 0; collision box size=1.0 1.0 3.0; visual box size=1.0 1.0 3
- added link block_5_15, mass 0; collision box size=1.0 1.0 3.0; visual box size=1.0 1.0 3
- added link block_6_15, mass 0; collision box size=1.0 1.0 3.0; visual box size=1.0 1.0 3
- added link block_7_15, mass 0; collision box size=1.0 1.0 3.0; visual box size=1.0 1.0 3
- added link block_8_15, mass 0; collision box size=1.0 1.0 3.0; visual box size=1.0 1.0 3
- added link block_9_15, mass 0; collision box size=1.0 1.0 3.0; visual box size=1.0 1.0 3
Joints:
- removed joint joint_block_10_13
- removed joint joint_block_11_13
- removed joint joint_block_12_13
- removed joint joint_block_13_13
- removed joint joint_block_14_13
- removed joint joint_block_15_13
- removed joint joint_block_16_13
- removed joint joint_block_17_13
- removed joint joint_block_18_13
- removed joint joint_block_1_13
- removed joint joint_block_2_13
- removed joint joint_block_3_13
- removed joint joint_block_4_13
- removed joint joint_block_5_13
- removed joint joint_block_6_13
- removed joint joint_block_7_13
- removed joint joint_block_8_13
- removed joint joint_block_9_13
- added joint joint_block_0_14: type fixed, parent struct_base, child block_0_14, origin xyz=6.5 9.5 1.5 rpy=0 0 0
- added joint joint_block_0_15: type fixed, parent struct_base, child block_0_15, origin xyz=7.5 9.5 1.5 rpy=0 0 0
- added joint joint_block_10_15: type fixed, parent struct_base, child block_10_15, origin xyz=7.5 -0.5 1.5 rpy=0 0 0
- added joint joint_block_11_15: type fixed, parent struct_base, child block_11_15, origin xyz=7.5 -1.5 1.5 rpy=0 0 0
- added joint joint_block_12_15: type fixed, parent struct_base, child block_12_15, origin xyz=7.5 -2.5 1.5 rpy=0 0 0
- added joint joint_block_13_15: type fixed, parent struct_base, child block_13_15, origin xyz=7.5 -3.5 1.5 rpy=0 0 0
- added joint joint_block_14_15: type fixed, parent struct_base, child block_14_15, origin xyz=7.5 -4.5 1.5 rpy=0 0 0
- added joint joint_block_15_15: type fixed, parent struct_base, child block_15_15, origin xyz=7.5 -5.5 1.5 rpy=0 0 0
- added joint joint_block_16_15: type fixed, parent struct_base, child block_16_15, origin xyz=7.5 -6.5 1.5 rpy=0 0 0
- added joint joint_block_17_15: type fixed, parent struct_base, child block_17_15, origin xyz=7.5 -7.5 1.5 rpy=0 0 0
- added joint joint_block_18_15: type fixed, parent struct_base, child block_18_15, origin xyz=7.5 -8.5 1.5 rpy=0 0 0
- added joint joint_block_19_14: type fixed, parent struct_base, child block_19_14, origin xyz=6.5 -9.5 1.5 rpy=0 0 0
- added joint joint_block_19_15: type fixed, parent struct_base, child block_19_15, origin xyz=7.5 -9.5 1.5 rpy=0 0 0
- added joint joint_block_1_15: type fixed, parent struct_base, child block_1_15, origin xyz=7.5 8.5 1.5 rpy=0 0 0
- added joint joint_block_2_15: type fixed, parent struct_base, child block_2_15, origin xyz=7.5 7.5 1.5 rpy=0 0 0
- added joint joint_block_3_15: type fixed, parent struct_base, child block_3_15, origin xyz=7.5 6.5 1.5 rpy=0 0 0
- added joint joint_block_4_15: type fixed, parent struct_base, child block_4_15, origin xyz=7.5 5.5 1.5 rpy=0 0 0
- added joint joint_block_5_15: type fixed, parent struct_base, child block_5_15, origin xyz=7.5 4.5 1.5 rpy=0 0 0
- added joint joint_block_6_15: type fixed, parent struct_base, child block_6_15, origin xyz=7.5 3.5 1.5 rpy=0 0 0
- added joint joint_block_7_15: type fixed, parent struct_base, child block_7_15, origin xyz=7.5 2.5 1.5 rpy=0 0 0
- added joint joint_block_8_15: type fixed, parent struct_base, child block_8_15, origin xyz=7.5 1.5 1.5 rpy=0 0 0
- added joint joint_block_9_15: type fixed, parent struct_base, child block_9_15, origin xyz=7.5 0.5 1.5 rpy=0 0 0
- joint joint_block_0_0: origin xyz=-6.5 9.5 1.5 rpy=0 0 0 -> xyz=-7.5 9.5 1.5 rpy=0 0 0
- joint joint_block_0_1: origin xyz=-5.5 9.5 1.5 rpy=0 0 0 -> xyz=-6.5 9.5 1.5 rpy=0 0 0
- joint joint_block_0_10: origin xyz=3.5 9.5 1.5 rpy=0 0 0 -> xyz=2.5 9.5 1.5 rpy=0 0 0
- joint joint_block_0_11: origin xyz=4.5 9.5 1.5 rpy=0 0 0 -> xyz=3.5 9.5 1.5 rpy=0 0 0
- joint joint_block_0_12: origin xyz=5.5 9.5 1.5 rpy=0 0 0 -> xyz=4.5 9.5 1.5 rpy=0 0 0
- joint joint_block_0_13: origin xyz=6.5 9.5 1.5 rpy=0 0 0 -> xyz=5.5 9.5 1.5 rpy=0 0 0
- joint joint_block_0_2: origin xyz=-4.5 9.5 1.5 rpy=0 0 0 -> xyz=-5.5 9.5 1.5 rpy=0 0 0
- joint joint_block_0_3: origin xyz=-3.5 9.5 1.5 rpy=0 0 0 -> xyz=-4.5 9.5 1.5 rpy=0 0 0
- joint joint_block_0_4: origin xyz=-2.5 9.5 1.5 rpy=0 0 0 -> xyz=-3.5 9.5 1.5 rpy=0 0 0
- joint joint_block_0_5: origin xyz=-1.5 9.5 1.5 rpy=0 0 0 -> xyz=-2.5 9.5 1.5 rpy=0 0 0
- joint joint_block_0_6: origin xyz=-0.5 9.5 1.5 rpy=0 0 0 -> xyz=-1.5 9.5 1.5 rpy=0 0 0
- joint joint_block_0_7: origin xyz=0.5 9.5 1.5 rpy=0 0 0 -> xyz=-0.5 9.5 1.5 rpy=0 0 0
- joint joint_block_0_8: origin xyz=1.5 9.5 1.5 rpy=0 0 0 -> xyz=0.5 9.5 1.5 rpy=0 0 0
- joint joint_block_0_9: origin xyz=2.5 9.5 1.5 rpy=0 0 0 -> xyz=1.5 9.5 1.5 rpy=0 0 0
- joint joint_block_10_0: origin xyz=-6.5 -0.5 1.5 rpy=0 0 0 -> xyz=-7.5 -0.5 1.5 rpy=0 0 0
- joint joint_block_11_0: origin xyz=-6.5 -1.5 1.5 rpy=0 0 0 -> xyz=-7.5 -1.5 1.5 rpy=0 0 0
- joint joint_block_12_0: origin xyz=-6.5 -2.5 1.5 rpy=0 0 0 -> xyz=-7.5 -2.5 1.5 rpy=0 0 0
- joint joint_block_13_0: origin xyz=-6.5 -3.5 1.5 rpy=0 0 0 -> xyz=-7.5 -3.5 1.5 rpy=0 0 0
- joint joint_block_14_0: origin xyz=-6.5 -4.5 1.5 rpy=0 0 0 -> xyz=-7.5 -4.5 1.5 rpy=0 0 0
- joint joint_block_15_0: origin xyz=-6.5 -5.5 1.5 rpy=0 0 0 -> xyz=-7.5 -5.5 1.5 rpy=0 0 0
- joint joint_block_16_0: origin xyz=-6.5 -6.5 1.5 rpy=0 0 0 -> xyz=-7.5 -6.5 1.5 rpy=0 0 0
- joint joint_block_17_0: origin xyz=-6.5 -7.5 1.5 rpy=0 0 0 -> xyz=-7.5 -7.5 1.5 rpy=0 0 0
- joint joint_block_18_0: origin xyz=-6.5 -8.5 1.5 rpy=0 0 0 -> xyz=-7.5 -8.5 1.5 rpy=0 0 0
- joint joint_block_19_0: origin xyz=-6.5 -9.5 1.5 rpy=0 0 0 -> xyz=-7.5 -9.5 1.5 rpy=0 0 0
- joint joint_block_19_1: origin xyz=-5.5 -9.5 1.5 rpy=0 0 0 -> xyz=-6.5 -9.5 1.5 rpy=0 0 0
- joint joint_block_19_10: origin xyz=3.5 -9.5 1.5 rpy=0 0 0 -> xyz=2.5 -9.5 1.5 rpy=0 0 0
- joint joint_block_19_11: origin xyz=4.5 -9.5 1.5 rpy=0 0 0 -> xyz=3.5 -9.5 1.5 rpy=0 0 0
- joint joint_block_19_12: origin xyz=5.5 -9.5 1.5 rpy=0 0 0 -> xyz=4.5 -9.5 1.5 rpy=0 0 0
- joint joint_block_19_13: origin xyz=6.5 -9.5 1.5 rpy=0 0 0 -> xyz=5.5 -9.5 1.5 rpy=0 0 0
- joint joint_block_19_2: origin xyz=-4.5 -9.5 1.5 rpy=0 0 0 -> xyz=-5.5 -9.5 1.5 rpy=0 0 0
- joint joint_block_19_3: origin xyz=-3.5 -9.5 1.5 rpy=0 0 0 -> xyz=-4.5 -9.5 1.5 rpy=0 0 0
- joint joint_block_19_4: origin xyz=-2.5 -9.5 1.5 rpy=0 0 0 -> xyz=-3.5 -9.5 1.5 rpy=0 0 0
- joint joint_block_19_5: origin xyz=-1.5 -9.5 1.5 rpy=0 0 0 -> xyz=-2.5 -9.5 1.5 rpy=0 0 0
- joint joint_block_19_6: origin xyz=-0.5 -9.5 1.5 rpy=0 0 0 -> xyz=-1.5 -9.5 1.5 rpy=0 0 0
- joint joint_block_19_7: origin xyz=0.5 -9.5 1.5 rpy=0 0 0 -> xyz=-0.5 -9.5 1.5 rpy=0 0 0
- joint joint_block_19_8: origin xyz=1.5 -9.5 1.5 rpy=0 0 0 -> xyz=0.5 -9.5 1.5 rpy=0 0 0
- joint joint_block_19_9: origin xyz=2.5 -9.5 1.5 rpy=0 0 0 -> xyz=1.5 -9.5 1.5 rpy=0 0 0
- joint joint_block_1_0: origin xyz=-6.5 8.5 1.5 rpy=0 0 0 -> xyz=-7.5 8.5 1.5 rpy=0 0 0
- joint joint_block_2_0: origin xyz=-6.5 7.5 1.5 rpy=0 0 0 -> xyz=-7.5 7.5 1.5 rpy=0 0 0
- joint joint_block_3_0: origin xyz=-6.5 6.5 1.5 rpy=0 0 0 -> xyz=-7.5 6.5 1.5 rpy=0 0 0
- joint joint_block_4_0: origin xyz=-6.5 5.5 1.5 rpy=0 0 0 -> xyz=-7.5 5.5 1.5 rpy=0 0 0
- joint joint_block_5_0: origin xyz=-6.5 4.5 1.5 rpy=0 0 0 -> xyz=-7.5 4.5 1.5 rpy=0 0 0
- joint joint_block_6_0: origin xyz=-6.5 3.5 1.5 rpy=0 0 0 -> xyz=-7.5 3.5 1.5 rpy=0 0 0
- joint joint_block_7_0: origin xyz=-6.5 2.5 1.5 rpy=0 0 0 -> xyz=-7.5 2.5 1.5 rpy=0 0 0
- joint joint_block_8_0: origin xyz=-6.5 1.5 1.5 rpy=0 0 0 -> xyz=-7.5 1.5 1.5 rpy=0 0 0
- joint joint_block_9_0: origin xyz=-6.5 0.5 1.5 rpy=0 0 0 -> xyz=-7.5 0.5 1.5 rpy=0 0 0
