Commit message: add deleting endpoint visual once delivery terminates and new delivery is assigned to a robot

File: assets/warehouse/workstations.urdf (robot description, URDF)
Before this commit: robot struct, 13 links, 12 joints
Links:
- removed link block_10_11
- removed link block_13_11
- removed link block_16_11
- removed link block_1_11
- removed link block_4_11
- removed link block_7_11
- added link block_10_13, mass 0; visual box size=1.0 1.0 1.5
- added link block_13_13, mass 0; visual box size=1.0 1.0 1.5
- added link block_16_13, mass 0; visual box size=1.0 1.0 1.5
- added link block_1_13, mass 0; visual box size=1.0 1.0 1.5
- added link block_4_13, mass 0; visual box size=1.0 1.0 1.5
- added link block_7_13, mass 0; visual box size=1.0 1.0 1.5
Joints:
- removed joint joint_block_10_11
- removed joint joint_block_13_11
- removed joint joint_block_16_11
- removed joint joint_block_1_11
- removed joint joint_block_4_11
- removed joint joint_block_7_11
- added joint joint_block_10_13: type fixed, parent struct_base, child block_10_13, origin xyz=6.5 -1.5 0.75 rpy=0 0 0
- added joint joint_block_13_13: type fixed, parent struct_base, child block_13_13, origin xyz=6.5 -4.5 0.75 rpy=0 0 0
- added joint joint_block_16_13: type fixed, parent struct_base, child block_16_13, origin xyz=6.5 -7.5 0.75 rpy=0 0 0
- added joint joint_block_1_13: type fixed, parent struct_base, child block_1_13, origin xyz=6.5 7.5 0.75 rpy=0 0 0
- added joint joint_block_4_13: type fixed, parent struct_base, child block_4_13, origin xyz=6.5 4.5 0.75 rpy=0 0 0
- added joint joint_block_7_13: type fixed, parent struct_base, child block_7_13, origin xyz=6.5 1.5 0.75 rpy=0 0 0
- joint joint_block_10_0: origin xyz=-5.5 -1.5 0.75 rpy=0 0 0 -> xyz=-6.5 -1.5 0.75 rpy=0 0 0
- joint joint_block_13_0: origin xyz=-5.5 -4.5 0.75 rpy=0 0 0 -> xyz=-6.5 -4.5 0.75 rpy=0 0 0
- joint joint_block_16_0: origin xyz=-5.5 -7.5 0.75 rpy=0 0 0 -> xyz=-6.5 -7.5 0.75 rpy=0 0 0
- joint joint_block_1_0: origin xyz=-5.5 7.5 0.75 rpy=0 0 0 -> xyz=-6.5 7.5 0.75 rpy=0 0 0
- joint joint_block_4_0: origin xyz=-5.5 4.5 0.75 rpy=0 0 0 -> xyz=-6.5 4.5 0.75 rpy=0 0 0
- joint joint_block_7_0: origin xyz=-5.5 1.5 0.75 rpy=0 0 0 -> xyz=-6.5 1.5 0.75 rpy=0 0 0

Commit message: fix bug when simulation terminates early even when task not all created

File: assets/warehouse/endpoints.urdf (robot description, URDF)
Before this commit: robot struct, 65 links, 64 joints
Links:
- removed link block_0_2
- removed link block_0_5
- removed link block_0_9
- removed link block_10_2
- removed link block_10_5
- removed link block_10_9
- removed link block_11_2
- removed link block_11_5
- removed link block_11_9
- removed link block_12_2
- removed link block_12_5
- removed link block_12_9
- removed link block_13_2
- removed link block_13_5
- removed link block_13_9
- removed link block_14_2
- removed link block_14_5
- removed link block_14_9
- removed link block_15_2
- removed link block_15_5
- removed link block_15_9
- removed link block_16_2
- removed link block_16_5
- removed link block_16_9
- removed link block_17_2
- removed link block_17_5
- removed link block_17_9
- removed link block_1_2
- removed link block_1_5
- removed link block_1_9
- removed link block_2_2
- removed link block_2_5
- removed link block_2_9
- removed link block_3_2
- removed link block_3_5
- removed link block_3_9
- removed link block_4_2
- removed link block_4_5
- removed link block_4_9
- removed link block_5_2
- removed link block_5_5
- removed link block_5_9
- removed link block_6_2
- removed link block_6_5
- removed link block_6_9
- removed link block_7_2
- removed link block_7_5
- removed link block_7_9
- added link block_0_10, mass 0; visual box size=1.0 1.0 0.3
- added link block_0_3, mass 0; visual box size=1.0 1.0 0.3
- added link block_0_7, mass 0; visual box size=1.0 1.0 0.3
- added link block_10_10, mass 0; visual box size=1.0 1.0 0.3
- added link block_10_3, mass 0; visual box size=1.0 1.0 0.3
- added link block_10_7, mass 0; visual box size=1.0 1.0 0.3
- added link block_11_10, mass 0; visual box size=1.0 1.0 0.3
- added link block_11_3, mass 0; visual box size=1.0 1.0 0.3
- added link block_11_7, mass 0; visual box size=1.0 1.0 0.3
- added link block_12_10, mass 0; visual box size=1.0 1.0 0.3
- added link block_12_3, mass 0; visual box size=1.0 1.0 0.3
- added link block_12_7, mass 0; visual box size=1.0 1.0 0.3
- added link block_13_10, mass 0; visual box size=1.0 1.0 0.3
- added link block_13_3, mass 0; visual box size=1.0 1.0 0.3
- added link block_13_7, mass 0; visual box size=1.0 1.0 0.3
- added link block_14_10, mass 0; visual box size=1.0 1.0 0.3
- added link block_14_3, mass 0; visual box size=1.0 1.0 0.3
- added link block_14_7, mass 0; visual box size=1.0 1.0 0.3
- added link block_15_10, mass 0; visual box size=1.0 1.0 0.3
- added link block_15_3, mass 0; visual box size=1.0 1.0 0.3
- added link block_15_7, mass 0; visual box size=1.0 1.0 0.3
- added link block_16_10, mass 0; visual box size=1.0 1.0 0.3
- added link block_16_3, mass 0; visual box size=1.0 1.0 0.3
- added link block_16_7, mass 0; visual box size=1.0 1.0 0.3
- added link block_17_10, mass 0; visual box size=1.0 1.0 0.3
- added link block_17_3, mass 0; visual box size=1.0 1.0 0.3
- added link block_17_7, mass 0; visual box size=1.0 1.0 0.3
- added link block_1_10, mass 0; visual box size=1.0 1.0 0.3
- added link block_1_3, mass 0; visual box size=1.0 1.0 0.3
- added link block_1_7, mass 0; visual box size=1.0 1.0 0.3
- added link block_2_10, mass 0; visual box size=1.0 1.0 0.3
- added link block_2_3, mass 0; visual box size=1.0 1.0 0.3
- added link block_2_7, mass 0; visual box size=1.0 1.0 0.3
- added link block_3_10, mass 0; visual box size=1.0 1.0 0.3
- added link block_3_3, mass 0; visual box size=1.0 1.0 0.3
- added link block_3_7, mass 0; visual box size=1.0 1.0 0.3
- added link block_4_10, mass 0; visual box size=1.0 1.0 0.3
- added link block_4_3, mass 0; visual box size=1.0 1.0 0.3
- added link block_4_7, mass 0; visual box size=1.0 1.0 0.3
- added link block_5_10, mass 0; visual box size=1.0 1.0 0.3
- added link block_5_3, mass 0; visual box size=1.0 1.0 0.3
- added link block_5_7, mass 0; visual box size=1.0 1.0 0.3
- added link block_6_10, mass 0; visual box size=1.0 1.0 0.3
- added link block_6_3, mass 0; visual box size=1.0 1.0 0.3
- added link block_6_7, mass 0; visual box size=1.0 1.0 0.3
- added link block_7_10, mass 0; visual box size=1.0 1.0 0.3
- added link block_7_3, mass 0; visual box size=1.0 1.0 0.3
- added link block_7_7, mass 0; visual box size=1.0 1.0 0.3
Joints:
- removed joint joint_block_0_2
- removed joint joint_block_0_5
- removed joint joint_block_0_9
- removed joint joint_block_10_2
- removed joint joint_block_10_5
- removed joint joint_block_10_9
- removed joint joint_block_11_2
- removed joint joint_block_11_5
- removed joint joint_block_11_9
- removed joint joint_block_12_2
- removed joint joint_block_12_5
- removed joint joint_block_12_9
- removed joint joint_block_13_2
- removed joint joint_block_13_5
- removed joint joint_block_13_9
- removed joint joint_block_14_2
- removed joint joint_block_14_5
- removed joint joint_block_14_9
- removed joint joint_block_15_2
- removed joint joint_block_15_5
- removed joint joint_block_15_9
- removed joint joint_block_16_2
- removed joint joint_block_16_5
- removed joint joint_block_16_9
- removed joint joint_block_17_2
- removed joint joint_block_17_5
- removed joint joint_block_17_9
- removed joint joint_block_1_2
- removed joint joint_block_1_5
- removed joint joint_block_1_9
- removed joint joint_block_2_2
- removed joint joint_block_2_5
- removed joint joint_block_2_9
- removed joint joint_block_3_2
- removed joint joint_block_3_5
- removed joint joint_block_3_9
- removed joint joint_block_4_2
- removed joint joint_block_4_5
- removed joint joint_block_4_9
- removed joint joint_block_5_2
- removed joint joint_block_5_5
- removed joint joint_block_5_9
- removed joint joint_block_6_2
- removed joint joint_block_6_5
- removed joint joint_block_6_9
- removed joint joint_block_7_2
- removed joint joint_block_7_5
- removed joint joint_block_7_9
- added joint joint_block_0_10: type fixed, parent struct_base, child block_0_10, origin xyz=3.5 8.5 0.15 rpy=0 0 0
- added joint joint_block_0_3: type fixed, parent struct_base, child block_0_3, origin xyz=-3.5 8.5 0.15 rpy=0 0 0
- added joint joint_block_0_7: type fixed, parent struct_base, child block_0_7, origin xyz=0.5 8.5 0.15 rpy=0 0 0
- added joint joint_block_10_10: type fixed, parent struct_base, child block_10_10, origin xyz=3.5 -1.5 0.15 rpy=0 0 0
- added joint joint_block_10_3: type fixed, parent struct_base, child block_10_3, origin xyz=-3.5 -1.5 0.15 rpy=0 0 0
- added joint joint_block_10_7: type fixed, parent struct_base, child block_10_7, origin xyz=0.5 -1.5 0.15 rpy=0 0 0
- added joint joint_block_11_10: type fixed, parent struct_base, child block_11_10, origin xyz=3.5 -2.5 0.15 rpy=0 0 0
- added joint joint_block_11_3: type fixed, parent struct_base, child block_11_3, origin xyz=-3.5 -2.5 0.15 rpy=0 0 0
- added joint joint_block_11_7: type fixed, parent struct_base, child block_11_7, origin xyz=0.5 -2.5 0.15 rpy=0 0 0
- added joint joint_block_12_10: type fixed, parent struct_base, child block_12_10, origin xyz=3.5 -3.5 0.15 rpy=0 0 0
- added joint joint_block_12_3: type fixed, parent struct_base, child block_12_3, origin xyz=-3.5 -3.5 0.15 rpy=0 0 0
- added joint joint_block_12_7: type fixed, parent struct_base, child block_12_7, origin xyz=0.5 -3.5 0.15 rpy=0 0 0
- added joint joint_block_13_10: type fixed, parent struct_base, child block_13_10, origin xyz=3.5 -4.5 0.15 rpy=0 0 0
- added joint joint_block_13_3: type fixed, parent struct_base, child block_13_3, origin xyz=-3.5 -4.5 0.15 rpy=0 0 0
- added joint joint_block_13_7: type fixed, parent struct_base, child block_13_7, origin xyz=0.5 -4.5 0.15 rpy=0 0 0
- added joint joint_block_14_10: type fixed, parent struct_base, child block_14_10, origin xyz=3.5 -5.5 0.15 rpy=0 0 0
- added joint joint_block_14_3: type fixed, parent struct_base, child block_14_3, origin xyz=-3.5 -5.5 0.15 rpy=0 0 0
- added joint joint_block_14_7: type fixed, parent struct_base, child block_14_7, origin xyz=0.5 -5.5 0.15 rpy=0 0 0
- added joint joint_block_15_10: type fixed, parent struct_base, child block_15_10, origin xyz=3.5 -6.5 0.15 rpy=0 0 0
- added joint joint_block_15_3: type fixed, parent struct_base, child block_15_3, origin xyz=-3.5 -6.5 0.15 rpy=0 0 0
- added joint joint_block_15_7: type fixed, parent struct_base, child block_15_7, origin xyz=0.5 -6.5 0.15 rpy=0 0 0
- added joint joint_block_16_10: type fixed, parent struct_base, child block_16_10, origin xyz=3.5 -7.5 0.15 rpy=0 0 0
- added joint joint_block_16_3: type fixed, parent struct_base, child block_16_3, origin xyz=-3.5 -7.5 0.15 rpy=0 0 0
- added joint joint_block_16_7: type fixed, parent struct_base, child block_16_7, origin xyz=0.5 -7.5 0.15 rpy=0 0 0
- added joint joint_block_17_10: type fixed, parent struct_base, child block_17_10, origin xyz=3.5 -8.5 0.15 rpy=0 0 0
- added joint joint_block_17_3: type fixed, parent struct_base, child block_17_3, origin xyz=-3.5 -8.5 0.15 rpy=0 0 0
- added joint joint_block_17_7: type fixed, parent struct_base, child block_17_7, origin xyz=0.5 -8.5 0.15 rpy=0 0 0
- added joint joint_block_1_10: type fixed, parent struct_base, child block_1_10, origin xyz=3.5 7.5 0.15 rpy=0 0 0
- added joint joint_block_1_3: type fixed, parent struct_base, child block_1_3, origin xyz=-3.5 7.5 0.15 rpy=0 0 0
- added joint joint_block_1_7: type fixed, parent struct_base, child block_1_7, origin xyz=0.5 7.5 0.15 rpy=0 0 0
- added joint joint_block_2_10: type fixed, parent struct_base, child block_2_10, origin xyz=3.5 6.5 0.15 rpy=0 0 0
- added joint joint_block_2_3: type fixed, parent struct_base, child block_2_3, origin xyz=-3.5 6.5 0.15 rpy=0 0 0
- added joint joint_block_2_7: type fixed, parent struct_base, child block_2_7, origin xyz=0.5 6.5 0.15 rpy=0 0 0
- added joint joint_block_3_10: type fixed, parent struct_base, child block_3_10, origin xyz=3.5 5.5 0.15 rpy=0 0 0
- added joint joint_block_3_3: type fixed, parent struct_base, child block_3_3, origin xyz=-3.5 5.5 0.15 rpy=0 0 0
- added joint joint_block_3_7: type fixed, parent struct_base, child block_3_7, origin xyz=0.5 5.5 0.15 rpy=0 0 0
- added joint joint_block_4_10: type fixed, parent struct_base, child block_4_10, origin xyz=3.5 4.5 0.15 rpy=0 0 0
- added joint joint_block_4_3: type fixed, parent struct_base, child block_4_3, origin xyz=-3.5 4.5 0.15 rpy=0 0 0
- added joint joint_block_4_7: type fixed, parent struct_base, child block_4_7, origin xyz=0.5 4.5 0.15 rpy=0 0 0
- added joint joint_block_5_10: type fixed, parent struct_base, child block_5_10, origin xyz=3.5 3.5 0.15 rpy=0 0 0
- added joint joint_block_5_3: type fixed, parent struct_base, child block_5_3, origin xyz=-3.5 3.5 0.15 rpy=0 0 0
- added joint joint_block_5_7: type fixed, parent struct_base, child block_5_7, origin xyz=0.5 3.5 0.15 rpy=0 0 0
- added joint joint_block_6_10: type fixed, parent struct_base, child block_6_10, origin xyz=3.5 2.5 0.15 rpy=0 0 0
- added joint joint_block_6_3: type fixed, parent struct_base, child block_6_3, origin xyz=-3.5 2.5 0.15 rpy=0 0 0
- added joint joint_block_6_7: type fixed, parent struct_base, child block_6_7, origin xyz=0.5 2.5 0.15 rpy=0 0 0
- added joint joint_block_7_10: type fixed, parent struct_base, child block_7_10, origin xyz=3.5 1.5 0.15 rpy=0 0 0
- added joint joint_block_7_3: type fixed, parent struct_base, child block_7_3, origin xyz=-3.5 1.5 0.15 rpy=0 0 0
- added joint joint_block_7_7: type fixed, parent struct_base, child block_7_7, origin xyz=0.5 1.5 0.15 rpy=0 0 0

File: assets/warehouse/shelves.urdf (robot description, URDF)
Before this commit: robot struct, 65 links, 64 joints
Links:
- removed link block_0_3
- removed link block_0_7
- removed link block_10_3
- removed link block_10_7
- removed link block_11_3
- removed link block_11_7
- removed link block_12_3
- removed link block_12_7
- removed link block_13_3
- removed link block_13_7
- removed link block_14_3
- removed link block_14_7
- removed link block_15_3
- removed link block_15_7
- removed link block_16_3
- removed link block_16_7
- removed link block_17_3
- removed link block_17_7
- removed link block_1_3
- removed link block_1_7
- removed link block_2_3
- removed link block_2_7
- removed link block_3_3
- removed link block_3_7
- removed link block_4_3
- removed link block_4_7
- removed link block_5_3
- removed link block_5_7
- removed link block_6_3
- removed link block_6_7
- removed link block_7_3
- removed link block_7_7
- added link block_0_5, mass 0; collision box size=0.7 0.7 0.7; visual box size=1.0 1.0 1
- added link block_0_9, mass 0; collision box size=0.7 0.7 0.7; visual box size=1.0 1.0 1
- added link block_10_5, mass 0; collision box size=0.7 0.7 0.7; visual box size=1.0 1.0 1
- added link block_10_9, mass 0; collision box size=0.7 0.7 0.7; visual box size=1.0 1.0 1
- added link block_11_5, mass 0; collision box size=0.7 0.7 0.7; visual box size=1.0 1.0 1
- added link block_11_9, mass 0; collision box size=0.7 0.7 0.7; visual box size=1.0 1.0 1
- added link block_12_5, mass 0; collision box size=0.7 0.7 0.7; visual box size=1.0 1.0 1
- added link block_12_9, mass 0; collision box size=0.7 0.7 0.7; visual box size=1.0 1.0 1
- added link block_13_5, mass 0; collision box size=0.7 0.7 0.7; visual box size=1.0 1.0 1
- added link block_13_9, mass 0; collision box size=0.7 0.7 0.7; visual box size=1.0 1.0 1
- added link block_14_5, mass 0; collision box size=0.7 0.7 0.7; visual box size=1.0 1.0 1
- added link block_14_9, mass 0; collision box size=0.7 0.7 0.7; visual box size=1.0 1.0 1
- added link block_15_5, mass 0; collision box size=0.7 0.7 0.7; visual box size=1.0 1.0 1
- added link block_15_9, mass 0; collision box size=0.7 0.7 0.7; visual box size=1.0 1.0 1
- added link block_16_5, mass 0; collision box size=0.7 0.7 0.7; visual box size=1.0 1.0 1
- added link block_16_9, mass 0; collision box size=0.7 0.7 0.7; visual box size=1.0 1.0 1
- added link block_17_5, mass 0; collision box size=0.7 0.7 0.7; visual box size=1.0 1.0 1
- added link block_17_9, mass 0; collision box size=0.7 0.7 0.7; visual box size=1.0 1.0 1
- added link block_1_5, mass 0; collision box size=0.7 0.7 0.7; visual box size=1.0 1.0 1
- added link block_1_9, mass 0; collision box size=0.7 0.7 0.7; visual box size=1.0 1.0 1
- added link block_2_5, mass 0; collision box size=0.7 0.7 0.7; visual box size=1.0 1.0 1
- added link block_2_9, mass 0; collision box size=0.7 0.7 0.7; visual box size=1.0 1.0 1
- added link block_3_5, mass 0; collision box size=0.7 0.7 0.7; visual box size=1.0 1.0 1
- added link block_3_9, mass 0; collision box size=0.7 0.7 0.7; visual box size=1.0 1.0 1
- added link block_4_5, mass 0; collision box size=0.7 0.7 0.7; visual box size=1.0 1.0 1
- added link block_4_9, mass 0; collision box size=0.7 0.7 0.7; visual box size=1.0 1.0 1
- added link block_5_5, mass 0; collision box size=0.7 0.7 0.7; visual box size=1.0 1.0 1
- added link block_5_9, mass 0; collision box size=0.7 0.7 0.7; visual box size=1.0 1.0 1
- added link block_6_5, mass 0; collision box size=0.7 0.7 0.7; visual box size=1.0 1.0 1
- added link block_6_9, mass 0; collision box size=0.7 0.7 0.7; visual box size=1.0 1.0 1
- added link block_7_5, mass 0; collision box size=0.7 0.7 0.7; visual box size=1.0 1.0 1
- added link block_7_9, mass 0; collision box size=0.7 0.7 0.7; visual box size=1.0 1.0 1
Joints:
- removed joint joint_block_0_3
- removed joint joint_block_0_7
- removed joint joint_block_10_3
- removed joint joint_block_10_7
- removed joint joint_block_11_3
- removed joint joint_block_11_7
- removed joint joint_block_12_3
- removed joint joint_block_12_7
- removed joint joint_block_13_3
- removed joint joint_block_13_7
- removed joint joint_block_14_3
- removed joint joint_block_14_7
- removed joint joint_block_15_3
- removed joint joint_block_15_7
- removed joint joint_block_16_3
- removed joint joint_block_16_7
- removed joint joint_block_17_3
- removed joint joint_block_17_7
- removed joint joint_block_1_3
- removed joint joint_block_1_7
- removed joint joint_block_2_3
- removed joint joint_block_2_7
- removed joint joint_block_3_3
- removed joint joint_block_3_7
- removed joint joint_block_4_3
- removed joint joint_block_4_7
- removed joint joint_block_5_3
- removed joint joint_block_5_7
- removed joint joint_block_6_3
- removed joint joint_block_6_7
- removed joint joint_block_7_3
- removed joint joint_block_7_7
- added joint joint_block_0_5: type fixed, parent struct_base, child block_0_5, origin xyz=-1.5 8.5 0.5 rpy=0 0 0
- added joint joint_block_0_9: type fixed, parent struct_base, child block_0_9, origin xyz=2.5 8.5 0.5 rpy=0 0 0
- added joint joint_block_10_5: type fixed, parent struct_base, child block_10_5, origin xyz=-1.5 -1.5 0.5 rpy=0 0 0
- added joint joint_block_10_9: type fixed, parent struct_base, child block_10_9, origin xyz=2.5 -1.5 0.5 rpy=0 0 0
- added joint joint_block_11_5: type fixed, parent struct_base, child block_11_5, origin xyz=-1.5 -2.5 0.5 rpy=0 0 0
- added joint joint_block_11_9: type fixed, parent struct_base, child block_11_9, origin xyz=2.5 -2.5 0.5 rpy=0 0 0
- added joint joint_block_12_5: type fixed, parent struct_base, child block_12_5, origin xyz=-1.5 -3.5 0.5 rpy=0 0 0
- added joint joint_block_12_9: type fixed, parent struct_base, child block_12_9, origin xyz=2.5 -3.5 0.5 rpy=0 0 0
- added joint joint_block_13_5: type fixed, parent struct_base, child block_13_5, origin xyz=-1.5 -4.5 0.5 rpy=0 0 0
- added joint joint_block_13_9: type fixed, parent struct_base, child block_13_9, origin xyz=2.5 -4.5 0.5 rpy=0 0 0
- added joint joint_block_14_5: type fixed, parent struct_base, child block_14_5, origin xyz=-1.5 -5.5 0.5 rpy=0 0 0
- added joint joint_block_14_9: type fixed, parent struct_base, child block_14_9, origin xyz=2.5 -5.5 0.5 rpy=0 0 0
- added joint joint_block_15_5: type fixed, parent struct_base, child block_15_5, origin xyz=-1.5 -6.5 0.5 rpy=0 0 0
- added joint joint_block_15_9: type fixed, parent struct_base, child block_15_9, origin xyz=2.5 -6.5 0.5 rpy=0 0 0
- added joint joint_block_16_5: type fixed, parent struct_base, child block_16_5, origin xyz=-1.5 -7.5 0.5 rpy=0 0 0
- added joint joint_block_16_9: type fixed, parent struct_base, child block_16_9, origin xyz=2.5 -7.5 0.5 rpy=0 0 0
- added joint joint_block_17_5: type fixed, parent struct_base, child block_17_5, origin xyz=-1.5 -8.5 0.5 rpy=0 0 0
- added joint joint_block_17_9: type fixed, parent struct_base, child block_17_9, origin xyz=2.5 -8.5 0.5 rpy=0 0 0
- added joint joint_block_1_5: type fixed, parent struct_base, child block_1_5, origin xyz=-1.5 7.5 0.5 rpy=0 0 0
- added joint joint_block_1_9: type fixed, parent struct_base, child block_1_9, origin xyz=2.5 7.5 0.5 rpy=0 0 0
- added joint joint_block_2_5: type fixed, parent struct_base, child block_2_5, origin xyz=-1.5 6.5 0.5 rpy=0 0 0
- added joint joint_block_2_9: type fixed, parent struct_base, child block_2_9, origin xyz=2.5 6.5 0.5 rpy=0 0 0
- added joint joint_block_3_5: type fixed, parent struct_base, child block_3_5, origin xyz=-1.5 5.5 0.5 rpy=0 0 0
- added joint joint_block_3_9: type fixed, parent struct_base, child block_3_9, origin xyz=2.5 5.5 0.5 rpy=0 0 0
- added joint joint_block_4_5: type fixed, parent struct_base, child block_4_5, origin xyz=-1.5 4.5 0.5 rpy=0 0 0
- added joint joint_block_4_9: type fixed, parent struct_base, child block_4_9, origin xyz=2.5 4.5 0.5 rpy=0 0 0
- added joint joint_block_5_5: type fixed, parent struct_base, child block_5_5, origin xyz=-1.5 3.5 0.5 rpy=0 0 0
- added joint joint_block_5_9: type fixed, parent struct_base, child block_5_9, origin xyz=2.5 3.5 0.5 rpy=0 0 0
- added joint joint_block_6_5: type fixed, parent struct_base, child block_6_5, origin xyz=-1.5 2.5 0.5 rpy=0 0 0
- added joint joint_block_6_9: type fixed, parent struct_base, child block_6_9, origin xyz=2.5 2.5 0.5 rpy=0 0 0
- added joint joint_block_7_5: type fixed, parent struct_base, child block_7_5, origin xyz=-1.5 1.5 0.5 rpy=0 0 0
- added joint joint_block_7_9: type fixed, parent struct_base, child block_7_9, origin xyz=2.5 1.5 0.5 rpy=0 0 0
