Commit message: add testing statement

File: assets/warehouse/endpoints.urdf (robot description, URDF)
Before this commit: robot struct, 65 links, 64 joints
Links:
- removed link block_0_10
- removed link block_0_3
- removed link block_0_6
- removed link block_0_7
- removed link block_10_10
- removed link block_10_3
- removed link block_10_6
- removed link block_10_7
- removed link block_11_10
- removed link block_11_3
- removed link block_11_6
- removed link block_11_7
- removed link block_12_10
- removed link block_12_3
- removed link block_12_6
- removed link block_12_7
- removed link block_13_10
- removed link block_13_3
- removed link block_13_6
- removed link block_13_7
- removed link block_14_10
- removed link block_14_3
- removed link block_14_6
- removed link block_14_7
- removed link block_15_10
- removed link block_15_3
- removed link block_15_6
- removed link block_15_7
- removed link block_16_10
- removed link block_16_3
- removed link block_16_6
- removed link block_16_7
- removed link block_17_10
- removed link block_17_3
- removed link block_17_6
- removed link block_17_7
- removed link block_1_10
- removed link block_1_3
- removed link block_1_6
- removed link block_1_7
- removed link block_2_10
- removed link block_2_3
- removed link block_2_6
- removed link block_2_7
- removed link block_3_10
- removed link block_3_6
- removed link block_3_7
- removed link block_4_10
- removed link block_4_3
- removed link block_4_6
- removed link block_4_7
- removed link block_5_10
- removed link block_5_3
- removed link block_5_6
- removed link block_5_7
- removed link block_6_10
- removed link block_6_3
- removed link block_6_6
- removed link block_6_7
- removed link block_7_10
- removed link block_7_3
- removed link block_7_6
- removed link block_7_7
- added link block_3_0, mass 0; visual box size=1.0 1.0 0.3
- added link block_3_1, mass 0; visual box size=1.0 1.0 0.3
- added link block_3_2, mass 0; visual box size=1.0 1.0 0.3
Joints:
- removed joint joint_block_0_10
- removed joint joint_block_0_3
- removed joint joint_block_0_6
- removed joint joint_block_0_7
- removed joint joint_block_10_10
- removed joint joint_block_10_3
- removed joint joint_block_10_6
- removed joint joint_block_10_7
- removed joint joint_block_11_10
- removed joint joint_block_11_3
- removed joint joint_block_11_6
- removed joint joint_block_11_7
- removed joint joint_block_12_10
- removed joint joint_block_12_3
- removed joint joint_block_12_6
- removed joint joint_block_12_7
- removed joint joint_block_13_10
- removed joint joint_block_13_3
- removed joint joint_block_13_6
- removed joint joint_block_13_7
- removed joint joint_block_14_10
- removed joint joint_block_14_3
- removed joint joint_block_14_6
- removed joint joint_block_14_7
- removed joint joint_block_15_10
- removed joint joint_block_15_3
- removed joint joint_block_15_6
- removed joint joint_block_15_7
- removed joint joint_block_16_10
- removed joint joint_block_16_3
- removed joint joint_block_16_6
- removed joint joint_block_16_7
- removed joint joint_block_17_10
- removed joint joint_block_17_3
- removed joint joint_block_17_6
- removed joint joint_block_17_7
- removed joint joint_block_1_10
- removed joint joint_block_1_3
- removed joint joint_block_1_6
- removed joint joint_block_1_7
- removed joint joint_block_2_10
- removed joint joint_block_2_3
- removed joint joint_block_2_6
- removed joint joint_block_2_7
- removed joint joint_block_3_10
- removed joint joint_block_3_6
- removed joint joint_block_3_7
- removed joint joint_block_4_10
- removed joint joint_block_4_3
- removed joint joint_block_4_6
- removed joint joint_block_4_7
- removed joint joint_block_5_10
- removed joint joint_block_5_3
- removed joint joint_block_5_6
- removed joint joint_block_5_7
- removed joint joint_block_6_10
- removed joint joint_block_6_3
- removed joint joint_block_6_6
- removed joint joint_block_6_7
- removed joint joint_block_7_10
- removed joint joint_block_7_3
- removed joint joint_block_7_6
- removed joint joint_block_7_7
- added joint joint_block_3_0: type fixed, parent struct_base, child block_3_0, origin xyz=-1.5 -1.5 0.15 rpy=0 0 0
- added joint joint_block_3_1: type fixed, parent struct_base, child block_3_1, origin xyz=-0.5 -1.5 0.15 rpy=0 0 0
- added joint joint_block_3_2: type fixed, parent struct_base, child block_3_2, origin xyz=0.5 -1.5 0.15 rpy=0 0 0
- joint joint_block_3_3: origin xyz=-3.5 5.5 0.15 rpy=0 0 0 -> xyz=1.5 -1.5 0.15 rpy=0 0 0

File: assets/warehouse/shelves.urdf (robot description, URDF)
Before this commit: robot struct, 65 links, 64 joints
Links:
- removed link block_0_4
- removed link block_0_5
- removed link block_0_8
- removed link block_0_9
- removed link block_10_4
- removed link block_10_5
- removed link block_10_8
- removed link block_10_9
- removed link block_11_4
- removed link block_11_5
- removed link block_11_8
- removed link block_11_9
- removed link block_12_4
- removed link block_12_5
- removed link block_12_8
- removed link block_12_9
- removed link block_13_4
- removed link block_13_5
- removed link block_13_8
- removed link block_13_9
- removed link block_14_4
- removed link block_14_5
- removed link block_14_8
- removed link block_14_9
- removed link block_15_4
- removed link block_15_5
- removed link block_15_8
- removed link block_15_9
- removed link block_16_4
- removed link block_16_5
- removed link block_16_8
- removed link block_16_9
- removed link block_17_4
- removed link block_17_5
- removed link block_17_8
- removed link block_17_9
- removed link block_1_4
- removed link block_1_5
- removed link block_1_8
- removed link block_1_9
- removed link block_2_4
- removed link block_2_5
- removed link block_2_8
- removed link block_2_9
- removed link block_3_4
- removed link block_3_5
- removed link block_3_8
- removed link block_3_9
- removed link block_4_4
- removed link block_4_5
- removed link block_4_8
- removed link block_4_9
- removed link block_5_4
- removed link block_5_5
- removed link block_5_8
- removed link block_5_9
- removed link block_6_4
- removed link block_6_5
- removed link block_6_8
- removed link block_6_9
- removed link block_7_4
- removed link block_7_5
- removed link block_7_8
- removed link block_7_9
- added link block_2_1, mass 0; collision box size=0.7 0.7 0.7; visual box size=1.0 1.0 1
- added link block_2_2, mass 0; collision box size=0.7 0.7 0.7; visual box size=1.0 1.0 1
- added link block_2_3, mass 0; collision box size=0.7 0.7 0.7; visual box size=1.0 1.0 1
Joints:
- removed joint joint_block_0_4
- removed joint joint_block_0_5
- removed joint joint_block_0_8
- removed joint joint_block_0_9
- removed joint joint_block_10_4
- removed joint joint_block_10_5
- removed joint joint_block_10_8
- removed joint joint_block_10_9
- removed joint joint_block_11_4
- removed joint joint_block_11_5
- removed joint joint_block_11_8
- removed joint joint_block_11_9
- removed joint joint_block_12_4
- removed joint joint_block_12_5
- removed joint joint_block_12_8
- removed joint joint_block_12_9
- removed joint joint_block_13_4
- removed joint joint_block_13_5
- removed joint joint_block_13_8
- removed joint joint_block_13_9
- removed joint joint_block_14_4
- removed joint joint_block_14_5
- removed joint joint_block_14_8
- removed joint joint_block_14_9
- removed joint joint_block_15_4
- removed joint joint_block_15_5
- removed joint joint_block_15_8
- removed joint joint_block_15_9
- removed joint joint_block_16_4
- removed joint joint_block_16_5
- removed joint joint_block_16_8
- removed joint joint_block_16_9
- removed joint joint_block_17_4
- removed joint joint_block_17_5
- removed joint joint_block_17_8
- removed joint joint_block_17_9
- removed joint joint_block_1_4
- removed joint joint_block_1_5
- removed joint joint_block_1_8
- removed joint joint_block_1_9
- removed joint joint_block_2_4
- removed joint joint_block_2_5
- removed joint joint_block_2_8
- removed joint joint_block_2_9
- removed joint joint_block_3_4
- removed joint joint_block_3_5
- removed joint joint_block_3_8
- removed joint joint_block_3_9
- removed joint joint_block_4_4
- removed joint joint_block_4_5
- removed joint joint_block_4_8
- removed joint joint_block_4_9
- removed joint joint_block_5_4
- removed joint joint_block_5_5
- removed joint joint_block_5_8
- removed joint joint_block_5_9
- removed joint joint_block_6_4
- removed joint joint_block_6_5
- removed joint joint_block_6_8
- removed joint joint_block_6_9
- removed joint joint_block_7_4
- removed joint joint_block_7_5
- removed joint joint_block_7_8
- removed joint joint_block_7_9
- added joint joint_block_2_1: type fixed, parent struct_base, child block_2_1, origin xyz=-0.5 -0.5 0.5 rpy=0 0 0
- added joint joint_block_2_2: type fixed, parent struct_base, child block_2_2, origin xyz=0.5 -0.5 0.5 rpy=0 0 0
- added joint joint_block_2_3: type fixed, parent struct_base, child block_2_3, origin xyz=1.5 -0.5 0.5 rpy=0 0 0

File: assets/warehouse/wall.urdf (robot description, URDF)
Before this commit: robot struct, 69 links, 68 joints
Links:
- removed link block_0_10
- removed link block_0_11
- removed link block_0_12
- removed link block_0_13
- removed link block_0_14
- removed link block_0_15
- removed link block_0_6
- removed link block_0_7
- removed link block_0_8
- removed link block_0_9
- removed link block_10_0
- removed link block_10_15
- removed link block_11_0
- removed link block_11_15
- removed link block_12_0
- removed link block_12_15
- removed link block_13_0
- removed link block_13_15
- removed link block_14_0
- removed link block_14_15
- removed link block_15_0
- removed link block_15_15
- removed link block_16_0
- removed link block_16_15
- removed link block_17_0
- removed link block_17_15
- removed link block_18_0
- removed link block_18_15
- removed link block_19_0
- removed link block_19_1
- removed link block_19_10
- removed link block_19_11
- removed link block_19_12
- removed link block_19_13
- removed link block_19_14
- removed link block_19_15
- removed link block_19_2
- removed link block_19_3
- removed link block_19_4
- removed link block_19_5
- removed link block_19_6
- removed link block_19_7
- removed link block_19_8
- removed link block_19_9
- removed link block_1_15
- removed link block_2_15
- removed link block_3_15
- removed link block_4_15
- removed link block_5_15
- removed link block_6_0
- removed link block_6_15
- removed link block_7_0
- removed link block_7_15
- removed link block_8_0
- removed link block_8_15
- removed link block_9_0
- removed link block_9_15
- added link block_1_5, mass 0; collision box size=1.0 1.0 3.0; visual box size=1.0 1.0 3
- added link block_2_5, mass 0; collision box size=1.0 1.0 3.0; visual box size=1.0 1.0 3
- added link block_3_5, mass 0; collision box size=1.0 1.0 3.0; visual box size=1.0 1.0 3
- added link block_4_5, mass 0; collision box size=1.0 1.0 3.0; visual box size=1.0 1.0 3
- added link block_5_1, mass 0; collision box size=1.0 1.0 3.0; visual box size=1.0 1.0 3
- added link block_5_2, mass 0; collision box size=1.0 1.0 3.0; visual box size=1.0 1.0 3
- added link block_5_3, mass 0; collision box size=1.0 1.0 3.0; visual box size=1.0 1.0 3
- added link block_5_4, mass 0; collision box size=1.0 1.0 3.0; visual box size=1.0 1.0 3
- added link block_5_5, mass 0; collision box size=1.0 1.0 3.0; visual box size=1.0 1.0 3
Joints:
- removed joint joint_block_0_10
- removed joint joint_block_0_11
- removed joint joint_block_0_12
- removed joint joint_block_0_13
- removed joint joint_block_0_14
- removed joint joint_block_0_15
- removed joint joint_block_0_6
- removed joint joint_block_0_7
- removed joint joint_block_0_8
- removed joint joint_block_0_9
- removed joint joint_block_10_0
- removed joint joint_block_10_15
- removed joint joint_block_11_0
- removed joint joint_block_11_15
- removed joint joint_block_12_0
- removed joint joint_block_12_15
- removed joint joint_block_13_0
- removed joint joint_block_13_15
- removed joint joint_block_14_0
- removed joint joint_block_14_15
- removed joint joint_block_15_0
- removed joint joint_block_15_15
- removed joint joint_block_16_0
- removed joint joint_block_16_15
- removed joint joint_block_17_0
- removed joint joint_block_17_15
- removed joint joint_block_18_0
- removed joint joint_block_18_15
- removed joint joint_block_19_0
- removed joint joint_block_19_1
- removed joint joint_block_19_10
- removed joint joint_block_19_11
- removed joint joint_block_19_12
- removed joint joint_block_19_13
- removed joint joint_block_19_14
- removed joint joint_block_19_15
- removed joint joint_block_19_2
- removed joint joint_block_19_3
- removed joint joint_block_19_4
- removed joint joint_block_19_5
- removed joint joint_block_19_6
- removed joint joint_block_19_7
- removed joint joint_block_19_8
- removed joint joint_block_19_9
- removed joint joint_block_1_15
- removed joint joint_block_2_15
- removed joint joint_block_3_15
- removed joint joint_block_4_15
- removed joint joint_block_5_15
- removed joint joint_block_6_0
- removed joint joint_block_6_15
- removed joint joint_block_7_0
- removed joint joint_block_7_15
- removed joint joint_block_8_0
- removed joint joint_block_8_15
- removed joint joint_block_9_0
- removed joint joint_block_9_15
- added joint joint_block_1_5: type fixed, parent struct_base, child block_1_5, origin xyz=2.5 1.5 1.5 rpy=0 0 0
- added joint joint_block_2_5: type fixed, parent struct_base, child block_2_5, origin xyz=2.5 0.5 1.5 rpy=0 0 0
- added joint joint_block_3_5: type fixed, parent struct_base, child block_3_5, origin xyz=2.5 -0.5 1.5 rpy=0 0 0
- added joint joint_block_4_5: type fixed, parent struct_base, child block_4_5, origin xyz=2.5 -1.5 1.5 rpy=0 0 0
- added joint joint_block_5_1: type fixed, parent struct_base, child block_5_1, origin xyz=-1.5 -2.5 1.5 rpy=0 0 0
- added joint joint_block_5_2: type fixed, parent struct_base, child block_5_2, origin xyz=-0.5 -2.5 1.5 rpy=0 0 0
- added joint joint_block_5_3: type fixed, parent struct_base, child block_5_3, origin xyz=0.5 -2.5 1.5 rpy=0 0 0
- added joint joint_block_5_4: type fixed, parent struct_base, child block_5_4, origin xyz=1.5 -2.5 1.5 rpy=0 0 0
- added joint joint_block_5_5: type fixed, parent struct_base, child block_5_5, origin xyz=2.5 -2.5 1.5 rpy=0 0 0
- joint joint_block_0_0: origin xyz=-7.5 9.5 1.5 rpy=0 0 0 -> xyz=-2.5 2.5 1.5 rpy=0 0 0
- joint joint_block_0_1: origin xyz=-6.5 9.5 1.5 rpy=0 0 0 -> xyz=-1.5 2.5 1.5 rpy=0 0 0
- joint joint_block_0_2: origin xyz=-5.5 9.5 1.5 rpy=0 0 0 -> xyz=-0.5 2.5 1.5 rpy=0 0 0
- joint joint_block_0_3: origin xyz=-4.5 9.5 1.5 rpy=0 0 0 -> xyz=0.5 2.5 1.5 rpy=0 0 0
- joint joint_block_0_4: origin xyz=-3.5 9.5 1.5 rpy=0 0 0 -> xyz=1.5 2.5 1.5 rpy=0 0 0
- joint joint_block_0_5: origin xyz=-2.5 9.5 1.5 rpy=0 0 0 -> xyz=2.5 2.5 1.5 rpy=0 0 0
- joint joint_block_1_0: origin xyz=-7.5 8.5 1.5 rpy=0 0 0 -> xyz=-2.5 1.5 1.5 rpy=0 0 0
- joint joint_block_2_0: origin xyz=-7.5 7.5 1.5 rpy=0 0 0 -> xyz=-2.5 0.5 1.5 rpy=0 0 0
- joint joint_block_3_0: origin xyz=-7.5 6.5 1.5 rpy=0 0 0 -> xyz=-2.5 -0.5 1.5 rpy=0 0 0
- joint joint_block_4_0: origin xyz=-7.5 5.5 1.5 rpy=0 0 0 -> xyz=-2.5 -1.5 1.5 rpy=0 0 0
- joint joint_block_5_0: origin xyz=-7.5 4.5 1.5 rpy=0 0 0 -> xyz=-2.5 -2.5 1.5 rpy=0 0 0

File: assets/warehouse/workstations.urdf (robot description, URDF)
Before this commit: robot struct, 13 links, 12 joints
Links:
- removed link block_10_0
- removed link block_10_13
- removed link block_13_0
- removed link block_13_13
- removed link block_16_0
- removed link block_16_13
- removed link block_1_0
- removed link block_1_13
- removed link block_4_0
- removed link block_4_13
- removed link block_7_0
- removed link block_7_13
- added link block_0_0, mass 0; visual box size=1.0 1.0 1.5
- added link block_0_1, mass 0; visual box size=1.0 1.0 1.5
- added link block_0_2, mass 0; visual box size=1.0 1.0 1.5
- added link block_0_3, mass 0; visual box size=1.0 1.0 1.5
Joints:
- removed joint joint_block_10_0
- removed joint joint_block_10_13
- removed joint joint_block_13_0
- removed joint joint_block_13_13
- removed joint joint_block_16_0
- removed joint joint_block_16_13
- removed joint joint_block_1_0
- removed joint joint_block_1_13
- removed joint joint_block_4_0
- removed joint joint_block_4_13
- removed joint joint_block_7_0
- removed joint joint_block_7_13
- added joint joint_block_0_0: type fixed, parent struct_base, child block_0_0, origin xyz=-1.5 1.5 0.75 rpy=0 0 0
- added joint joint_block_0_1: type fixed, parent struct_base, child block_0_1, origin xyz=-0.5 1.5 0.75 rpy=0 0 0
- added joint joint_block_0_2: type fixed, parent struct_base, child block_0_2, origin xyz=0.5 1.5 0.75 rpy=0 0 0
- added joint joint_block_0_3: type fixed, parent struct_base, child block_0_3, origin xyz=1.5 1.5 0.75 rpy=0 0 0
