Commit message: add shy-cbs

File: assets/warehouse/endpoints.urdf (robot description, URDF)
Before this commit: robot struct, 5 links, 4 joints
Links:
- removed link block_3_0
- removed link block_3_1
- removed link block_3_2
- removed link block_3_3
- added link block_7_0, mass 0; visual box size=1.0 1.0 0.3
- added link block_7_1, mass 0; visual box size=1.0 1.0 0.3
- added link block_7_2, mass 0; visual box size=1.0 1.0 0.3
- added link block_7_3, mass 0; visual box size=1.0 1.0 0.3
- added link block_7_4, mass 0; visual box size=1.0 1.0 0.3
- added link block_7_5, mass 0; visual box size=1.0 1.0 0.3
- added link block_7_6, mass 0; visual box size=1.0 1.0 0.3
- added link block_7_7, mass 0; visual box size=1.0 1.0 0.3
- added link block_7_8, mass 0; visual box size=1.0 1.0 0.3
- added link block_7_9, mass 0; visual box size=1.0 1.0 0.3
Joints:
- removed joint joint_block_3_0
- removed joint joint_block_3_1
- removed joint joint_block_3_2
- removed joint joint_block_3_3
- added joint joint_block_7_0: type fixed, parent struct_base, child block_7_0, origin xyz=-4.5 -3.5 0.15 rpy=0 0 0
- added joint joint_block_7_1: type fixed, parent struct_base, child block_7_1, origin xyz=-3.5 -3.5 0.15 rpy=0 0 0
- added joint joint_block_7_2: type fixed, parent struct_base, child block_7_2, origin xyz=-2.5 -3.5 0.15 rpy=0 0 0
- added joint joint_block_7_3: type fixed, parent struct_base, child block_7_3, origin xyz=-1.5 -3.5 0.15 rpy=0 0 0
- added joint joint_block_7_4: type fixed, parent struct_base, child block_7_4, origin xyz=-0.5 -3.5 0.15 rpy=0 0 0
- added joint joint_block_7_5: type fixed, parent struct_base, child block_7_5, origin xyz=0.5 -3.5 0.15 rpy=0 0 0
- added joint joint_block_7_6: type fixed, parent struct_base, child block_7_6, origin xyz=1.5 -3.5 0.15 rpy=0 0 0
- added joint joint_block_7_7: type fixed, parent struct_base, child block_7_7, origin xyz=2.5 -3.5 0.15 rpy=0 0 0
- added joint joint_block_7_8: type fixed, parent struct_base, child block_7_8, origin xyz=3.5 -3.5 0.15 rpy=0 0 0
- added joint joint_block_7_9: type fixed, parent struct_base, child block_7_9, origin xyz=4.5 -3.5 0.15 rpy=0 0 0

File: assets/warehouse/shelves.urdf (robot description, URDF)
Before this commit: robot struct, 4 links, 3 joints
Links:
- removed link block_2_1
- removed link block_2_2
- removed link block_2_3
- added link block_5_1, mass 0; collision box size=0.7 0.7 0.7; visual box size=1.0 1.0 1
- added link block_5_2, mass 0; collision box size=0.7 0.7 0.7; visual box size=1.0 1.0 1
- added link block_5_3, mass 0; collision box size=0.7 0.7 0.7; visual box size=1.0 1.0 1
- added link block_5_4, mass 0; collision box size=0.7 0.7 0.7; visual box size=1.0 1.0 1
- added link block_5_5, mass 0; collision box size=0.7 0.7 0.7; visual box size=1.0 1.0 1
- added link block_5_6, mass 0; collision box size=0.7 0.7 0.7; visual box size=1.0 1.0 1
- added link block_5_7, mass 0; collision box size=0.7 0.7 0.7; visual box size=1.0 1.0 1
- added link block_5_8, mass 0; collision box size=0.7 0.7 0.7; visual box size=1.0 1.0 1
- added link block_5_9, mass 0; collision box size=0.7 0.7 0.7; visual box size=1.0 1.0 1
Joints:
- removed joint joint_block_2_1
- removed joint joint_block_2_2
- removed joint joint_block_2_3
- added joint joint_block_5_1: type fixed, parent struct_base, child block_5_1, origin xyz=-3.5 -1.5 0.5 rpy=0 0 0
- added joint joint_block_5_2: type fixed, parent struct_base, child block_5_2, origin xyz=-2.5 -1.5 0.5 rpy=0 0 0
- added joint joint_block_5_3: type fixed, parent struct_base, child block_5_3, origin xyz=-1.5 -1.5 0.5 rpy=0 0 0
- added joint joint_block_5_4: type fixed, parent struct_base, child block_5_4, origin xyz=-0.5 -1.5 0.5 rpy=0 0 0
- added joint joint_block_5_5: type fixed, parent struct_base, child block_5_5, origin xyz=0.5 -1.5 0.5 rpy=0 0 0
- added joint joint_block_5_6: type fixed, parent struct_base, child block_5_6, origin xyz=1.5 -1.5 0.5 rpy=0 0 0
- added joint joint_block_5_7: type fixed, parent struct_base, child block_5_7, origin xyz=2.5 -1.5 0.5 rpy=0 0 0
- added joint joint_block_5_8: type fixed, parent struct_base, child block_5_8, origin xyz=3.5 -1.5 0.5 rpy=0 0 0
- added joint joint_block_5_9: type fixed, parent struct_base, child block_5_9, origin xyz=4.5 -1.5 0.5 rpy=0 0 0

File: assets/warehouse/wall.urdf (robot description, URDF)
Before this commit: robot struct, 21 links, 20 joints
Links:
- removed link block_1_5
- removed link block_2_5
- removed link block_3_5
- removed link block_4_5
- removed link block_5_1
- removed link block_5_2
- removed link block_5_3
- removed link block_5_4
- removed link block_5_5
- added link block_0_10, mass 0; collision box size=1.0 1.0 3.0; visual box size=1.0 1.0 3
- added link block_0_11, mass 0; collision box size=1.0 1.0 3.0; visual box size=1.0 1.0 3
- added link block_0_6, mass 0; collision box size=1.0 1.0 3.0; visual box size=1.0 1.0 3
- added link block_0_7, mass 0; collision box size=1.0 1.0 3.0; visual box size=1.0 1.0 3
- added link block_0_8, mass 0; collision box size=1.0 1.0 3.0; visual box size=1.0 1.0 3
- added link block_0_9, mass 0; collision box size=1.0 1.0 3.0; visual box size=1.0 1.0 3
- added link block_1_11, mass 0; collision box size=1.0 1.0 3.0; visual box size=1.0 1.0 3
- added link block_2_11, mass 0; collision box size=1.0 1.0 3.0; visual box size=1.0 1.0 3
- added link block_3_11, mass 0; collision box size=1.0 1.0 3.0; visual box size=1.0 1.0 3
- added link block_4_11, mass 0; collision box size=1.0 1.0 3.0; visual box size=1.0 1.0 3
- added link block_5_11, mass 0; collision box size=1.0 1.0 3.0; visual box size=1.0 1.0 3
- added link block_6_0, mass 0; collision box size=1.0 1.0 3.0; visual box size=1.0 1.0 3
- added link block_6_11, mass 0; collision box size=1.0 1.0 3.0; visual box size=1.0 1.0 3
- added link block_7_0, mass 0; collision box size=1.0 1.0 3.0; visual box size=1.0 1.0 3
- added link block_7_11, mass 0; collision box size=1.0 1.0 3.0; visual box size=1.0 1.0 3
- added link block_8_0, mass 0; collision box size=1.0 1.0 3.0; visual box size=1.0 1.0 3
- added link block_8_11, mass 0; collision box size=1.0 1.0 3.0; visual box size=1.0 1.0 3
- added link block_9_0, mass 0; collision box size=1.0 1.0 3.0; visual box size=1.0 1.0 3
- added link block_9_1, mass 0; collision box size=1.0 1.0 3.0; visual box size=1.0 1.0 3
- added link block_9_10, mass 0; collision box size=1.0 1.0 3.0; visual box size=1.0 1.0 3
- added link block_9_11, mass 0; collision box size=1.0 1.0 3.0; visual box size=1.0 1.0 3
- added link block_9_2, mass 0; collision box size=1.0 1.0 3.0; visual box size=1.0 1.0 3
- added link block_9_3, mass 0; collision box size=1.0 1.0 3.0; visual box size=1.0 1.0 3
- added link block_9_4, mass 0; collision box size=1.0 1.0 3.0; visual box size=1.0 1.0 3
- added link block_9_5, mass 0; collision box size=1.0 1.0 3.0; visual box size=1.0 1.0 3
- added link block_9_6, mass 0; collision box size=1.0 1.0 3.0; visual box size=1.0 1.0 3
- added link block_9_7, mass 0; collision box size=1.0 1.0 3.0; visual box size=1.0 1.0 3
- added link block_9_8, mass 0; collision box size=1.0 1.0 3.0; visual box size=1.0 1.0 3
- added link block_9_9, mass 0; collision box size=1.0 1.0 3.0; visual box size=1.0 1.0 3
Joints:
- removed joint joint_block_1_5
- removed joint joint_block_2_5
- removed joint joint_block_3_5
- removed joint joint_block_4_5
- removed joint joint_block_5_1
- removed joint joint_block_5_2
- removed joint joint_block_5_3
- removed joint joint_block_5_4
- removed joint joint_block_5_5
- added joint joint_block_0_10: type fixed, parent struct_base, child block_0_10, origin xyz=4.5 4.5 1.5 rpy=0 0 0
- added joint joint_block_0_11: type fixed, parent struct_base, child block_0_11, origin xyz=5.5 4.5 1.5 rpy=0 0 0
- added joint joint_block_0_6: type fixed, parent struct_base, child block_0_6, origin xyz=0.5 4.5 1.5 rpy=0 0 0
- added joint joint_block_0_7: type fixed, parent struct_base, child block_0_7, origin xyz=1.5 4.5 1.5 rpy=0 0 0
- added joint joint_block_0_8: type fixed, parent struct_base, child block_0_8, origin xyz=2.5 4.5 1.5 rpy=0 0 0
- added joint joint_block_0_9: type fixed, parent struct_base, child block_0_9, origin xyz=3.5 4.5 1.5 rpy=0 0 0
- added joint joint_block_1_11: type fixed, parent struct_base, child block_1_11, origin xyz=5.5 3.5 1.5 rpy=0 0 0
- added joint joint_block_2_11: type fixed, parent struct_base, child block_2_11, origin xyz=5.5 2.5 1.5 rpy=0 0 0
- added joint joint_block_3_11: type fixed, parent struct_base, child block_3_11, origin xyz=5.5 1.5 1.5 rpy=0 0 0
- added joint joint_block_4_11: type fixed, parent struct_base, child block_4_11, origin xyz=5.5 0.5 1.5 rpy=0 0 0
- added joint joint_block_5_11: type fixed, parent struct_base, child block_5_11, origin xyz=5.5 -0.5 1.5 rpy=0 0 0
- added joint joint_block_6_0: type fixed, parent struct_base, child block_6_0, origin xyz=-5.5 -1.5 1.5 rpy=0 0 0
- added joint joint_block_6_11: type fixed, parent struct_base, child block_6_11, origin xyz=5.5 -1.5 1.5 rpy=0 0 0
- added joint joint_block_7_0: type fixed, parent struct_base, child block_7_0, origin xyz=-5.5 -2.5 1.5 rpy=0 0 0
- added joint joint_block_7_11: type fixed, parent struct_base, child block_7_11, origin xyz=5.5 -2.5 1.5 rpy=0 0 0
- added joint joint_block_8_0: type fixed, parent struct_base, child block_8_0, origin xyz=-5.5 -3.5 1.5 rpy=0 0 0
- added joint joint_block_8_11: type fixed, parent struct_base, child block_8_11, origin xyz=5.5 -3.5 1.5 rpy=0 0 0
- added joint joint_block_9_0: type fixed, parent struct_base, child block_9_0, origin xyz=-5.5 -4.5 1.5 rpy=0 0 0
- added joint joint_block_9_1: type fixed, parent struct_base, child block_9_1, origin xyz=-4.5 -4.5 1.5 rpy=0 0 0
- added joint joint_block_9_10: type fixed, parent struct_base, child block_9_10, origin xyz=4.5 -4.5 1.5 rpy=0 0 0
- added joint joint_block_9_11: type fixed, parent struct_base, child block_9_11, origin xyz=5.5 -4.5 1.5 rpy=0 0 0
- added joint joint_block_9_2: type fixed, parent struct_base, child block_9_2, origin xyz=-3.5 -4.5 1.5 rpy=0 0 0
- added joint joint_block_9_3: type fixed, parent struct_base, child block_9_3, origin xyz=-2.5 -4.5 1.5 rpy=0 0 0
- added joint joint_block_9_4: type fixed, parent struct_base, child block_9_4, origin xyz=-1.5 -4.5 1.5 rpy=0 0 0
- added joint joint_block_9_5: type fixed, parent struct_base, child block_9_5, origin xyz=-0.5 -4.5 1.5 rpy=0 0 0
- added joint joint_block_9_6: type fixed, parent struct_base, child block_9_6, origin xyz=0.5 -4.5 1.5 rpy=0 0 0
- added joint joint_block_9_7: type fixed, parent struct_base, child block_9_7, origin xyz=1.5 -4.5 1.5 rpy=0 0 0
- added joint joint_block_9_8: type fixed, parent struct_base, child block_9_8, origin xyz=2.5 -4.5 1.5 rpy=0 0 0
- added joint joint_block_9_9: type fixed, parent struct_base, child block_9_9, origin xyz=3.5 -4.5 1.5 rpy=0 0 0
- joint joint_block_0_0: origin xyz=-2.5 2.5 1.5 rpy=0 0 0 -> xyz=-5.5 4.5 1.5 rpy=0 0 0
- joint joint_block_0_1: origin xyz=-1.5 2.5 1.5 rpy=0 0 0 -> xyz=-4.5 4.5 1.5 rpy=0 0 0
- joint joint_block_0_2: origin xyz=-0.5 2.5 1.5 rpy=0 0 0 -> xyz=-3.5 4.5 1.5 rpy=0 0 0
- joint joint_block_0_3: origin xyz=0.5 2.5 1.5 rpy=0 0 0 -> xyz=-2.5 4.5 1.5 rpy=0 0 0
- joint joint_block_0_4: origin xyz=1.5 2.5 1.5 rpy=0 0 0 -> xyz=-1.5 4.5 1.5 rpy=0 0 0
- joint joint_block_0_5: origin xyz=2.5 2.5 1.5 rpy=0 0 0 -> xyz=-0.5 4.5 1.5 rpy=0 0 0
- joint joint_block_1_0: origin xyz=-2.5 1.5 1.5 rpy=0 0 0 -> xyz=-5.5 3.5 1.5 rpy=0 0 0
- joint joint_block_2_0: origin xyz=-2.5 0.5 1.5 rpy=0 0 0 -> xyz=-5.5 2.5 1.5 rpy=0 0 0
- joint joint_block_3_0: origin xyz=-2.5 -0.5 1.5 rpy=0 0 0 -> xyz=-5.5 1.5 1.5 rpy=0 0 0
- joint joint_block_4_0: origin xyz=-2.5 -1.5 1.5 rpy=0 0 0 -> xyz=-5.5 0.5 1.5 rpy=0 0 0
- joint joint_block_5_0: origin xyz=-2.5 -2.5 1.5 rpy=0 0 0 -> xyz=-5.5 -0.5 1.5 rpy=0 0 0

File: assets/warehouse/workstations.urdf (robot description, URDF)
Before this commit: robot struct, 5 links, 4 joints
Links:
- added link block_0_4, mass 0; visual box size=1.0 1.0 1.5
- added link block_0_5, mass 0; visual box size=1.0 1.0 1.5
- added link block_0_6, mass 0; visual box size=1.0 1.0 1.5
- added link block_0_7, mass 0; visual box size=1.0 1.0 1.5
- added link block_0_8, mass 0; visual box size=1.0 1.0 1.5
- added link block_0_9, mass 0; visual box size=1.0 1.0 1.5
Joints:
- added joint joint_block_0_4: type fixed, parent struct_base, child block_0_4, origin xyz=-0.5 3.5 0.75 rpy=0 0 0
- added joint joint_block_0_5: type fixed, parent struct_base, child block_0_5, origin xyz=0.5 3.5 0.75 rpy=0 0 0
- added joint joint_block_0_6: type fixed, parent struct_base, child block_0_6, origin xyz=1.5 3.5 0.75 rpy=0 0 0
- added joint joint_block_0_7: type fixed, parent struct_base, child block_0_7, origin xyz=2.5 3.5 0.75 rpy=0 0 0
- added joint joint_block_0_8: type fixed, parent struct_base, child block_0_8, origin xyz=3.5 3.5 0.75 rpy=0 0 0
- added joint joint_block_0_9: type fixed, parent struct_base, child block_0_9, origin xyz=4.5 3.5 0.75 rpy=0 0 0
- joint joint_block_0_0: origin xyz=-1.5 1.5 0.75 rpy=0 0 0 -> xyz=-4.5 3.5 0.75 rpy=0 0 0
- joint joint_block_0_1: origin xyz=-0.5 1.5 0.75 rpy=0 0 0 -> xyz=-3.5 3.5 0.75 rpy=0 0 0
- joint joint_block_0_2: origin xyz=0.5 1.5 0.75 rpy=0 0 0 -> xyz=-2.5 3.5 0.75 rpy=0 0 0
- joint joint_block_0_3: origin xyz=1.5 1.5 0.75 rpy=0 0 0 -> xyz=-1.5 3.5 0.75 rpy=0 0 0

Commit message: fix shy cbs not working according to specification

File: assets/warehouse/endpoints.urdf (robot description, URDF)
Before this commit: robot struct, 11 links, 10 joints
Links:
- removed link block_7_0
- removed link block_7_1
- removed link block_7_2
- removed link block_7_3
- removed link block_7_4
- removed link block_7_5
- removed link block_7_6
- removed link block_7_7
- removed link block_7_8
- removed link block_7_9
- added link block_3_0, mass 0; visual box size=1.0 1.0 0.3
- added link block_3_1, mass 0; visual box size=1.0 1.0 0.3
- added link block_3_2, mass 0; visual box size=1.0 1.0 0.3
- added link block_3_3, mass 0; visual box size=1.0 1.0 0.3
Joints:
- removed joint joint_block_7_0
- removed joint joint_block_7_1
- removed joint joint_block_7_2
- removed joint joint_block_7_3
- removed joint joint_block_7_4
- removed joint joint_block_7_5
- removed joint joint_block_7_6
- removed joint joint_block_7_7
- removed joint joint_block_7_8
- removed joint joint_block_7_9
- added joint joint_block_3_0: type fixed, parent struct_base, child block_3_0, origin xyz=-1.5 -1.5 0.15 rpy=0 0 0
- added joint joint_block_3_1: type fixed, parent struct_base, child block_3_1, origin xyz=-0.5 -1.5 0.15 rpy=0 0 0
- added joint joint_block_3_2: type fixed, parent struct_base, child block_3_2, origin xyz=0.5 -1.5 0.15 rpy=0 0 0
- added joint joint_block_3_3: type fixed, parent struct_base, child block_3_3, origin xyz=1.5 -1.5 0.15 rpy=0 0 0

File: assets/warehouse/shelves.urdf (robot description, URDF)
Before this commit: robot struct, 10 links, 9 joints
Links:
- removed link block_5_1
- removed link block_5_2
- removed link block_5_3
- removed link block_5_4
- removed link block_5_5
- removed link block_5_6
- removed link block_5_7
- removed link block_5_8
- removed link block_5_9
- added link block_2_1, mass 0; collision box size=0.7 0.7 0.7; visual box size=1.0 1.0 1
- added link block_2_2, mass 0; collision box size=0.7 0.7 0.7; visual box size=1.0 1.0 1
- added link block_2_3, mass 0; collision box size=0.7 0.7 0.7; visual box size=1.0 1.0 1
Joints:
- removed joint joint_block_5_1
- removed joint joint_block_5_2
- removed joint joint_block_5_3
- removed joint joint_block_5_4
- removed joint joint_block_5_5
- removed joint joint_block_5_6
- removed joint joint_block_5_7
- removed joint joint_block_5_8
- removed joint joint_block_5_9
- added joint joint_block_2_1: type fixed, parent struct_base, child block_2_1, origin xyz=-0.5 -0.5 0.5 rpy=0 0 0
- added joint joint_block_2_2: type fixed, parent struct_base, child block_2_2, origin xyz=0.5 -0.5 0.5 rpy=0 0 0
- added joint joint_block_2_3: type fixed, parent struct_base, child block_2_3, origin xyz=1.5 -0.5 0.5 rpy=0 0 0

File: assets/warehouse/wall.urdf (robot description, URDF)
Before this commit: robot struct, 41 links, 40 joints
Links:
- removed link block_0_10
- removed link block_0_11
- removed link block_0_6
- removed link block_0_7
- removed link block_0_8
- removed link block_0_9
- removed link block_1_11
- removed link block_2_11
- removed link block_3_11
- removed link block_4_11
- removed link block_5_11
- removed link block_6_0
- removed link block_6_11
- removed link block_7_0
- removed link block_7_11
- removed link block_8_0
- removed link block_8_11
- removed link block_9_0
- removed link block_9_1
- removed link block_9_10
- removed link block_9_11
- removed link block_9_2
- removed link block_9_3
- removed link block_9_4
- removed link block_9_5
- removed link block_9_6
- removed link block_9_7
- removed link block_9_8
- removed link block_9_9
- added link block_1_5, mass 0; collision box size=1.0 1.0 3.0; visual box size=1.0 1.0 3
- added link block_2_5, mass 0; collision box size=1.0 1.0 3.0; visual box size=1.0 1.0 3
- added link block_3_5, mass 0; collision box size=1.0 1.0 3.0; visual box size=1.0 1.0 3
- added link block_4_5, mass 0; collision box size=1.0 1.0 3.0; visual box size=1.0 1.0 3
- added link block_5_1, mass 0; collision box size=1.0 1.0 3.0; visual box size=1.0 1.0 3
- added link block_5_2, mass 0; collision box size=1.0 1.0 3.0; visual box size=1.0 1.0 3
- added link block_5_3, mass 0; collision box size=1.0 1.0 3.0; visual box size=1.0 1.0 3
- added link block_5_4, mass 0; collision box size=1.0 1.0 3.0; visual box size=1.0 1.0 3
- added link block_5_5, mass 0; collision box size=1.0 1.0 3.0; visual box size=1.0 1.0 3
Joints:
- removed joint joint_block_0_10
- removed joint joint_block_0_11
- removed joint joint_block_0_6
- removed joint joint_block_0_7
- removed joint joint_block_0_8
- removed joint joint_block_0_9
- removed joint joint_block_1_11
- removed joint joint_block_2_11
- removed joint joint_block_3_11
- removed joint joint_block_4_11
- removed joint joint_block_5_11
- removed joint joint_block_6_0
- removed joint joint_block_6_11
- removed joint joint_block_7_0
- removed joint joint_block_7_11
- removed joint joint_block_8_0
- removed joint joint_block_8_11
- removed joint joint_block_9_0
- removed joint joint_block_9_1
- removed joint joint_block_9_10
- removed joint joint_block_9_11
- removed joint joint_block_9_2
- removed joint joint_block_9_3
- removed joint joint_block_9_4
- removed joint joint_block_9_5
- removed joint joint_block_9_6
- removed joint joint_block_9_7
- removed joint joint_block_9_8
- removed joint joint_block_9_9
- added joint joint_block_1_5: type fixed, parent struct_base, child block_1_5, origin xyz=2.5 1.5 1.5 rpy=0 0 0
- added joint joint_block_2_5: type fixed, parent struct_base, child block_2_5, origin xyz=2.5 0.5 1.5 rpy=0 0 0
- added joint joint_block_3_5: type fixed, parent struct_base, child block_3_5, origin xyz=2.5 -0.5 1.5 rpy=0 0 0
- added joint joint_block_4_5: type fixed, parent struct_base, child block_4_5, origin xyz=2.5 -1.5 1.5 rpy=0 0 0
- added joint joint_block_5_1: type fixed, parent struct_base, child block_5_1, origin xyz=-1.5 -2.5 1.5 rpy=0 0 0
- added joint joint_block_5_2: type fixed, parent struct_base, child block_5_2, origin xyz=-0.5 -2.5 1.5 rpy=0 0 0
- added joint joint_block_5_3: type fixed, parent struct_base, child block_5_3, origin xyz=0.5 -2.5 1.5 rpy=0 0 0
- added joint joint_block_5_4: type fixed, parent struct_base, child block_5_4, origin xyz=1.5 -2.5 1.5 rpy=0 0 0
- added joint joint_block_5_5: type fixed, parent struct_base, child block_5_5, origin xyz=2.5 -2.5 1.5 rpy=0 0 0
- joint joint_block_0_0: origin xyz=-5.5 4.5 1.5 rpy=0 0 0 -> xyz=-2.5 2.5 1.5 rpy=0 0 0
- joint joint_block_0_1: origin xyz=-4.5 4.5 1.5 rpy=0 0 0 -> xyz=-1.5 2.5 1.5 rpy=0 0 0
- joint joint_block_0_2: origin xyz=-3.5 4.5 1.5 rpy=0 0 0 -> xyz=-0.5 2.5 1.5 rpy=0 0 0
- joint joint_block_0_3: origin xyz=-2.5 4.5 1.5 rpy=0 0 0 -> xyz=0.5 2.5 1.5 rpy=0 0 0
- joint joint_block_0_4: origin xyz=-1.5 4.5 1.5 rpy=0 0 0 -> xyz=1.5 2.5 1.5 rpy=0 0 0
- joint joint_block_0_5: origin xyz=-0.5 4.5 1.5 rpy=0 0 0 -> xyz=2.5 2.5 1.5 rpy=0 0 0
- joint joint_block_1_0: origin xyz=-5.5 3.5 1.5 rpy=0 0 0 -> xyz=-2.5 1.5 1.5 rpy=0 0 0
- joint joint_block_2_0: origin xyz=-5.5 2.5 1.5 rpy=0 0 0 -> xyz=-2.5 0.5 1.5 rpy=0 0 0
- joint joint_block_3_0: origin xyz=-5.5 1.5 1.5 rpy=0 0 0 -> xyz=-2.5 -0.5 1.5 rpy=0 0 0
- joint joint_block_4_0: origin xyz=-5.5 0.5 1.5 rpy=0 0 0 -> xyz=-2.5 -1.5 1.5 rpy=0 0 0
- joint joint_block_5_0: origin xyz=-5.5 -0.5 1.5 rpy=0 0 0 -> xyz=-2.5 -2.5 1.5 rpy=0 0 0

File: assets/warehouse/workstations.urdf (robot description, URDF)
Before this commit: robot struct, 11 links, 10 joints
Links:
- removed link block_0_4
- removed link block_0_5
- removed link block_0_6
- removed link block_0_7
- removed link block_0_8
- removed link block_0_9
Joints:
- removed joint joint_block_0_4
- removed joint joint_block_0_5
- removed joint joint_block_0_6
- removed joint joint_block_0_7
- removed joint joint_block_0_8
- removed joint joint_block_0_9
- joint joint_block_0_0: origin xyz=-4.5 3.5 0.75 rpy=0 0 0 -> xyz=-1.5 1.5 0.75 rpy=0 0 0
- joint joint_block_0_1: origin xyz=-3.5 3.5 0.75 rpy=0 0 0 -> xyz=-0.5 1.5 0.75 rpy=0 0 0
- joint joint_block_0_2: origin xyz=-2.5 3.5 0.75 rpy=0 0 0 -> xyz=0.5 1.5 0.75 rpy=0 0 0
- joint joint_block_0_3: origin xyz=-1.5 3.5 0.75 rpy=0 0 0 -> xyz=1.5 1.5 0.75 rpy=0 0 0

Commit message: replace endpoint allocation rng with replace=True for consistency, add new warehouse layouts

File: assets/warehouse/endpoints.urdf (robot description, URDF)
Before this commit: robot struct, 5 links, 4 joints
Links:
- removed link block_3_0
- removed link block_3_1
- removed link block_3_2
- removed link block_3_3
- added link block_1_0, mass 0; visual box size=1.0 1.0 0.3
- added link block_1_1, mass 0; visual box size=1.0 1.0 0.3
- added link block_1_2, mass 0; visual box size=1.0 1.0 0.3
- added link block_1_3, mass 0; visual box size=1.0 1.0 0.3
Joints:
- removed joint joint_block_3_0
- removed joint joint_block_3_1
- removed joint joint_block_3_2
- removed joint joint_block_3_3
- added joint joint_block_1_0: type fixed, parent struct_base, child block_1_0, origin xyz=-1.5 0.5 0.15 rpy=0 0 0
- added joint joint_block_1_1: type fixed, parent struct_base, child block_1_1, origin xyz=-0.5 0.5 0.15 rpy=0 0 0
- added joint joint_block_1_2: type fixed, parent struct_base, child block_1_2, origin xyz=0.5 0.5 0.15 rpy=0 0 0
- added joint joint_block_1_3: type fixed, parent struct_base, child block_1_3, origin xyz=1.5 0.5 0.15 rpy=0 0 0

File: assets/warehouse/shelves.urdf (robot description, URDF)
Before this commit: robot struct, 4 links, 3 joints
Links:
- added link block_2_0, mass 0; collision box size=0.7 0.7 0.7; visual box size=1.0 1.0 1
Joints:
- added joint joint_block_2_0: type fixed, parent struct_base, child block_2_0, origin xyz=-1.5 -0.5 0.5 rpy=0 0 0
