Commit message: add improved metrics like grid_time to standardize timings

File: assets/warehouse/endpoints.urdf (robot description, URDF)
Before this commit: robot struct, 5 links, 4 joints
Links:
- removed link block_1_1
- removed link block_1_2
- removed link block_2_1
- removed link block_2_2
- added link block_0_10, mass 0; visual box size=1.0 1.0 0.3
- added link block_0_3, mass 0; visual box size=1.0 1.0 0.3
- added link block_0_6, mass 0; visual box size=1.0 1.0 0.3
- added link block_0_7, mass 0; visual box size=1.0 1.0 0.3
- added link block_10_10, mass 0; visual box size=1.0 1.0 0.3
- added link block_10_3, mass 0; visual box size=1.0 1.0 0.3
- added link block_10_6, mass 0; visual box size=1.0 1.0 0.3
- added link block_10_7, mass 0; visual box size=1.0 1.0 0.3
- added link block_11_10, mass 0; visual box size=1.0 1.0 0.3
- added link block_11_3, mass 0; visual box size=1.0 1.0 0.3
- added link block_11_6, mass 0; visual box size=1.0 1.0 0.3
- added link block_11_7, mass 0; visual box size=1.0 1.0 0.3
- added link block_12_10, mass 0; visual box size=1.0 1.0 0.3
- added link block_12_3, mass 0; visual box size=1.0 1.0 0.3
- added link block_12_6, mass 0; visual box size=1.0 1.0 0.3
- added link block_12_7, mass 0; visual box size=1.0 1.0 0.3
- added link block_13_10, mass 0; visual box size=1.0 1.0 0.3
- added link block_13_3, mass 0; visual box size=1.0 1.0 0.3
- added link block_13_6, mass 0; visual box size=1.0 1.0 0.3
- added link block_13_7, mass 0; visual box size=1.0 1.0 0.3
- added link block_14_10, mass 0; visual box size=1.0 1.0 0.3
- added link block_14_3, mass 0; visual box size=1.0 1.0 0.3
- added link block_14_6, mass 0; visual box size=1.0 1.0 0.3
- added link block_14_7, mass 0; visual box size=1.0 1.0 0.3
- added link block_15_10, mass 0; visual box size=1.0 1.0 0.3
- added link block_15_3, mass 0; visual box size=1.0 1.0 0.3
- added link block_15_6, mass 0; visual box size=1.0 1.0 0.3
- added link block_15_7, mass 0; visual box size=1.0 1.0 0.3
- added link block_16_10, mass 0; visual box size=1.0 1.0 0.3
- added link block_16_3, mass 0; visual box size=1.0 1.0 0.3
- added link block_16_6, mass 0; visual box size=1.0 1.0 0.3
- added link block_16_7, mass 0; visual box size=1.0 1.0 0.3
- added link block_17_10, mass 0; visual box size=1.0 1.0 0.3
- added link block_17_3, mass 0; visual box size=1.0 1.0 0.3
- added link block_17_6, mass 0; visual box size=1.0 1.0 0.3
- added link block_17_7, mass 0; visual box size=1.0 1.0 0.3
- added link block_1_10, mass 0; visual box size=1.0 1.0 0.3
- added link block_1_3, mass 0; visual box size=1.0 1.0 0.3
- added link block_1_6, mass 0; visual box size=1.0 1.0 0.3
- added link block_1_7, mass 0; visual box size=1.0 1.0 0.3
- added link block_2_10, mass 0; visual box size=1.0 1.0 0.3
- added link block_2_3, mass 0; visual box size=1.0 1.0 0.3
- added link block_2_6, mass 0; visual box size=1.0 1.0 0.3
- added link block_2_7, mass 0; visual box size=1.0 1.0 0.3
- added link block_3_10, mass 0; visual box size=1.0 1.0 0.3
- added link block_3_3, mass 0; visual box size=1.0 1.0 0.3
- added link block_3_6, mass 0; visual box size=1.0 1.0 0.3
- added link block_3_7, mass 0; visual box size=1.0 1.0 0.3
- added link block_4_10, mass 0; visual box size=1.0 1.0 0.3
- added link block_4_3, mass 0; visual box size=1.0 1.0 0.3
- added link block_4_6, mass 0; visual box size=1.0 1.0 0.3
- added link block_4_7, mass 0; visual box size=1.0 1.0 0.3
- added link block_5_10, mass 0; visual box size=1.0 1.0 0.3
- added link block_5_3, mass 0; visual box size=1.0 1.0 0.3
- added link block_5_6, mass 0; visual box size=1.0 1.0 0.3
- added link block_5_7, mass 0; visual box size=1.0 1.0 0.3
- added link block_6_10, mass 0; visual box size=1.0 1.0 0.3
- added link block_6_3, mass 0; visual box size=1.0 1.0 0.3
- added link block_6_6, mass 0; visual box size=1.0 1.0 0.3
- added link block_6_7, mass 0; visual box size=1.0 1.0 0.3
- added link block_7_10, mass 0; visual box size=1.0 1.0 0.3
- added link block_7_3, mass 0; visual box size=1.0 1.0 0.3
- added link block_7_6, mass 0; visual box size=1.0 1.0 0.3
- added link block_7_7, mass 0; visual box size=1.0 1.0 0.3
Joints:
- removed joint joint_block_1_1
- removed joint joint_block_1_2
- removed joint joint_block_2_1
- removed joint joint_block_2_2
- added joint joint_block_0_10: type fixed, parent struct_base, child block_0_10, origin xyz=3.5 8.5 0.15 rpy=0 0 0
- added joint joint_block_0_3: type fixed, parent struct_base, child block_0_3, origin xyz=-3.5 8.5 0.15 rpy=0 0 0
- added joint joint_block_0_6: type fixed, parent struct_base, child block_0_6, origin xyz=-0.5 8.5 0.15 rpy=0 0 0
- added joint joint_block_0_7: type fixed, parent struct_base, child block_0_7, origin xyz=0.5 8.5 0.15 rpy=0 0 0
- added joint joint_block_10_10: type fixed, parent struct_base, child block_10_10, origin xyz=3.5 -1.5 0.15 rpy=0 0 0
- added joint joint_block_10_3: type fixed, parent struct_base, child block_10_3, origin xyz=-3.5 -1.5 0.15 rpy=0 0 0
- added joint joint_block_10_6: type fixed, parent struct_base, child block_10_6, origin xyz=-0.5 -1.5 0.15 rpy=0 0 0
- added joint joint_block_10_7: type fixed, parent struct_base, child block_10_7, origin xyz=0.5 -1.5 0.15 rpy=0 0 0
- added joint joint_block_11_10: type fixed, parent struct_base, child block_11_10, origin xyz=3.5 -2.5 0.15 rpy=0 0 0
- added joint joint_block_11_3: type fixed, parent struct_base, child block_11_3, origin xyz=-3.5 -2.5 0.15 rpy=0 0 0
- added joint joint_block_11_6: type fixed, parent struct_base, child block_11_6, origin xyz=-0.5 -2.5 0.15 rpy=0 0 0
- added joint joint_block_11_7: type fixed, parent struct_base, child block_11_7, origin xyz=0.5 -2.5 0.15 rpy=0 0 0
- added joint joint_block_12_10: type fixed, parent struct_base, child block_12_10, origin xyz=3.5 -3.5 0.15 rpy=0 0 0
- added joint joint_block_12_3: type fixed, parent struct_base, child block_12_3, origin xyz=-3.5 -3.5 0.15 rpy=0 0 0
- added joint joint_block_12_6: type fixed, parent struct_base, child block_12_6, origin xyz=-0.5 -3.5 0.15 rpy=0 0 0
- added joint joint_block_12_7: type fixed, parent struct_base, child block_12_7, origin xyz=0.5 -3.5 0.15 rpy=0 0 0
- added joint joint_block_13_10: type fixed, parent struct_base, child block_13_10, origin xyz=3.5 -4.5 0.15 rpy=0 0 0
- added joint joint_block_13_3: type fixed, parent struct_base, child block_13_3, origin xyz=-3.5 -4.5 0.15 rpy=0 0 0
- added joint joint_block_13_6: type fixed, parent struct_base, child block_13_6, origin xyz=-0.5 -4.5 0.15 rpy=0 0 0
- added joint joint_block_13_7: type fixed, parent struct_base, child block_13_7, origin xyz=0.5 -4.5 0.15 rpy=0 0 0
- added joint joint_block_14_10: type fixed, parent struct_base, child block_14_10, origin xyz=3.5 -5.5 0.15 rpy=0 0 0
- added joint joint_block_14_3: type fixed, parent struct_base, child block_14_3, origin xyz=-3.5 -5.5 0.15 rpy=0 0 0
- added joint joint_block_14_6: type fixed, parent struct_base, child block_14_6, origin xyz=-0.5 -5.5 0.15 rpy=0 0 0
- added joint joint_block_14_7: type fixed, parent struct_base, child block_14_7, origin xyz=0.5 -5.5 0.15 rpy=0 0 0
- added joint joint_block_15_10: type fixed, parent struct_base, child block_15_10, origin xyz=3.5 -6.5 0.15 rpy=0 0 0
- added joint joint_block_15_3: type fixed, parent struct_base, child block_15_3, origin xyz=-3.5 -6.5 0.15 rpy=0 0 0
- added joint joint_block_15_6: type fixed, parent struct_base, child block_15_6, origin xyz=-0.5 -6.5 0.15 rpy=0 0 0
- added joint joint_block_15_7: type fixed, parent struct_base, child block_15_7, origin xyz=0.5 -6.5 0.15 rpy=0 0 0
- added joint joint_block_16_10: type fixed, parent struct_base, child block_16_10, origin xyz=3.5 -7.5 0.15 rpy=0 0 0
- added joint joint_block_16_3: type fixed, parent struct_base, child block_16_3, origin xyz=-3.5 -7.5 0.15 rpy=0 0 0
- added joint joint_block_16_6: type fixed, parent struct_base, child block_16_6, origin xyz=-0.5 -7.5 0.15 rpy=0 0 0
- added joint joint_block_16_7: type fixed, parent struct_base, child block_16_7, origin xyz=0.5 -7.5 0.15 rpy=0 0 0
- added joint joint_block_17_10: type fixed, parent struct_base, child block_17_10, origin xyz=3.5 -8.5 0.15 rpy=0 0 0
- added joint joint_block_17_3: type fixed, parent struct_base, child block_17_3, origin xyz=-3.5 -8.5 0.15 rpy=0 0 0
- added joint joint_block_17_6: type fixed, parent struct_base, child block_17_6, origin xyz=-0.5 -8.5 0.15 rpy=0 0 0
- added joint joint_block_17_7: type fixed, parent struct_base, child block_17_7, origin xyz=0.5 -8.5 0.15 rpy=0 0 0
- added joint joint_block_1_10: type fixed, parent struct_base, child block_1_10, origin xyz=3.5 7.5 0.15 rpy=0 0 0
- added joint joint_block_1_3: type fixed, parent struct_base, child block_1_3, origin xyz=-3.5 7.5 0.15 rpy=0 0 0
- added joint joint_block_1_6: type fixed, parent struct_base, child block_1_6, origin xyz=-0.5 7.5 0.15 rpy=0 0 0
- added joint joint_block_1_7: type fixed, parent struct_base, child block_1_7, origin xyz=0.5 7.5 0.15 rpy=0 0 0
- added joint joint_block_2_10: type fixed, parent struct_base, child block_2_10, origin xyz=3.5 6.5 0.15 rpy=0 0 0
- added joint joint_block_2_3: type fixed, parent struct_base, child block_2_3, origin xyz=-3.5 6.5 0.15 rpy=0 0 0
- added joint joint_block_2_6: type fixed, parent struct_base, child block_2_6, origin xyz=-0.5 6.5 0.15 rpy=0 0 0
- added joint joint_block_2_7: type fixed, parent struct_base, child block_2_7, origin xyz=0.5 6.5 0.15 rpy=0 0 0
- added joint joint_block_3_10: type fixed, parent struct_base, child block_3_10, origin xyz=3.5 5.5 0.15 rpy=0 0 0
- added joint joint_block_3_3: type fixed, parent struct_base, child block_3_3, origin xyz=-3.5 5.5 0.15 rpy=0 0 0
- added joint joint_block_3_6: type fixed, parent struct_base, child block_3_6, origin xyz=-0.5 5.5 0.15 rpy=0 0 0
- added joint joint_block_3_7: type fixed, parent struct_base, child block_3_7, origin xyz=0.5 5.5 0.15 rpy=0 0 0
- added joint joint_block_4_10: type fixed, parent struct_base, child block_4_10, origin xyz=3.5 4.5 0.15 rpy=0 0 0
- added joint joint_block_4_3: type fixed, parent struct_base, child block_4_3, origin xyz=-3.5 4.5 0.15 rpy=0 0 0
- added joint joint_block_4_6: type fixed, parent struct_base, child block_4_6, origin xyz=-0.5 4.5 0.15 rpy=0 0 0
- added joint joint_block_4_7: type fixed, parent struct_base, child block_4_7, origin xyz=0.5 4.5 0.15 rpy=0 0 0
- added joint joint_block_5_10: type fixed, parent struct_base, child block_5_10, origin xyz=3.5 3.5 0.15 rpy=0 0 0
- added joint joint_block_5_3: type fixed, parent struct_base, child block_5_3, origin xyz=-3.5 3.5 0.15 rpy=0 0 0
- added joint joint_block_5_6: type fixed, parent struct_base, child block_5_6, origin xyz=-0.5 3.5 0.15 rpy=0 0 0
- added joint joint_block_5_7: type fixed, parent struct_base, child block_5_7, origin xyz=0.5 3.5 0.15 rpy=0 0 0
- added joint joint_block_6_10: type fixed, parent struct_base, child block_6_10, origin xyz=3.5 2.5 0.15 rpy=0 0 0
- added joint joint_block_6_3: type fixed, parent struct_base, child block_6_3, origin xyz=-3.5 2.5 0.15 rpy=0 0 0
- added joint joint_block_6_6: type fixed, parent struct_base, child block_6_6, origin xyz=-0.5 2.5 0.15 rpy=0 0 0
- added joint joint_block_6_7: type fixed, parent struct_base, child block_6_7, origin xyz=0.5 2.5 0.15 rpy=0 0 0
- added joint joint_block_7_10: type fixed, parent struct_base, child block_7_10, origin xyz=3.5 1.5 0.15 rpy=0 0 0
- added joint joint_block_7_3: type fixed, parent struct_base, child block_7_3, origin xyz=-3.5 1.5 0.15 rpy=0 0 0
- added joint joint_block_7_6: type fixed, parent struct_base, child block_7_6, origin xyz=-0.5 1.5 0.15 rpy=0 0 0
- added joint joint_block_7_7: type fixed, parent struct_base, child block_7_7, origin xyz=0.5 1.5 0.15 rpy=0 0 0
