Commit message: add improved metrics like grid_time to standardize timings

File: assets/warehouse/shelves.urdf (robot description, URDF)
Before this commit: robot struct, 5 links, 4 joints
Links:
- removed link block_0_0
- removed link block_0_3
- removed link block_3_0
- removed link block_3_3
- added link block_0_4, mass 0; collision box size=0.7 0.7 0.7; visual box size=1.0 1.0 1
- added link block_0_5, mass 0; collision box size=0.7 0.7 0.7; visual box size=1.0 1.0 1
- added link block_0_8, mass 0; collision box size=0.7 0.7 0.7; visual box size=1.0 1.0 1
- added link block_0_9, mass 0; collision box size=0.7 0.7 0.7; visual box size=1.0 1.0 1
- added link block_10_4, mass 0; collision box size=0.7 0.7 0.7; visual box size=1.0 1.0 1
- added link block_10_5, mass 0; collision box size=0.7 0.7 0.7; visual box size=1.0 1.0 1
- added link block_10_8, mass 0; collision box size=0.7 0.7 0.7; visual box size=1.0 1.0 1
- added link block_10_9, mass 0; collision box size=0.7 0.7 0.7; visual box size=1.0 1.0 1
- added link block_11_4, mass 0; collision box size=0.7 0.7 0.7; visual box size=1.0 1.0 1
- added link block_11_5, mass 0; collision box size=0.7 0.7 0.7; visual box size=1.0 1.0 1
- added link block_11_8, mass 0; collision box size=0.7 0.7 0.7; visual box size=1.0 1.0 1
- added link block_11_9, mass 0; collision box size=0.7 0.7 0.7; visual box size=1.0 1.0 1
- added link block_12_4, mass 0; collision box size=0.7 0.7 0.7; visual box size=1.0 1.0 1
- added link block_12_5, mass 0; collision box size=0.7 0.7 0.7; visual box size=1.0 1.0 1
- added link block_12_8, mass 0; collision box size=0.7 0.7 0.7; visual box size=1.0 1.0 1
- added link block_12_9, mass 0; collision box size=0.7 0.7 0.7; visual box size=1.0 1.0 1
- added link block_13_4, mass 0; collision box size=0.7 0.7 0.7; visual box size=1.0 1.0 1
- added link block_13_5, mass 0; collision box size=0.7 0.7 0.7; visual box size=1.0 1.0 1
- added link block_13_8, mass 0; collision box size=0.7 0.7 0.7; visual box size=1.0 1.0 1
- added link block_13_9, mass 0; collision box size=0.7 0.7 0.7; visual box size=1.0 1.0 1
- added link block_14_4, mass 0; collision box size=0.7 0.7 0.7; visual box size=1.0 1.0 1
- added link block_14_5, mass 0; collision box size=0.7 0.7 0.7; visual box size=1.0 1.0 1
- added link block_14_8, mass 0; collision box size=0.7 0.7 0.7; visual box size=1.0 1.0 1
- added link block_14_9, mass 0; collision box size=0.7 0.7 0.7; visual box size=1.0 1.0 1
- added link block_15_4, mass 0; collision box size=0.7 0.7 0.7; visual box size=1.0 1.0 1
- added link block_15_5, mass 0; collision box size=0.7 0.7 0.7; visual box size=1.0 1.0 1
- added link block_15_8, mass 0; collision box size=0.7 0.7 0.7; visual box size=1.0 1.0 1
- added link block_15_9, mass 0; collision box size=0.7 0.7 0.7; visual box size=1.0 1.0 1
- added link block_16_4, mass 0; collision box size=0.7 0.7 0.7; visual box size=1.0 1.0 1
- added link block_16_5, mass 0; collision box size=0.7 0.7 0.7; visual box size=1.0 1.0 1
- added link block_16_8, mass 0; collision box size=0.7 0.7 0.7; visual box size=1.0 1.0 1
- added link block_16_9, mass 0; collision box size=0.7 0.7 0.7; visual box size=1.0 1.0 1
- added link block_17_4, mass 0; collision box size=0.7 0.7 0.7; visual box size=1.0 1.0 1
- added link block_17_5, mass 0; collision box size=0.7 0.7 0.7; visual box size=1.0 1.0 1
- added link block_17_8, mass 0; collision box size=0.7 0.7 0.7; visual box size=1.0 1.0 1
- added link block_17_9, mass 0; collision box size=0.7 0.7 0.7; visual box size=1.0 1.0 1
- added link block_1_4, mass 0; collision box size=0.7 0.7 0.7; visual box size=1.0 1.0 1
- added link block_1_5, mass 0; collision box size=0.7 0.7 0.7; visual box size=1.0 1.0 1
- added link block_1_8, mass 0; collision box size=0.7 0.7 0.7; visual box size=1.0 1.0 1
- added link block_1_9, mass 0; collision box size=0.7 0.7 0.7; visual box size=1.0 1.0 1
- added link block_2_4, mass 0; collision box size=0.7 0.7 0.7; visual box size=1.0 1.0 1
- added link block_2_5, mass 0; collision box size=0.7 0.7 0.7; visual box size=1.0 1.0 1
- added link block_2_8, mass 0; collision box size=0.7 0.7 0.7; visual box size=1.0 1.0 1
- added link block_2_9, mass 0; collision box size=0.7 0.7 0.7; visual box size=1.0 1.0 1
- added link block_3_4, mass 0; collision box size=0.7 0.7 0.7; visual box size=1.0 1.0 1
- added link block_3_5, mass 0; collision box size=0.7 0.7 0.7; visual box size=1.0 1.0 1
- added link block_3_8, mass 0; collision box size=0.7 0.7 0.7; visual box size=1.0 1.0 1
- added link block_3_9, mass 0; collision box size=0.7 0.7 0.7; visual box size=1.0 1.0 1
- added link block_4_4, mass 0; collision box size=0.7 0.7 0.7; visual box size=1.0 1.0 1
- added link block_4_5, mass 0; collision box size=0.7 0.7 0.7; visual box size=1.0 1.0 1
- added link block_4_8, mass 0; collision box size=0.7 0.7 0.7; visual box size=1.0 1.0 1
- added link block_4_9, mass 0; collision box size=0.7 0.7 0.7; visual box size=1.0 1.0 1
- added link block_5_4, mass 0; collision box size=0.7 0.7 0.7; visual box size=1.0 1.0 1
- added link block_5_5, mass 0; collision box size=0.7 0.7 0.7; visual box size=1.0 1.0 1
- added link block_5_8, mass 0; collision box size=0.7 0.7 0.7; visual box size=1.0 1.0 1
- added link block_5_9, mass 0; collision box size=0.7 0.7 0.7; visual box size=1.0 1.0 1
- added link block_6_4, mass 0; collision box size=0.7 0.7 0.7; visual box size=1.0 1.0 1
- added link block_6_5, mass 0; collision box size=0.7 0.7 0.7; visual box size=1.0 1.0 1
- added link block_6_8, mass 0; collision box size=0.7 0.7 0.7; visual box size=1.0 1.0 1
- added link block_6_9, mass 0; collision box size=0.7 0.7 0.7; visual box size=1.0 1.0 1
- added link block_7_4, mass 0; collision box size=0.7 0.7 0.7; visual box size=1.0 1.0 1
- added link block_7_5, mass 0; collision box size=0.7 0.7 0.7; visual box size=1.0 1.0 1
- added link block_7_8, mass 0; collision box size=0.7 0.7 0.7; visual box size=1.0 1.0 1
- added link block_7_9, mass 0; collision box size=0.7 0.7 0.7; visual box size=1.0 1.0 1
Joints:
- removed joint joint_block_0_0
- removed joint joint_block_0_3
- removed joint joint_block_3_0
- removed joint joint_block_3_3
- added joint joint_block_0_4: type fixed, parent struct_base, child block_0_4, origin xyz=-2.5 8.5 0.5 rpy=0 0 0
- added joint joint_block_0_5: type fixed, parent struct_base, child block_0_5, origin xyz=-1.5 8.5 0.5 rpy=0 0 0
- added joint joint_block_0_8: type fixed, parent struct_base, child block_0_8, origin xyz=1.5 8.5 0.5 rpy=0 0 0
- added joint joint_block_0_9: type fixed, parent struct_base, child block_0_9, origin xyz=2.5 8.5 0.5 rpy=0 0 0
- added joint joint_block_10_4: type fixed, parent struct_base, child block_10_4, origin xyz=-2.5 -1.5 0.5 rpy=0 0 0
- added joint joint_block_10_5: type fixed, parent struct_base, child block_10_5, origin xyz=-1.5 -1.5 0.5 rpy=0 0 0
- added joint joint_block_10_8: type fixed, parent struct_base, child block_10_8, origin xyz=1.5 -1.5 0.5 rpy=0 0 0
- added joint joint_block_10_9: type fixed, parent struct_base, child block_10_9, origin xyz=2.5 -1.5 0.5 rpy=0 0 0
- added joint joint_block_11_4: type fixed, parent struct_base, child block_11_4, origin xyz=-2.5 -2.5 0.5 rpy=0 0 0
- added joint joint_block_11_5: type fixed, parent struct_base, child block_11_5, origin xyz=-1.5 -2.5 0.5 rpy=0 0 0
- added joint joint_block_11_8: type fixed, parent struct_base, child block_11_8, origin xyz=1.5 -2.5 0.5 rpy=0 0 0
- added joint joint_block_11_9: type fixed, parent struct_base, child block_11_9, origin xyz=2.5 -2.5 0.5 rpy=0 0 0
- added joint joint_block_12_4: type fixed, parent struct_base, child block_12_4, origin xyz=-2.5 -3.5 0.5 rpy=0 0 0
- added joint joint_block_12_5: type fixed, parent struct_base, child block_12_5, origin xyz=-1.5 -3.5 0.5 rpy=0 0 0
- added joint joint_block_12_8: type fixed, parent struct_base, child block_12_8, origin xyz=1.5 -3.5 0.5 rpy=0 0 0
- added joint joint_block_12_9: type fixed, parent struct_base, child block_12_9, origin xyz=2.5 -3.5 0.5 rpy=0 0 0
- added joint joint_block_13_4: type fixed, parent struct_base, child block_13_4, origin xyz=-2.5 -4.5 0.5 rpy=0 0 0
- added joint joint_block_13_5: type fixed, parent struct_base, child block_13_5, origin xyz=-1.5 -4.5 0.5 rpy=0 0 0
- added joint joint_block_13_8: type fixed, parent struct_base, child block_13_8, origin xyz=1.5 -4.5 0.5 rpy=0 0 0
- added joint joint_block_13_9: type fixed, parent struct_base, child block_13_9, origin xyz=2.5 -4.5 0.5 rpy=0 0 0
- added joint joint_block_14_4: type fixed, parent struct_base, child block_14_4, origin xyz=-2.5 -5.5 0.5 rpy=0 0 0
- added joint joint_block_14_5: type fixed, parent struct_base, child block_14_5, origin xyz=-1.5 -5.5 0.5 rpy=0 0 0
- added joint joint_block_14_8: type fixed, parent struct_base, child block_14_8, origin xyz=1.5 -5.5 0.5 rpy=0 0 0
- added joint joint_block_14_9: type fixed, parent struct_base, child block_14_9, origin xyz=2.5 -5.5 0.5 rpy=0 0 0
- added joint joint_block_15_4: type fixed, parent struct_base, child block_15_4, origin xyz=-2.5 -6.5 0.5 rpy=0 0 0
- added joint joint_block_15_5: type fixed, parent struct_base, child block_15_5, origin xyz=-1.5 -6.5 0.5 rpy=0 0 0
- added joint joint_block_15_8: type fixed, parent struct_base, child block_15_8, origin xyz=1.5 -6.5 0.5 rpy=0 0 0
- added joint joint_block_15_9: type fixed, parent struct_base, child block_15_9, origin xyz=2.5 -6.5 0.5 rpy=0 0 0
- added joint joint_block_16_4: type fixed, parent struct_base, child block_16_4, origin xyz=-2.5 -7.5 0.5 rpy=0 0 0
- added joint joint_block_16_5: type fixed, parent struct_base, child block_16_5, origin xyz=-1.5 -7.5 0.5 rpy=0 0 0
- added joint joint_block_16_8: type fixed, parent struct_base, child block_16_8, origin xyz=1.5 -7.5 0.5 rpy=0 0 0
- added joint joint_block_16_9: type fixed, parent struct_base, child block_16_9, origin xyz=2.5 -7.5 0.5 rpy=0 0 0
- added joint joint_block_17_4: type fixed, parent struct_base, child block_17_4, origin xyz=-2.5 -8.5 0.5 rpy=0 0 0
- added joint joint_block_17_5: type fixed, parent struct_base, child block_17_5, origin xyz=-1.5 -8.5 0.5 rpy=0 0 0
- added joint joint_block_17_8: type fixed, parent struct_base, child block_17_8, origin xyz=1.5 -8.5 0.5 rpy=0 0 0
- added joint joint_block_17_9: type fixed, parent struct_base, child block_17_9, origin xyz=2.5 -8.5 0.5 rpy=0 0 0
- added joint joint_block_1_4: type fixed, parent struct_base, child block_1_4, origin xyz=-2.5 7.5 0.5 rpy=0 0 0
- added joint joint_block_1_5: type fixed, parent struct_base, child block_1_5, origin xyz=-1.5 7.5 0.5 rpy=0 0 0
- added joint joint_block_1_8: type fixed, parent struct_base, child block_1_8, origin xyz=1.5 7.5 0.5 rpy=0 0 0
- added joint joint_block_1_9: type fixed, parent struct_base, child block_1_9, origin xyz=2.5 7.5 0.5 rpy=0 0 0
- added joint joint_block_2_4: type fixed, parent struct_base, child block_2_4, origin xyz=-2.5 6.5 0.5 rpy=0 0 0
- added joint joint_block_2_5: type fixed, parent struct_base, child block_2_5, origin xyz=-1.5 6.5 0.5 rpy=0 0 0
- added joint joint_block_2_8: type fixed, parent struct_base, child block_2_8, origin xyz=1.5 6.5 0.5 rpy=0 0 0
- added joint joint_block_2_9: type fixed, parent struct_base, child block_2_9, origin xyz=2.5 6.5 0.5 rpy=0 0 0
- added joint joint_block_3_4: type fixed, parent struct_base, child block_3_4, origin xyz=-2.5 5.5 0.5 rpy=0 0 0
- added joint joint_block_3_5: type fixed, parent struct_base, child block_3_5, origin xyz=-1.5 5.5 0.5 rpy=0 0 0
- added joint joint_block_3_8: type fixed, parent struct_base, child block_3_8, origin xyz=1.5 5.5 0.5 rpy=0 0 0
- added joint joint_block_3_9: type fixed, parent struct_base, child block_3_9, origin xyz=2.5 5.5 0.5 rpy=0 0 0
- added joint joint_block_4_4: type fixed, parent struct_base, child block_4_4, origin xyz=-2.5 4.5 0.5 rpy=0 0 0
- added joint joint_block_4_5: type fixed, parent struct_base, child block_4_5, origin xyz=-1.5 4.5 0.5 rpy=0 0 0
- added joint joint_block_4_8: type fixed, parent struct_base, child block_4_8, origin xyz=1.5 4.5 0.5 rpy=0 0 0
- added joint joint_block_4_9: type fixed, parent struct_base, child block_4_9, origin xyz=2.5 4.5 0.5 rpy=0 0 0
- added joint joint_block_5_4: type fixed, parent struct_base, child block_5_4, origin xyz=-2.5 3.5 0.5 rpy=0 0 0
- added joint joint_block_5_5: type fixed, parent struct_base, child block_5_5, origin xyz=-1.5 3.5 0.5 rpy=0 0 0
- added joint joint_block_5_8: type fixed, parent struct_base, child block_5_8, origin xyz=1.5 3.5 0.5 rpy=0 0 0
- added joint joint_block_5_9: type fixed, parent struct_base, child block_5_9, origin xyz=2.5 3.5 0.5 rpy=0 0 0
- added joint joint_block_6_4: type fixed, parent struct_base, child block_6_4, origin xyz=-2.5 2.5 0.5 rpy=0 0 0
- added joint joint_block_6_5: type fixed, parent struct_base, child block_6_5, origin xyz=-1.5 2.5 0.5 rpy=0 0 0
- added joint joint_block_6_8: type fixed, parent struct_base, child block_6_8, origin xyz=1.5 2.5 0.5 rpy=0 0 0
- added joint joint_block_6_9: type fixed, parent struct_base, child block_6_9, origin xyz=2.5 2.5 0.5 rpy=0 0 0
- added joint joint_block_7_4: type fixed, parent struct_base, child block_7_4, origin xyz=-2.5 1.5 0.5 rpy=0 0 0
- added joint joint_block_7_5: type fixed, parent struct_base, child block_7_5, origin xyz=-1.5 1.5 0.5 rpy=0 0 0
- added joint joint_block_7_8: type fixed, parent struct_base, child block_7_8, origin xyz=1.5 1.5 0.5 rpy=0 0 0
- added joint joint_block_7_9: type fixed, parent struct_base, child block_7_9, origin xyz=2.5 1.5 0.5 rpy=0 0 0

File: assets/warehouse/workstations.urdf (robot description, URDF)
Before this commit: robot struct, 9 links, 8 joints
Links:
- removed link block_0_1
- removed link block_0_2
- removed link block_1_3
- removed link block_2_0
- removed link block_2_3
- removed link block_3_1
- removed link block_3_2
- added link block_10_0, mass 0; visual box size=1.0 1.0 1.5
- added link block_10_13, mass 0; visual box size=1.0 1.0 1.5
- added link block_13_0, mass 0; visual box size=1.0 1.0 1.5
- added link block_13_13, mass 0; visual box size=1.0 1.0 1.5
- added link block_16_0, mass 0; visual box size=1.0 1.0 1.5
- added link block_16_13, mass 0; visual box size=1.0 1.0 1.5
- added link block_1_13, mass 0; visual box size=1.0 1.0 1.5
- added link block_4_0, mass 0; visual box size=1.0 1.0 1.5
- added link block_4_13, mass 0; visual box size=1.0 1.0 1.5
- added link block_7_0, mass 0; visual box size=1.0 1.0 1.5
- added link block_7_13, mass 0; visual box size=1.0 1.0 1.5
Joints:
- removed joint joint_block_0_1
- removed joint joint_block_0_2
- removed joint joint_block_1_3
- removed joint joint_block_2_0
- removed joint joint_block_2_3
- removed joint joint_block_3_1
- removed joint joint_block_3_2
- added joint joint_block_10_0: type fixed, parent struct_base, child block_10_0, origin xyz=-6.5 -1.5 0.75 rpy=0 0 0
- added joint joint_block_10_13: type fixed, parent struct_base, child block_10_13, origin xyz=6.5 -1.5 0.75 rpy=0 0 0
- added joint joint_block_13_0: type fixed, parent struct_base, child block_13_0, origin xyz=-6.5 -4.5 0.75 rpy=0 0 0
- added joint joint_block_13_13: type fixed, parent struct_base, child block_13_13, origin xyz=6.5 -4.5 0.75 rpy=0 0 0
- added joint joint_block_16_0: type fixed, parent struct_base, child block_16_0, origin xyz=-6.5 -7.5 0.75 rpy=0 0 0
- added joint joint_block_16_13: type fixed, parent struct_base, child block_16_13, origin xyz=6.5 -7.5 0.75 rpy=0 0 0
- added joint joint_block_1_13: type fixed, parent struct_base, child block_1_13, origin xyz=6.5 7.5 0.75 rpy=0 0 0
- added joint joint_block_4_0: type fixed, parent struct_base, child block_4_0, origin xyz=-6.5 4.5 0.75 rpy=0 0 0
- added joint joint_block_4_13: type fixed, parent struct_base, child block_4_13, origin xyz=6.5 4.5 0.75 rpy=0 0 0
- added joint joint_block_7_0: type fixed, parent struct_base, child block_7_0, origin xyz=-6.5 1.5 0.75 rpy=0 0 0
- added joint joint_block_7_13: type fixed, parent struct_base, child block_7_13, origin xyz=6.5 1.5 0.75 rpy=0 0 0
- joint joint_block_1_0: origin xyz=-1.5 0.5 0.75 rpy=0 0 0 -> xyz=-6.5 7.5 0.75 rpy=0 0 0
