Commit message: cleanup unused code, add readme

File: assets/warehouse/endpoints.urdf (robot description, URDF)
Before this commit: robot struct, 421 links, 420 joints
Links:
- removed link block_12_10
- removed link block_12_11
- removed link block_12_13
- removed link block_12_14
- removed link block_12_15
- removed link block_12_16
- removed link block_12_17
- removed link block_12_18
- removed link block_12_19
- removed link block_12_2
- removed link block_12_20
- removed link block_12_21
- removed link block_12_22
- removed link block_12_24
- removed link block_12_25
- removed link block_12_26
- removed link block_12_27
- removed link block_12_28
- removed link block_12_29
- removed link block_12_3
- removed link block_12_30
- removed link block_12_31
- removed link block_12_32
- removed link block_12_33
- removed link block_12_4
- removed link block_12_5
- removed link block_12_6
- removed link block_12_7
- removed link block_12_8
- removed link block_12_9
- removed link block_13_10
- removed link block_13_11
- removed link block_13_13
- removed link block_13_14
- removed link block_13_15
- removed link block_13_16
- removed link block_13_17
- removed link block_13_18
- removed link block_13_19
- removed link block_13_2
- removed link block_13_20
- removed link block_13_21
- removed link block_13_22
- removed link block_13_24
- removed link block_13_25
- removed link block_13_26
- removed link block_13_27
- removed link block_13_28
- removed link block_13_29
- removed link block_13_3
- removed link block_13_30
- removed link block_13_31
- removed link block_13_32
- removed link block_13_33
- removed link block_13_4
- removed link block_13_5
- removed link block_13_6
- removed link block_13_7
- removed link block_13_8
- removed link block_13_9
- removed link block_16_10
- removed link block_16_11
- removed link block_16_13
- removed link block_16_14
- removed link block_16_15
- removed link block_16_16
- removed link block_16_17
- removed link block_16_18
- removed link block_16_19
- removed link block_16_2
- removed link block_16_20
- removed link block_16_21
- removed link block_16_22
- removed link block_16_24
- removed link block_16_25
- removed link block_16_26
- removed link block_16_27
- removed link block_16_28
- removed link block_16_29
- removed link block_16_3
- removed link block_16_30
- removed link block_16_31
- removed link block_16_32
- removed link block_16_33
- removed link block_16_4
- removed link block_16_5
- removed link block_16_6
- removed link block_16_7
- removed link block_16_8
- removed link block_16_9
- removed link block_17_10
- removed link block_17_11
- removed link block_17_13
- removed link block_17_14
- removed link block_17_15
- removed link block_17_16
- removed link block_17_17
- removed link block_17_18
- removed link block_17_19
- removed link block_17_2
- removed link block_17_20
- removed link block_17_21
- removed link block_17_22
- removed link block_17_24
- removed link block_17_25
- removed link block_17_26
- removed link block_17_27
- removed link block_17_28
- removed link block_17_29
- removed link block_17_3
- removed link block_17_30
- removed link block_17_31
- removed link block_17_32
- removed link block_17_33
- removed link block_17_4
- removed link block_17_5
- removed link block_17_6
- removed link block_17_7
- removed link block_17_8
- removed link block_17_9
- removed link block_1_10
- removed link block_1_11
- removed link block_1_13
- removed link block_1_14
- removed link block_1_15
- removed link block_1_16
- removed link block_1_17
- removed link block_1_18
- removed link block_1_19
- removed link block_1_20
- removed link block_1_21
- removed link block_1_22
- removed link block_1_24
- removed link block_1_25
- removed link block_1_26
- removed link block_1_27
- removed link block_1_28
- removed link block_1_29
- removed link block_1_3
- removed link block_1_30
- removed link block_1_31
- removed link block_1_32
- removed link block_1_33
- removed link block_1_4
- removed link block_1_5
- removed link block_1_6
- removed link block_1_7
- removed link block_1_8
- removed link block_1_9
- removed link block_20_10
- removed link block_20_11
- removed link block_20_13
- removed link block_20_14
- removed link block_20_15
- removed link block_20_16
- removed link block_20_17
- removed link block_20_18
- removed link block_20_19
- removed link block_20_2
- removed link block_20_20
- removed link block_20_21
- removed link block_20_22
- removed link block_20_24
- removed link block_20_25
- removed link block_20_26
- removed link block_20_27
- removed link block_20_28
- removed link block_20_29
- removed link block_20_3
- removed link block_20_30
- removed link block_20_31
- removed link block_20_32
- removed link block_20_33
- removed link block_20_4
- removed link block_20_5
- removed link block_20_6
- removed link block_20_7
- removed link block_20_8
- removed link block_20_9
- removed link block_21_10
- removed link block_21_11
- removed link block_21_13
- removed link block_21_14
- removed link block_21_15
- removed link block_21_16
- removed link block_21_17
- removed link block_21_18
- removed link block_21_19
- removed link block_21_2
- removed link block_21_20
- removed link block_21_21
- removed link block_21_22
- removed link block_21_24
- removed link block_21_25
- removed link block_21_26
- removed link block_21_27
- removed link block_21_28
- removed link block_21_29
- removed link block_21_3
- removed link block_21_30
- removed link block_21_31
- removed link block_21_32
- removed link block_21_33
- removed link block_21_4
- removed link block_21_5
- removed link block_21_6
- removed link block_21_7
- removed link block_21_8
- removed link block_21_9
- removed link block_24_10
- removed link block_24_11
- removed link block_24_13
- removed link block_24_14
- removed link block_24_15
- removed link block_24_16
- removed link block_24_17
- removed link block_24_18
- removed link block_24_19
- removed link block_24_2
- removed link block_24_20
- removed link block_24_21
- removed link block_24_22
- removed link block_24_24
- removed link block_24_25
- removed link block_24_26
- removed link block_24_27
- removed link block_24_28
- removed link block_24_29
- removed link block_24_3
- removed link block_24_30
- removed link block_24_31
- removed link block_24_32
- removed link block_24_33
- removed link block_24_4
- removed link block_24_5
- removed link block_24_6
- removed link block_24_7
- removed link block_24_8
- removed link block_24_9
- removed link block_25_10
- removed link block_25_11
- removed link block_25_13
- removed link block_25_14
- removed link block_25_15
- removed link block_25_16
- removed link block_25_17
- removed link block_25_18
- removed link block_25_19
- removed link block_25_2
- removed link block_25_20
- removed link block_25_21
- removed link block_25_22
- removed link block_25_24
- removed link block_25_25
- removed link block_25_26
- removed link block_25_27
- removed link block_25_28
- removed link block_25_29
- removed link block_25_3
- removed link block_25_30
- removed link block_25_31
- removed link block_25_32
- removed link block_25_33
- removed link block_25_4
- removed link block_25_5
- removed link block_25_6
- removed link block_25_7
- removed link block_25_8
- removed link block_25_9
- removed link block_28_10
- removed link block_28_11
- removed link block_28_13
- removed link block_28_14
- removed link block_28_15
- removed link block_28_16
- removed link block_28_17
- removed link block_28_18
- removed link block_28_19
- removed link block_28_2
- removed link block_28_20
- removed link block_28_21
- removed link block_28_22
- removed link block_28_24
- removed link block_28_25
- removed link block_28_26
- removed link block_28_27
- removed link block_28_28
- removed link block_28_29
- removed link block_28_3
- removed link block_28_30
- removed link block_28_31
- removed link block_28_32
- removed link block_28_33
- removed link block_28_4
- removed link block_28_5
- removed link block_28_6
- removed link block_28_7
- removed link block_28_8
- removed link block_28_9
- removed link block_4_10
- removed link block_4_11
- removed link block_4_13
- removed link block_4_14
- removed link block_4_15
- removed link block_4_16
- removed link block_4_17
- removed link block_4_18
- removed link block_4_19
- removed link block_4_2
- removed link block_4_20
- removed link block_4_21
- removed link block_4_22
- removed link block_4_24
- removed link block_4_25
- removed link block_4_26
- removed link block_4_27
- removed link block_4_28
- removed link block_4_29
- removed link block_4_3
- removed link block_4_30
- removed link block_4_31
- removed link block_4_32
- removed link block_4_33
- removed link block_4_4
- removed link block_4_5
- removed link block_4_6
- removed link block_4_7
- removed link block_4_8
- removed link block_4_9
- removed link block_5_10
- removed link block_5_11
- removed link block_5_13
- removed link block_5_14
- removed link block_5_15
- removed link block_5_16
- removed link block_5_17
- removed link block_5_18
- removed link block_5_19
- removed link block_5_2
- removed link block_5_20
- removed link block_5_21
- removed link block_5_22
- removed link block_5_24
- removed link block_5_25
- removed link block_5_26
- removed link block_5_27
- removed link block_5_28
- removed link block_5_29
- removed link block_5_3
- removed link block_5_30
- removed link block_5_31
- removed link block_5_32
- removed link block_5_33
- removed link block_5_4
- removed link block_5_5
- removed link block_5_6
- removed link block_5_7
- removed link block_5_8
- removed link block_5_9
- removed link block_8_10
- removed link block_8_11
- removed link block_8_13
- removed link block_8_14
- removed link block_8_15
- removed link block_8_16
- removed link block_8_17
- removed link block_8_18
- removed link block_8_19
- removed link block_8_2
- removed link block_8_20
- removed link block_8_21
- removed link block_8_22
- removed link block_8_24
- removed link block_8_25
- removed link block_8_26
- removed link block_8_27
- removed link block_8_28
- removed link block_8_29
- removed link block_8_3
- removed link block_8_30
- removed link block_8_31
- removed link block_8_32
- removed link block_8_33
- removed link block_8_4
- removed link block_8_5
- removed link block_8_6
- removed link block_8_7
- removed link block_8_8
- removed link block_8_9
- removed link block_9_10
- removed link block_9_11
- removed link block_9_13
- removed link block_9_14
- removed link block_9_15
- removed link block_9_16
- removed link block_9_17
- removed link block_9_18
- removed link block_9_19
- removed link block_9_2
- removed link block_9_20
- removed link block_9_21
- removed link block_9_22
- removed link block_9_24
- removed link block_9_25
- removed link block_9_26
- removed link block_9_27
- removed link block_9_28
- removed link block_9_29
- removed link block_9_3
- removed link block_9_30
- removed link block_9_31
- removed link block_9_32
- removed link block_9_33
- removed link block_9_4
- removed link block_9_5
- removed link block_9_6
- removed link block_9_7
- removed link block_9_8
- removed link block_9_9
- added link block_1_1, mass 0; visual box size=1.0 1.0 0.3
- added link block_2_1, mass 0; visual box size=1.0 1.0 0.3
- added link block_2_2, mass 0; visual box size=1.0 1.0 0.3
Joints:
- removed joint joint_block_12_10
- removed joint joint_block_12_11
- removed joint joint_block_12_13
- removed joint joint_block_12_14
- removed joint joint_block_12_15
- removed joint joint_block_12_16
- removed joint joint_block_12_17
- removed joint joint_block_12_18
- removed joint joint_block_12_19
- removed joint joint_block_12_2
- removed joint joint_block_12_20
- removed joint joint_block_12_21
- removed joint joint_block_12_22
- removed joint joint_block_12_24
- removed joint joint_block_12_25
- removed joint joint_block_12_26
- removed joint joint_block_12_27
- removed joint joint_block_12_28
- removed joint joint_block_12_29
- removed joint joint_block_12_3
- removed joint joint_block_12_30
- removed joint joint_block_12_31
- removed joint joint_block_12_32
- removed joint joint_block_12_33
- removed joint joint_block_12_4
- removed joint joint_block_12_5
- removed joint joint_block_12_6
- removed joint joint_block_12_7
- removed joint joint_block_12_8
- removed joint joint_block_12_9
- removed joint joint_block_13_10
- removed joint joint_block_13_11
- removed joint joint_block_13_13
- removed joint joint_block_13_14
- removed joint joint_block_13_15
- removed joint joint_block_13_16
- removed joint joint_block_13_17
- removed joint joint_block_13_18
- removed joint joint_block_13_19
- removed joint joint_block_13_2
- removed joint joint_block_13_20
- removed joint joint_block_13_21
- removed joint joint_block_13_22
- removed joint joint_block_13_24
- removed joint joint_block_13_25
- removed joint joint_block_13_26
- removed joint joint_block_13_27
- removed joint joint_block_13_28
- removed joint joint_block_13_29
- removed joint joint_block_13_3
- removed joint joint_block_13_30
- removed joint joint_block_13_31
- removed joint joint_block_13_32
- removed joint joint_block_13_33
- removed joint joint_block_13_4
- removed joint joint_block_13_5
- removed joint joint_block_13_6
- removed joint joint_block_13_7
- removed joint joint_block_13_8
- removed joint joint_block_13_9
- removed joint joint_block_16_10
- removed joint joint_block_16_11
- removed joint joint_block_16_13
- removed joint joint_block_16_14
- removed joint joint_block_16_15
- removed joint joint_block_16_16
- removed joint joint_block_16_17
- removed joint joint_block_16_18
- removed joint joint_block_16_19
- removed joint joint_block_16_2
- removed joint joint_block_16_20
- removed joint joint_block_16_21
- removed joint joint_block_16_22
- removed joint joint_block_16_24
- removed joint joint_block_16_25
- removed joint joint_block_16_26
- removed joint joint_block_16_27
- removed joint joint_block_16_28
- removed joint joint_block_16_29
- removed joint joint_block_16_3
- removed joint joint_block_16_30
- removed joint joint_block_16_31
- removed joint joint_block_16_32
- removed joint joint_block_16_33
- removed joint joint_block_16_4
- removed joint joint_block_16_5
- removed joint joint_block_16_6
- removed joint joint_block_16_7
- removed joint joint_block_16_8
- removed joint joint_block_16_9
- removed joint joint_block_17_10
- removed joint joint_block_17_11
- removed joint joint_block_17_13
- removed joint joint_block_17_14
- removed joint joint_block_17_15
- removed joint joint_block_17_16
- removed joint joint_block_17_17
- removed joint joint_block_17_18
- removed joint joint_block_17_19
- removed joint joint_block_17_2
- removed joint joint_block_17_20
- removed joint joint_block_17_21
- removed joint joint_block_17_22
- removed joint joint_block_17_24
- removed joint joint_block_17_25
- removed joint joint_block_17_26
- removed joint joint_block_17_27
- removed joint joint_block_17_28
- removed joint joint_block_17_29
- removed joint joint_block_17_3
- removed joint joint_block_17_30
- removed joint joint_block_17_31
- removed joint joint_block_17_32
- removed joint joint_block_17_33
- removed joint joint_block_17_4
- removed joint joint_block_17_5
- removed joint joint_block_17_6
- removed joint joint_block_17_7
- removed joint joint_block_17_8
- removed joint joint_block_17_9
- removed joint joint_block_1_10
- removed joint joint_block_1_11
- removed joint joint_block_1_13
- removed joint joint_block_1_14
- removed joint joint_block_1_15
- removed joint joint_block_1_16
- removed joint joint_block_1_17
- removed joint joint_block_1_18
- removed joint joint_block_1_19
- removed joint joint_block_1_20
- removed joint joint_block_1_21
- removed joint joint_block_1_22
- removed joint joint_block_1_24
- removed joint joint_block_1_25
- removed joint joint_block_1_26
- removed joint joint_block_1_27
- removed joint joint_block_1_28
- removed joint joint_block_1_29
- removed joint joint_block_1_3
- removed joint joint_block_1_30
- removed joint joint_block_1_31
- removed joint joint_block_1_32
- removed joint joint_block_1_33
- removed joint joint_block_1_4
- removed joint joint_block_1_5
- removed joint joint_block_1_6
- removed joint joint_block_1_7
- removed joint joint_block_1_8
- removed joint joint_block_1_9
- removed joint joint_block_20_10
- removed joint joint_block_20_11
- removed joint joint_block_20_13
- removed joint joint_block_20_14
- removed joint joint_block_20_15
- removed joint joint_block_20_16
- removed joint joint_block_20_17
- removed joint joint_block_20_18
- removed joint joint_block_20_19
- removed joint joint_block_20_2
- removed joint joint_block_20_20
- removed joint joint_block_20_21
- removed joint joint_block_20_22
- removed joint joint_block_20_24
- removed joint joint_block_20_25
- removed joint joint_block_20_26
- removed joint joint_block_20_27
- removed joint joint_block_20_28
- removed joint joint_block_20_29
- removed joint joint_block_20_3
- removed joint joint_block_20_30
- removed joint joint_block_20_31
- removed joint joint_block_20_32
- removed joint joint_block_20_33
- removed joint joint_block_20_4
- removed joint joint_block_20_5
- removed joint joint_block_20_6
- removed joint joint_block_20_7
- removed joint joint_block_20_8
- removed joint joint_block_20_9
- removed joint joint_block_21_10
- removed joint joint_block_21_11
- removed joint joint_block_21_13
- removed joint joint_block_21_14
- removed joint joint_block_21_15
- removed joint joint_block_21_16
- removed joint joint_block_21_17
- removed joint joint_block_21_18
- removed joint joint_block_21_19
- removed joint joint_block_21_2
- removed joint joint_block_21_20
- removed joint joint_block_21_21
- removed joint joint_block_21_22
- removed joint joint_block_21_24
- removed joint joint_block_21_25
- removed joint joint_block_21_26
- removed joint joint_block_21_27
- removed joint joint_block_21_28
- removed joint joint_block_21_29
- removed joint joint_block_21_3
- removed joint joint_block_21_30
- removed joint joint_block_21_31
- removed joint joint_block_21_32
- removed joint joint_block_21_33
- removed joint joint_block_21_4
- removed joint joint_block_21_5
- removed joint joint_block_21_6
- removed joint joint_block_21_7
- removed joint joint_block_21_8
- removed joint joint_block_21_9
- removed joint joint_block_24_10
- removed joint joint_block_24_11
- removed joint joint_block_24_13
- removed joint joint_block_24_14
- removed joint joint_block_24_15
- removed joint joint_block_24_16
- removed joint joint_block_24_17
- removed joint joint_block_24_18
- removed joint joint_block_24_19
- removed joint joint_block_24_2
- removed joint joint_block_24_20
- removed joint joint_block_24_21
- removed joint joint_block_24_22
- removed joint joint_block_24_24
- removed joint joint_block_24_25
- removed joint joint_block_24_26
- removed joint joint_block_24_27
- removed joint joint_block_24_28
- removed joint joint_block_24_29
- removed joint joint_block_24_3
- removed joint joint_block_24_30
- removed joint joint_block_24_31
- removed joint joint_block_24_32
- removed joint joint_block_24_33
- removed joint joint_block_24_4
- removed joint joint_block_24_5
- removed joint joint_block_24_6
- removed joint joint_block_24_7
- removed joint joint_block_24_8
- removed joint joint_block_24_9
- removed joint joint_block_25_10
- removed joint joint_block_25_11
- removed joint joint_block_25_13
- removed joint joint_block_25_14
- removed joint joint_block_25_15
- removed joint joint_block_25_16
- removed joint joint_block_25_17
- removed joint joint_block_25_18
- removed joint joint_block_25_19
- removed joint joint_block_25_2
- removed joint joint_block_25_20
- removed joint joint_block_25_21
- removed joint joint_block_25_22
- removed joint joint_block_25_24
- removed joint joint_block_25_25
- removed joint joint_block_25_26
- removed joint joint_block_25_27
- removed joint joint_block_25_28
- removed joint joint_block_25_29
- removed joint joint_block_25_3
- removed joint joint_block_25_30
- removed joint joint_block_25_31
- removed joint joint_block_25_32
- removed joint joint_block_25_33
- removed joint joint_block_25_4
- removed joint joint_block_25_5
- removed joint joint_block_25_6
- removed joint joint_block_25_7
- removed joint joint_block_25_8
- removed joint joint_block_25_9
- removed joint joint_block_28_10
- removed joint joint_block_28_11
- removed joint joint_block_28_13
- removed joint joint_block_28_14
- removed joint joint_block_28_15
- removed joint joint_block_28_16
- removed joint joint_block_28_17
- removed joint joint_block_28_18
- removed joint joint_block_28_19
- removed joint joint_block_28_2
- removed joint joint_block_28_20
- removed joint joint_block_28_21
- removed joint joint_block_28_22
- removed joint joint_block_28_24
- removed joint joint_block_28_25
- removed joint joint_block_28_26
- removed joint joint_block_28_27
- removed joint joint_block_28_28
- removed joint joint_block_28_29
- removed joint joint_block_28_3
- removed joint joint_block_28_30
- removed joint joint_block_28_31
- removed joint joint_block_28_32
- removed joint joint_block_28_33
- removed joint joint_block_28_4
- removed joint joint_block_28_5
- removed joint joint_block_28_6
- removed joint joint_block_28_7
- removed joint joint_block_28_8
- removed joint joint_block_28_9
- removed joint joint_block_4_10
- removed joint joint_block_4_11
- removed joint joint_block_4_13
- removed joint joint_block_4_14
- removed joint joint_block_4_15
- removed joint joint_block_4_16
- removed joint joint_block_4_17
- removed joint joint_block_4_18
- removed joint joint_block_4_19
- removed joint joint_block_4_2
- removed joint joint_block_4_20
- removed joint joint_block_4_21
- removed joint joint_block_4_22
- removed joint joint_block_4_24
- removed joint joint_block_4_25
- removed joint joint_block_4_26
- removed joint joint_block_4_27
- removed joint joint_block_4_28
- removed joint joint_block_4_29
- removed joint joint_block_4_3
- removed joint joint_block_4_30
- removed joint joint_block_4_31
- removed joint joint_block_4_32
- removed joint joint_block_4_33
- removed joint joint_block_4_4
- removed joint joint_block_4_5
- removed joint joint_block_4_6
- removed joint joint_block_4_7
- removed joint joint_block_4_8
- removed joint joint_block_4_9
- removed joint joint_block_5_10
- removed joint joint_block_5_11
- removed joint joint_block_5_13
- removed joint joint_block_5_14
- removed joint joint_block_5_15
- removed joint joint_block_5_16
- removed joint joint_block_5_17
- removed joint joint_block_5_18
- removed joint joint_block_5_19
- removed joint joint_block_5_2
- removed joint joint_block_5_20
- removed joint joint_block_5_21
- removed joint joint_block_5_22
- removed joint joint_block_5_24
- removed joint joint_block_5_25
- removed joint joint_block_5_26
- removed joint joint_block_5_27
- removed joint joint_block_5_28
- removed joint joint_block_5_29
- removed joint joint_block_5_3
- removed joint joint_block_5_30
- removed joint joint_block_5_31
- removed joint joint_block_5_32
- removed joint joint_block_5_33
- removed joint joint_block_5_4
- removed joint joint_block_5_5
- removed joint joint_block_5_6
- removed joint joint_block_5_7
- removed joint joint_block_5_8
- removed joint joint_block_5_9
- removed joint joint_block_8_10
- removed joint joint_block_8_11
- removed joint joint_block_8_13
- removed joint joint_block_8_14
- removed joint joint_block_8_15
- removed joint joint_block_8_16
- removed joint joint_block_8_17
- removed joint joint_block_8_18
- removed joint joint_block_8_19
- removed joint joint_block_8_2
- removed joint joint_block_8_20
- removed joint joint_block_8_21
- removed joint joint_block_8_22
- removed joint joint_block_8_24
- removed joint joint_block_8_25
- removed joint joint_block_8_26
- removed joint joint_block_8_27
- removed joint joint_block_8_28
- removed joint joint_block_8_29
- removed joint joint_block_8_3
- removed joint joint_block_8_30
- removed joint joint_block_8_31
- removed joint joint_block_8_32
- removed joint joint_block_8_33
- removed joint joint_block_8_4
- removed joint joint_block_8_5
- removed joint joint_block_8_6
- removed joint joint_block_8_7
- removed joint joint_block_8_8
- removed joint joint_block_8_9
- removed joint joint_block_9_10
- removed joint joint_block_9_11
- removed joint joint_block_9_13
- removed joint joint_block_9_14
- removed joint joint_block_9_15
- removed joint joint_block_9_16
- removed joint joint_block_9_17
- removed joint joint_block_9_18
- removed joint joint_block_9_19
- removed joint joint_block_9_2
- removed joint joint_block_9_20
- removed joint joint_block_9_21
- removed joint joint_block_9_22
- removed joint joint_block_9_24
- removed joint joint_block_9_25
- removed joint joint_block_9_26
- removed joint joint_block_9_27
- removed joint joint_block_9_28
- removed joint joint_block_9_29
- removed joint joint_block_9_3
- removed joint joint_block_9_30
- removed joint joint_block_9_31
- removed joint joint_block_9_32
- removed joint joint_block_9_33
- removed joint joint_block_9_4
- removed joint joint_block_9_5
- removed joint joint_block_9_6
- removed joint joint_block_9_7
- removed joint joint_block_9_8
- removed joint joint_block_9_9
- added joint joint_block_1_1: type fixed, parent struct_base, child block_1_1, origin xyz=-0.5 0.5 0.15 rpy=0 0 0
- added joint joint_block_2_1: type fixed, parent struct_base, child block_2_1, origin xyz=-0.5 -0.5 0.15 rpy=0 0 0
- added joint joint_block_2_2: type fixed, parent struct_base, child block_2_2, origin xyz=0.5 -0.5 0.15 rpy=0 0 0
- joint joint_block_1_2: origin xyz=-15.5 13.5 0.15 rpy=0 0 0 -> xyz=0.5 0.5 0.15 rpy=0 0 0
